File: hardware/control_panel/can.kicad_sch (KiCad schematic)
At the start: 20 parts, among them J4 Screw_Terminal_CAN, U2 74LVC1G57, U4 TJA1051T-3

Commit message: hw layout
Parts:
- D2: footprint Package_TO_SOT_SMD:SOT-23 -> Package_TO_SOT_SMD:SOT-23_Handsoldering
- U2: footprint Package_TO_SOT_SMD:SOT-563 -> Package_TO_SOT_SMD:SOT-363_SC-70-6
Connections:
- net VBUS: no longer C58.1, D1.1 (K)
- net Vin: now also C58.1, D1.1 (K)
Other:
- moved on the sheet: F1
Changed lines of the file:
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@@
   (junction (at 167.64 71.12) (diameter 0) (color 0 0 0 0)
   )
+  (wire (pts (xy 171.45 35.56) (xy 168.91 35.56))
+    (stroke (width 0) (type default))
+  )
   (wire (pts (xy 104.14 46.99) (xy 107.95 46.99))
     (stroke (width 0) (type default))
@@
     (stroke (width 0) (type default))
   )
+  (wire (pts (xy 171.45 33.02) (xy 171.45 35.56))
+    (stroke (width 0) (type default))
+  )
   (wire (pts (xy 167.64 101.6) (xy 167.64 107.95))
     (stroke (width 0) (type default))
@@
     (stroke (width 0) (type default))
   )
-  (wire (pts (xy 156.21 33.02) (xy 156.21 35.56))
+  (wire (pts (xy 156.21 35.56) (xy 161.29 35.56))
     (stroke (width 0) (type default))
   )
@@
     (stroke (width 0) (type default))
   )
-  (wire (pts (xy 144.78 35.56) (xy 147.32 35.56))
-    (stroke (width 0) (type default))
-  )
   (wire (pts (xy 229.87 107.95) (xy 229.87 105.41))
     (stroke (width 0) (type default))
@@
     (stroke (width 0) (type default))
   )
-  (wire (pts (xy 134.62 35.56) (xy 137.16 35.56))
+  (wire (pts (xy 134.62 35.56) (xy 147.32 35.56))
     (stroke (width 0) (type default))
   )
@@
     )
   )
-  (symbol (lib_id "Device:Fuse") (at 140.97 35.56 90) (unit 1)
-    (in_bom yes) (on_board yes) (dnp no) (fields_autoplaced)
-    (property "Reference" "F1" (at 140.97 31.0982 90)
-      (effects (font (size 1.27 1.27)))
-    )
-    (property "Value" "Fuse" (at 140.97 33.6351 90)
-      (effects (font (size 1.27 1.27)))
-    )
-    (property "Footprint" "Fuse:Fuse_1206_3216Metric_Pad1.42x1.75mm_HandSolder" (at 140.97 37.338 90)
-      (effects (font (size 1.27 1.27)) hide)
-    )
-    (property "Datasheet" "~" (at 140.97 35.56 0)
+  (symbol (lib_id "Device:Fuse") (at 165.1 35.56 90) (unit 1)
+    (in_bom yes) (on_board yes) (dnp no) (fields_autoplaced)
+    (property "Reference" "F1" (at 165.1 31.0982 90)
+      (effects (font (size 1.27 1.27)))
+    )
+    (property "Value" "Fuse" (at 165.1 33.6351 90)
+      (effects (font (size 1.27 1.27)))
+    )
+    (property "Footprint" "Fuse:Fuse_1206_3216Metric_Pad1.42x1.75mm_HandSolder" (at 165.1 37.338 90)
+      (effects (font (size 1.27 1.27)) hide)
+    )
+    (property "Datasheet" "~" (at 165.1 35.56 0)
       (effects (font (size 1.27 1.27)) hide)
     )
@@
       (effects (font (size 1.27 1.27)))
     )
-    (property "Footprint" "Package_TO_SOT_SMD:SOT-23" (at 157.48 80.01 0)
+    (property "Footprint" "Package_TO_SOT_SMD:SOT-23_Handsoldering" (at 157.48 80.01 0)
       (effects (font (size 1.27 1.27)) hide)
     )
@@
     )
   )
-  (symbol (lib_id "power:VBUS") (at 156.21 33.02 0) (unit 1)
-    (in_bom yes) (on_board yes) (dnp no) (fields_autoplaced)
-    (property "Reference" "#PWR0221" (at 156.21 36.83 0)
-      (effects (font (size 1.27 1.27)) hide)
-    )
-    (property "Value" "VBUS" (at 156.21 29.4442 0)
-      (effects (font (size 1.27 1.27)))
-    )
-    (property "Footprint" "" (at 156.21 33.02 0)
-      (effects (font (size 1.27 1.27)) hide)
-    )
-    (property "Datasheet" "" (at 156.21 33.02 0)
+  (symbol (lib_id "power:VBUS") (at 171.45 33.02 0) (unit 1)
+    (in_bom yes) (on_board yes) (dnp no) (fields_autoplaced)
+    (property "Reference" "#PWR0221" (at 171.45 36.83 0)
+      (effects (font (size 1.27 1.27)) hide)
+    )
+    (property "Value" "VBUS" (at 171.45 29.4442 0)
+      (effects (font (size 1.27 1.27)))
+    )
+    (property "Footprint" "" (at 171.45 33.02 0)
+      (effects (font (size 1.27 1.27)) hide)
+    )
+    (property "Datasheet" "" (at 171.45 33.02 0)
       (effects (font (size 1.27 1.27)) hide)
     )
@@
       (effects (font (size 1.27 1.27)))
     )
-    (property "Footprint" "Package_TO_SOT_SMD:SOT-563" (at 240.03 55.88 0)
-      (effects (font (size 1.27 1.27)) hide)
-    )
+    (property "Footprint" "Package_TO_SOT_SMD:SOT-363_SC-70-6" (at 240.03 55.88 0)
+      (effects (font (size 1.27 1.27)) hide)
+    )
