File: hardware/control_panel/pi_i2c.kicad_sch (KiCad schematic)
At the start: 20 parts, among them J14 Conn_01x07, J5 Screw_Terminal_01x04, U1 P82B96, U12 LM397

Commit message: hw layout
Parts:
- removed J14: Conn_01x07, Connector_PinHeader_2.54mm:PinHeader_1x07_P2.54mm_Vertical, symbol Connector_Generic:Conn_01x07
- D5, D6, D7: footprint Package_TO_SOT_SMD:SOT-23 -> Package_TO_SOT_SMD:SOT-23_Handsoldering
Changed lines of the file:
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@@
       (effects (font (size 1.27 1.27)))
     )
-    (property "Footprint" "Package_TO_SOT_SMD:SOT-23" (at 207.01 127 0)
+    (property "Footprint" "Package_TO_SOT_SMD:SOT-23_Handsoldering" (at 207.01 127 0)
       (effects (font (size 1.27 1.27)) hide)
     )
@@
     )
   )
-  (symbol (lib_id "Connector_Generic:Conn_01x07") (at 175.26 101.6 0) (mirror x) (unit 1)
-    (in_bom yes) (on_board yes) (dnp no)
-    (property "Reference" "J14" (at 177.8 102.87 0)
+  (symbol (lib_id "power:+5VD") (at 187.96 67.31 0) (unit 1)
+    (in_bom yes) (on_board yes) (dnp no) (fields_autoplaced)
+    (property "Reference" "#PWR04" (at 187.96 71.12 0)
+      (effects (font (size 1.27 1.27)) hide)
+    )
+    (property "Value" "+5VD" (at 187.96 63.754 0)
+      (effects (font (size 1.27 1.27)))
+    )
+    (property "Footprint" "" (at 187.96 67.31 0)
+      (effects (font (size 1.27 1.27)) hide)
+    )
+    (property "Datasheet" "" (at 187.96 67.31 0)
+      (effects (font (size 1.27 1.27)) hide)
+    )
+    (pin "1")
+    (instances
+      (project "control_panel"
+        (path "/e63e39d7-6ac0-4ffd-8aa3-1841a4541b55/8ca9797e-e63e-4e59-a184-ef2a887eb814"
+          (reference "#PWR04") (unit 1)
+        )
+      )
+    )
+  )
+  (symbol (lib_id "Device:C") (at 255.27 148.59 0) (unit 1)
+    (in_bom yes) (on_board yes) (dnp no) (fields_autoplaced)
+    (property "Reference" "C76" (at 258.191 147.7553 0)
       (effects (font (size 1.27 1.27)) (justify left))
     )
-    (property "Value" "Conn_01x07" (at 177.8 100.33 0)
+    (property "Value" "100n" (at 258.191 150.2922 0)
       (effects (font (size 1.27 1.27)) (justify left))
     )
-    (property "Footprint" "Connector_PinHeader_2.54mm:PinHeader_1x07_P2.54mm_Vertical" (at 175.26 101.6 0)
-      (effects (font (size 1.27 1.27)) hide)
-    )
-    (property "Datasheet" "~" (at 175.26 101.6 0)
+    (property "Footprint" "Capacitor_SMD:C_0603_1608Metric" (at 256.2352 152.4 0)
+      (effects (font (size 1.27 1.27)) hide)
+    )
+    (property "Datasheet" "~" (at 255.27 148.59 0)
+      (effects (font (size 1.27 1.27)) hide)
+    )
+    (pin "1")
+    (pin "2")
+    (instances
+      (project "control_panel"
+        (path "/e63e39d7-6ac0-4ffd-8aa3-1841a4541b55/8ca9797e-e63e-4e59-a184-ef2a887eb814"
+          (reference "C76") (unit 1)
+        )
+      )
+    )
+  )
+  (symbol (lib_id "Comparator:LM397") (at 224.79 148.59 0) (unit 1)
+    (in_bom yes) (on_board yes) (dnp no) (fields_autoplaced)
+    (property "Reference" "U12" (at 234.95 144.3991 0)
+      (effects (font (size 1.27 1.27)))
+    )
+    (property "Value" "LM397" (at 234.95 146.9391 0)
+      (effects (font (size 1.27 1.27)))
+    )
+    (property "Footprint" "Package_TO_SOT_SMD:SOT-23-5" (at 226.06 163.83 0)
+      (effects (font (size 1.27 1.27)) hide)
+    )
+    (property "Datasheet" "http://www.ti.com/lit/ds/symlink/lm397.pdf" (at 224.79 143.51 0)
       (effects (font (size 1.27 1.27)) hide)
     )
@@
     (pin "4")
     (pin "5")
-    (pin "6")
-    (pin "7")
-    (instances
-      (project "control_panel"
-        (path "/e63e39d7-6ac0-4ffd-8aa3-1841a4541b55/8ca9797e-e63e-4e59-a184-ef2a887eb814"
-          (reference "J14") (unit 1)
-        )
-      )
-    )
-  )
-  (symbol (lib_id "power:+5VD") (at 187.96 67.31 0) (unit 1)
-    (in_bom yes) (on_board yes) (dnp no) (fields_autoplaced)
-    (property "Reference" "#PWR04" (at 187.96 71.12 0)
-      (effects (font (size 1.27 1.27)) hide)
-    )
-    (property "Value" "+5VD" (at 187.96 63.754 0)
-      (effects (font (size 1.27 1.27)))
-    )
-    (property "Footprint" "" (at 187.96 67.31 0)
-      (effects (font (size 1.27 1.27)) hide)
-    )
-    (property "Datasheet" "" (at 187.96 67.31 0)
-      (effects (font (size 1.27 1.27)) hide)
-    )
-    (pin "1")
-    (instances
-      (project "control_panel"
-        (path "/e63e39d7-6ac0-4ffd-8aa3-1841a4541b55/8ca9797e-e63e-4e59-a184-ef2a887eb814"
-          (reference "#PWR04") (unit 1)
-        )
-      )
-    )
-  )
-  (symbol (lib_id "Device:C") (at 255.27 148.59 0) (unit 1)
-    (in_bom yes) (on_board yes) (dnp no) (fields_autoplaced)
-    (property "Reference" "C76" (at 258.191 147.7553 0)
-      (effects (font (size 1.27 1.27)) (justify left))
-    )
-    (property "Value" "100n" (at 258.191 150.2922 0)
-      (effects (font (size 1.27 1.27)) (justify left))
-    )
-    (property "Footprint" "Capacitor_SMD:C_0603_1608Metric" (at 256.2352 152.4 0)
-      (effects (font (size 1.27 1.27)) hide)
-    )
-    (property "Datasheet" "~" (at 255.27 148.59 0)
-      (effects (font (size 1.27 1.27)) hide)
-    )
-    (pin "1")
-    (pin "2")
-    (instances
-      (project "control_panel"
-        (path "/e63e39d7-6ac0-4ffd-8aa3-1841a4541b55/8ca9797e-e63e-4e59-a184-ef2a887eb814"
-          (reference "C76") (unit 1)
-        )
-      )
-    )
-  )
-  (symbol (lib_id "Comparator:LM397") (at 224.79 148.59 0) (unit 1)
-    (in_bom yes) (on_board yes) (dnp no) (fields_autoplaced)
-    (property "Reference" "U12" (at 234.95 144.3991 0)
-      (effects (font (size 1.27 1.27)))
-    )
-    (property "Value" "LM397" (at 234.95 146.9391 0)
-      (effects (font (size 1.27 1.27)))
-    )
-    (property "Footprint" "Package_TO_SOT_SMD:SOT-23-5" (at 226.06 163.83 0)
-      (effects (font (size 1.27 1.27)) hide)
-    )
-    (property "Datasheet" "http://www.ti.com/lit/ds/symlink/lm397.pdf" (at 224.79 143.51 0)
-      (effects (font (size 1.27 1.27)) hide)
-    )
-    (pin "1")
-    (pin "2")
-    (pin "3")
-    (pin "4")
-    (pin "5")
     (instances
       (project "control_panel"
@@
       (effects (font (size 1.27 1.27)))
     )
-    (property "Footprint" "Package_TO_SOT_SMD:SOT-23" (at 265.43 127 0)
+    (property "Footprint" "Package_TO_SOT_SMD:SOT-23_Handsoldering" (at 265.43 127 0)
       (effects (font (size 1.27 1.27)) hide)
     )
@@
       (effects (font (size 1.27 1.27)))
     )
-    (property "Footprint" "Package_TO_SOT_SMD:SOT-23" (at 176.53 140.97 0)
-      (effects (font (size 1.27 1.27)) hide)
-    )
+    (property "Footprint" "Package_TO_SOT_SMD:SOT-23_Handsoldering" (at 176.53 140.97 0)
+      (effects (font (size 1.27 1.27)) hide)
+    )
