File: hardware/control_panel/audio.kicad_sch (KiCad schematic)
At the start: 45 parts, among them J10 Conn_01x03, J7 Conn_01x02, J8 Conn_01x04, J9 Conn_01x03, U7 SPX3819M5-L-3-3, X1 SG-8002CE

Commit message: led balance and corridor ready
Parts:
- added TP1: RIN3, project_footprints:TestPoint_Pad_D1.5mm, symbol Connector:TestPoint
- added TP1: OUT3, project_footprints:TestPoint_Pad_D1.5mm, symbol Connector:TestPoint
- added TP1: HP_R, project_footprints:TestPoint_Pad_D1.5mm, symbol Connector:TestPoint
- added TP1: HP_L, project_footprints:TestPoint_Pad_D1.5mm, symbol Connector:TestPoint
- added TP1: LIN3, project_footprints:TestPoint_Pad_D1.5mm, symbol Connector:TestPoint
- DA1: footprint Package_DFN_QFN:QFN-32-1EP_5x5mm_P0.5mm_EP3.45x3.45mm_ThermalVias -> project_footprints:QFN-32-1EP_5x5mm_P0.5mm_EP3.45x3.45mm_ThermalVias; Addr 0x34 -> (none); I2C I2C addr -> (none); I2C address (none) -> 0x34
Connections:
- net HP_L: now also TP1.1
- net HP_R: now also TP1.1
- net LIN3: now also TP1.1
- net OUT3: now also TP1.1
- net RIN3: now also TP1.1
Changed lines of the file:
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@@
+    (stroke (width 0) (type default))
+  )
+  (wire (pts (xy 97.79 137.16) (xy 105.41 137.16))
+    (stroke (width 0) (type default))
+  )
+  (wire (pts (xy 97.79 134.62) (xy 105.41 134.62))
     (stroke (width 0) (type default))
   )
@@
     (stroke (width 0) (type default))
   )
-  (wire (pts (xy 48.26 168.91) (xy 50.8 168.91))
+  (wire (pts (xy 43.18 168.91) (xy 50.8 168.91))
     (stroke (width 0) (type default))
   )
@@
     (stroke (width 0) (type default))
   )
-  (wire (pts (xy 97.79 132.08) (xy 100.33 132.08))
+  (wire (pts (xy 97.79 132.08) (xy 105.41 132.08))
     (stroke (width 0) (type default))
   )
@@
     (stroke (width 0) (type default))
   )
-  (wire (pts (xy 48.26 161.29) (xy 50.8 161.29))
+  (wire (pts (xy 43.18 161.29) (xy 50.8 161.29))
     (stroke (width 0) (type default))
   )
@@
     (stroke (width 0) (type default))
   )
-  (wire (pts (xy 97.79 134.62) (xy 100.33 134.62))
-    (stroke (width 0) (type default))
-  )
   (wire (pts (xy 97.79 171.45) (xy 100.33 171.45))
     (stroke (width 0) (type default))
@@
   )
   (wire (pts (xy 48.26 118.11) (xy 50.8 118.11))
-    (stroke (width 0) (type default))
-  )
-  (wire (pts (xy 97.79 137.16) (xy 100.33 137.16))
     (stroke (width 0) (type default))
   )
@@
     )
   )
+  (symbol (lib_id "Connector:TestPoint") (at 43.18 168.91 90) (unit 1)
+    (in_bom no) (on_board yes) (dnp no)
+    (property "Reference" "TP1" (at 38.1 168.91 90)
+      (effects (font (size 1.27 1.27)) (justify left))
+    )
+    (property "Value" "RIN3" (at 33.02 168.91 90)
+      (effects (font (size 1.27 1.27)) (justify left))
+    )
+    (property "Footprint" "project_footprints:TestPoint_Pad_D1.5mm" (at 43.18 163.83 0)
+      (effects (font (size 1.27 1.27)) hide)
+    )
+    (property "Datasheet" "~" (at 43.18 163.83 0)
+      (effects (font (size 1.27 1.27)) hide)
+    )
+    (pin "1")
+    (instances
+      (project "control_panel"
+        (path "/e63e39d7-6ac0-4ffd-8aa3-1841a4541b55/17827faa-2bd7-4315-b62a-454e8ea9e1b3"
+          (reference "TP1") (unit 1)
+        )
+        (path "/e63e39d7-6ac0-4ffd-8aa3-1841a4541b55/de3cff99-a77a-4ec0-aa51-1947b344db19"
+          (reference "TP11") (unit 1)
+        )
+      )
+    )
+  )
   (symbol (lib_id "power:GND") (at 242.57 85.09 180) (unit 1)
     (in_bom yes) (on_board yes) (dnp no) (fields_autoplaced)
@@
     )
   )
+  (symbol (lib_id "Connector:TestPoint") (at 105.41 134.62 270) (unit 1)
+    (in_bom no) (on_board yes) (dnp no)
+    (property "Reference" "TP1" (at 110.49 134.62 90)
+      (effects (font (size 1.27 1.27)) (justify left))
+    )
+    (property "Value" "OUT3" (at 115.57 134.62 90)
+      (effects (font (size 1.27 1.27)) (justify left))
+    )
+    (property "Footprint" "project_footprints:TestPoint_Pad_D1.5mm" (at 105.41 139.7 0)
+      (effects (font (size 1.27 1.27)) hide)
+    )
+    (property "Datasheet" "~" (at 105.41 139.7 0)
+      (effects (font (size 1.27 1.27)) hide)
+    )
+    (pin "1")
+    (instances
+      (project "control_panel"
+        (path "/e63e39d7-6ac0-4ffd-8aa3-1841a4541b55/17827faa-2bd7-4315-b62a-454e8ea9e1b3"
+          (reference "TP1") (unit 1)
+        )
+        (path "/e63e39d7-6ac0-4ffd-8aa3-1841a4541b55/de3cff99-a77a-4ec0-aa51-1947b344db19"
+          (reference "TP8") (unit 1)
+        )
+      )
+    )
+  )
   (symbol (lib_id "Device:C") (at 243.84 53.34 90) (unit 1)
     (in_bom yes) (on_board yes) (dnp no) (fields_autoplaced)
@@
         (path "/e63e39d7-6ac0-4ffd-8aa3-1841a4541b55/de3cff99-a77a-4ec0-aa51-1947b344db19"
           (reference "C50") (unit 1)
+        )
+      )
+    )
+  )
+  (symbol (lib_id "Connector:TestPoint") (at 105.41 132.08 270) (unit 1)
+    (in_bom no) (on_board yes) (dnp no)
+    (property "Reference" "TP1" (at 110.49 132.08 90)
+      (effects (font (size 1.27 1.27)) (justify left))
+    )
+    (property "Value" "HP_R" (at 115.57 132.08 90)
+      (effects (font (size 1.27 1.27)) (justify left))
+    )
+    (property "Footprint" "project_footprints:TestPoint_Pad_D1.5mm" (at 105.41 137.16 0)
+      (effects (font (size 1.27 1.27)) hide)
+    )
+    (property "Datasheet" "~" (at 105.41 137.16 0)
+      (effects (font (size 1.27 1.27)) hide)
+    )
+    (pin "1")
+    (instances
+      (project "control_panel"
+        (path "/e63e39d7-6ac0-4ffd-8aa3-1841a4541b55/17827faa-2bd7-4315-b62a-454e8ea9e1b3"
+          (reference "TP1") (unit 1)
+        )
+        (path "/e63e39d7-6ac0-4ffd-8aa3-1841a4541b55/de3cff99-a77a-4ec0-aa51-1947b344db19"
+          (reference "TP7") (unit 1)
         )
       )
@@
       (effects (font (size 1.27 1.27)))
     )
-    (property "Footprint" "Package_DFN_QFN:QFN-32-1EP_5x5mm_P0.5mm_EP3.45x3.45mm_ThermalVias" (at 87.63 177.8 0)
+    (property "Footprint" "project_footprints:QFN-32-1EP_5x5mm_P0.5mm_EP3.45x3.45mm_ThermalVias" (at 87.63 177.8 0)
       (effects (font (size 1.27 1.27)) hide)
     )
@@
       (effects (font (size 1.27 1.27)) hide)
     )
-    (property "I2C" "I2C addr" (at 74.295 111.9972 0)
-      (effects (font (size 1.27 1.27)))
-    )
-    (property "Addr" "0x34" (at 74.295 114.5341 0)
+    (property "I2C address" "0x34" (at 74.295 111.9972 0) (show_name)
       (effects (font (size 1.27 1.27)))
     )
@@
     )
   )
+  (symbol (lib_id "Connector:TestPoint") (at 105.41 137.16 270) (unit 1)
+    (in_bom no) (on_board yes) (dnp no)
+    (property "Reference" "TP1" (at 110.49 137.16 90)
+      (effects (font (size 1.27 1.27)) (justify left))
+    )
+    (property "Value" "HP_L" (at 115.57 137.16 90)
+      (effects (font (size 1.27 1.27)) (justify left))
+    )
+    (property "Footprint" "project_footprints:TestPoint_Pad_D1.5mm" (at 105.41 142.24 0)
+      (effects (font (size 1.27 1.27)) hide)
+    )
+    (property "Datasheet" "~" (at 105.41 142.24 0)
+      (effects (font (size 1.27 1.27)) hide)
+    )
+    (pin "1")
+    (instances
+      (project "control_panel"
+        (path "/e63e39d7-6ac0-4ffd-8aa3-1841a4541b55/17827faa-2bd7-4315-b62a-454e8ea9e1b3"
+          (reference "TP1") (unit 1)
+        )
+        (path "/e63e39d7-6ac0-4ffd-8aa3-1841a4541b55/de3cff99-a77a-4ec0-aa51-1947b344db19"
+          (reference "TP9") (unit 1)
+        )
+      )
+    )
+  )
   (symbol (lib_id "power:GND") (at 139.7 101.6 0) (unit 1)
     (in_bom yes) (on_board yes) (dnp no) (fields_autoplaced)
@@
         )
       )
+    )
+  )
+  (symbol (lib_id "Connector:TestPoint") (at 43.18 161.29 90) (unit 1)
+    (in_bom no) (on_board yes) (dnp no)
+    (property "Reference" "TP1" (at 38.1 161.29 90)
+      (effects (font (size 1.27 1.27)) (justify left))
+    )
+    (property "Value" "LIN3" (at 33.02 161.29 90)
+      (effects (font (size 1.27 1.27)) (justify left))
+    )
+    (property "Footprint" "project_footprints:TestPoint_Pad_D1.5mm" (at 43.18 156.21 0)
+      (effects (font (size 1.27 1.27)) hide)
+    )
+    (property "Datasheet" "~" (at 43.18 156.21 0)
+      (effects (font (size 1.27 1.27)) hide)
+    )
+    (pin "1")
+    (instances
+      (project "control_panel"
+        (path "/e63e39d7-6ac0-4ffd-8aa3-1841a4541b55/17827faa-2bd7-4315-b62a-454e8ea9e1b3"
+          (reference "TP1") (unit 1)
+        )
+        (path "/e63e39d7-6ac0-4ffd-8aa3-1841a4541b55/de3cff99-a77a-4ec0-aa51-1947b344db19"
+          (reference "TP10") (unit 1)
+        )
+      )
