File: hardware/control_panel/mcu.kicad_sch (KiCad schematic)
At the start: 26 parts, among them J12 AVR-ISP-6, Q1 Q_Dual_NMOS_S1G1D2S2G2D1, SW1 SW_Push, U6 ATmega328PB-A, Y2 Crystal_GND24

Commit message: hw layout
Parts:
- added C13, C39: 1u, Capacitor_SMD:C_0603_1608Metric, symbol Device:C
- J12: footprint project_footprints:Tag-Connect_TC2030-IDC-NL_2x03_P1.27mm_Vertical -> Connector_PinHeader_2.54mm:PinHeader_2x03_P2.54mm_Vertical
Connections:
- net +5V: now also C13.2, C39.2
- net GND: now also C13.1, C39.1
- net IRQ: now also U6.3 (PE0); no longer U6.1 (PD3)
- net ~{INT}: now also U6.1 (PD3)
Changed lines of the file:
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@@
   (junction (at 252.73 68.58) (diameter 0) (color 0 0 0 0)
   )
+  (junction (at 68.58 46.99) (diameter 0) (color 0 0 0 0)
+  )
   (junction (at 34.29 99.06) (diameter 0) (color 0 0 0 0)
   )
@@
     (stroke (width 0) (type default))
   )
-  (wire (pts (xy 120.65 127) (xy 123.19 127))
+  (wire (pts (xy 120.65 127) (xy 128.27 127))
     (stroke (width 0) (type default))
   )
@@
     (effects (font (size 1.27 1.27)) (justify right bottom))
   )
-  (label "IRQ" (at 123.19 127 0) (fields_autoplaced)
-    (effects (font (size 1.27 1.27)) (justify left bottom))
+  (label "IRQ" (at 87.63 119.38 180) (fields_autoplaced)
+    (effects (font (size 1.27 1.27)) (justify right bottom))
   )
   (label "IRQ" (at 184.15 137.16 0) (fields_autoplaced)
@@
     (effects (font (size 1.27 1.27)) (justify right))
   )
-  (hierarchical_label "~{INT}" (shape input) (at 151.13 123.19 0) (fields_autoplaced)
+  (hierarchical_label "~{INT}" (shape input) (at 128.27 127 0) (fields_autoplaced)
     (effects (font (size 1.27 1.27)) (justify left))
   )
@@
         (path "/e63e39d7-6ac0-4ffd-8aa3-1841a4541b55/17827faa-2bd7-4315-b62a-454e8ea9e1b3"
           (reference "#PWR029") (unit 1)
+        )
+      )
+    )
+  )
+  (symbol (lib_id "power:+5V") (at 29.21 52.07 0) (unit 1)
+    (in_bom yes) (on_board yes) (dnp no)
+    (property "Reference" "#PWR048" (at 29.21 55.88 0)
+      (effects (font (size 1.27 1.27)) hide)
+    )
+    (property "Value" "+5V" (at 29.21 46.99 90)
+      (effects (font (size 1.27 1.27)))
+    )
+    (property "Footprint" "" (at 29.21 52.07 0)
+      (effects (font (size 1.27 1.27)) hide)
+    )
+    (property "Datasheet" "" (at 29.21 52.07 0)
+      (effects (font (size 1.27 1.27)) hide)
+    )
+    (pin "1")
+    (instances
+      (project "control_panel"
+        (path "/e63e39d7-6ac0-4ffd-8aa3-1841a4541b55/17827faa-2bd7-4315-b62a-454e8ea9e1b3"
+          (reference "#PWR048") (unit 1)
         )
       )
@@
     )
   )
+  (symbol (lib_id "power:GND") (at 68.58 54.61 0) (unit 1)
+    (in_bom yes) (on_board yes) (dnp no) (fields_autoplaced)
+    (property "Reference" "#PWR050" (at 68.58 60.96 0)
+      (effects (font (size 1.27 1.27)) hide)
+    )
+    (property "Value" "GND" (at 68.58 59.0534 0)
+      (effects (font (size 1.27 1.27)))
+    )
+    (property "Footprint" "" (at 68.58 54.61 0)
+      (effects (font (size 1.27 1.27)) hide)
+    )
+    (property "Datasheet" "" (at 68.58 54.61 0)
+      (effects (font (size 1.27 1.27)) hide)
+    )
+    (pin "1")
+    (instances
+      (project "control_panel"
+        (path "/e63e39d7-6ac0-4ffd-8aa3-1841a4541b55/17827faa-2bd7-4315-b62a-454e8ea9e1b3"
+          (reference "#PWR050") (unit 1)
+        )
+      )
+    )
+  )
   (symbol (lib_id "power:+5V") (at 232.41 123.19 0) (unit 1)
     (in_bom yes) (on_board yes) (dnp no)
@@
     )
   )
+  (symbol (lib_id "power:GND") (at 29.21 59.69 0) (unit 1)
+    (in_bom yes) (on_board yes) (dnp no) (fields_autoplaced)
+    (property "Reference" "#PWR049" (at 29.21 66.04 0)
+      (effects (font (size 1.27 1.27)) hide)
+    )
+    (property "Value" "GND" (at 29.21 64.1334 0)
+      (effects (font (size 1.27 1.27)))
+    )
+    (property "Footprint" "" (at 29.21 59.69 0)
+      (effects (font (size 1.27 1.27)) hide)
+    )
+    (property "Datasheet" "" (at 29.21 59.69 0)
+      (effects (font (size 1.27 1.27)) hide)
+    )
+    (pin "1")
+    (instances
+      (project "control_panel"
+        (path "/e63e39d7-6ac0-4ffd-8aa3-1841a4541b55/17827faa-2bd7-4315-b62a-454e8ea9e1b3"
+          (reference "#PWR049") (unit 1)
+        )
+      )
+    )
+  )
   (symbol (lib_id "power:GND") (at 232.41 177.8 0) (unit 1)
     (in_bom yes) (on_board yes) (dnp no) (fields_autoplaced)
@@
         (path "/e63e39d7-6ac0-4ffd-8aa3-1841a4541b55/17827faa-2bd7-4315-b62a-454e8ea9e1b3"
           (reference "#PWR033") (unit 1)
+        )
+      )
+    )
+  )
+  (symbol (lib_id "Device:C") (at 29.21 55.88 180) (unit 1)
+    (in_bom yes) (on_board yes) (dnp no) (fields_autoplaced)
+    (property "Reference" "C13" (at 33.02 54.61 0)
+      (effects (font (size 1.27 1.27)) (justify right))
+    )
+    (property "Value" "1u" (at 33.02 57.15 0)
+      (effects (font (size 1.27 1.27)) (justify right))
+    )
+    (property "Footprint" "Capacitor_SMD:C_0603_1608Metric" (at 28.2448 52.07 0)
+      (effects (font (size 1.27 1.27)) hide)
+    )
+    (property "Datasheet" "~" (at 29.21 55.88 0)
+      (effects (font (size 1.27 1.27)) hide)
+    )
+    (pin "1")
+    (pin "2")
+    (instances
+      (project "control_panel"
+        (path "/e63e39d7-6ac0-4ffd-8aa3-1841a4541b55/17827faa-2bd7-4315-b62a-454e8ea9e1b3"
+          (reference "C13") (unit 1)
         )
       )
@@
       (effects (font (size 1.27 1.27)) (justify right))
     )
-    (property "Footprint" "project_footprints:Tag-Connect_TC2030-IDC-NL_2x03_P1.27mm_Vertical" (at 201.93 55.88 90)
+    (property "Footprint" "Connector_PinHeader_2.54mm:PinHeader_2x03_P2.54mm_Vertical" (at 201.93 55.88 90)
       (effects (font (size 1.27 1.27)) hide)
     )
@@
         )
       )
+    )
+  )
+  (symbol (lib_id "Device:C") (at 68.58 50.8 180) (unit 1)
+    (in_bom yes) (on_board yes) (dnp no) (fields_autoplaced)
+    (property "Reference" "C39" (at 72.39 49.53 0)
+      (effects (font (size 1.27 1.27)) (justify right))
+    )
+    (property "Value" "1u" (at 72.39 52.07 0)
+      (effects (font (size 1.27 1.27)) (justify right))
+    )
+    (property "Footprint" "Capacitor_SMD:C_0603_1608Metric" (at 67.6148 46.99 0)
+      (effects (font (size 1.27 1.27)) hide)
+    )
+    (property "Datasheet" "~" (at 68.58 50.8 0)
+      (effects (font (size 1.27 1.27)) hide)
+    )
+    (pin "1")
+    (pin "2")
+    (instances
+      (project "control_panel"
+        (path "/e63e39d7-6ac0-4ffd-8aa3-1841a4541b55/17827faa-2bd7-4315-b62a-454e8ea9e1b3"
+          (reference "C39") (unit 1)
+        )
+      )

Commit message: led balance and corridor ready
Parts:
- added TP1: PB0, project_footprints:TestPoint_Pad_D1.5mm, symbol Connector:TestPoint
- added TP2: PD4, project_footprints:TestPoint_Pad_D1.5mm, symbol Connector:TestPoint
- added TP3: PD5, project_footprints:TestPoint_Pad_D1.5mm, symbol Connector:TestPoint
- added TP4: PD6, project_footprints:TestPoint_Pad_D1.5mm, symbol Connector:TestPoint
- added TP5: PD7, project_footprints:TestPoint_Pad_D1.5mm, symbol Connector:TestPoint
- added TP6: PE1, project_footprints:TestPoint_Pad_D1.5mm, symbol Connector:TestPoint
- Q1: value Q_Dual_NMOS_S1G1D2S2G2D1 -> 2N7002DW
Connections:
- net PEN: now also U6.14 (PB2)
- net RUN: now also U6.13 (PB1)
- net at U6.10 (PD6): now also TP4.1
- net at U6.12 (PB0): now also TP1.1
- net at U6.6 (PE1): now also TP6.1
- net at U6.9 (PD5): now also TP3.1
- net BT_0: no longer names the net of U6.2 (PD4)
- net BT_0: now also TP2.1
- net BT_1: no longer names the net of U6.11 (PD7)
- net BT_1: now also TP5.1
Changed lines of the file:
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@@
     (stroke (width 0) (type default))
   )
-  (wire (pts (xy 120.65 76.2) (xy 123.19 76.2))
+  (wire (pts (xy 120.65 76.2) (xy 127 76.2))
     (stroke (width 0) (type default))
   )
@@
     (stroke (width 0) (type default))
   )
-  (wire (pts (xy 87.63 121.92) (xy 90.17 121.92))
+  (wire (pts (xy 83.82 121.92) (xy 90.17 121.92))
     (stroke (width 0) (type default))
   )
@@
     (effects (font (size 1.27 1.27)) (justify left bottom))
   )
-  (label "BT_1" (at 123.19 137.16 0) (fields_autoplaced)
-    (effects (font (size 1.27 1.27)) (justify left bottom))
-  )
   (label "SDA" (at 123.19 109.22 0) (fields_autoplaced)
     (effects (font (size 1.27 1.27)) (justify left bottom))
@@
     (effects (font (size 1.27 1.27)) (justify right bottom))
   )
-  (label "BT_0" (at 123.19 129.54 0) (fields_autoplaced)
-    (effects (font (size 1.27 1.27)) (justify left bottom))
-  )
   (label "XTAL1" (at 154.94 95.25 180) (fields_autoplaced)
     (effects (font (size 1.27 1.27)) (justify right bottom))
@@
     (effects (font (size 1.27 1.27)) (justify left bottom))
   )
-  (label "PEN" (at 139.7 130.81 0) (fields_autoplaced)
+  (label "PEN" (at 123.19 81.28 0) (fields_autoplaced)
     (effects (font (size 1.27 1.27)) (justify left bottom))
   )
@@
     (effects (font (size 1.27 1.27)) (justify left bottom))
   )
-  (label "RUN" (at 139.7 96.52 0) (fields_autoplaced)
+  (label "RUN" (at 123.19 78.74 0) (fields_autoplaced)
     (effects (font (size 1.27 1.27)) (justify left bottom))
   )
@@
       (effects (font (size 1.27 1.27)) (justify left))
     )
-    (property "Value" "Q_Dual_NMOS_S1G1D2S2G2D1" (at 246.38 168.91 0)
+    (property "Value" "2N7002DW" (at 246.38 168.91 0)
       (effects (font (size 1.27 1.27)) (justify left))
     )
@@
     )
   )
+  (symbol (lib_id "Connector:TestPoint") (at 123.19 129.54 270) (unit 1)
+    (in_bom no) (on_board yes) (dnp no)
+    (property "Reference" "TP2" (at 128.27 129.54 90)
+      (effects (font (size 1.27 1.27)) (justify left))
+    )
+    (property "Value" "PD4" (at 133.35 129.54 90)
+      (effects (font (size 1.27 1.27)) (justify left))
+    )
+    (property "Footprint" "project_footprints:TestPoint_Pad_D1.5mm" (at 123.19 134.62 0)
+      (effects (font (size 1.27 1.27)) hide)
+    )
+    (property "Datasheet" "~" (at 123.19 134.62 0)
+      (effects (font (size 1.27 1.27)) hide)
+    )
+    (pin "1")
+    (instances
+      (project "control_panel"
+        (path "/e63e39d7-6ac0-4ffd-8aa3-1841a4541b55/17827faa-2bd7-4315-b62a-454e8ea9e1b3"
+          (reference "TP2") (unit 1)
+        )
+      )
+    )
+  )
   (symbol (lib_id "Device:R") (at 25.4 92.71 0) (unit 1)
     (in_bom yes) (on_board yes) (dnp no) (fields_autoplaced)
@@
         (path "/e63e39d7-6ac0-4ffd-8aa3-1841a4541b55/17827faa-2bd7-4315-b62a-454e8ea9e1b3"
           (reference "C69") (unit 1)
+        )
+      )
+    )
+  )
+  (symbol (lib_id "Connector:TestPoint") (at 83.82 121.92 90) (unit 1)
+    (in_bom no) (on_board yes) (dnp no) (fields_autoplaced)
+    (property "Reference" "TP6" (at 80.518 116.84 90)
+      (effects (font (size 1.27 1.27)))
+    )
+    (property "Value" "PE1" (at 80.518 119.38 90)
+      (effects (font (size 1.27 1.27)))
+    )
+    (property "Footprint" "project_footprints:TestPoint_Pad_D1.5mm" (at 83.82 116.84 0)
+      (effects (font (size 1.27 1.27)) hide)
+    )
+    (property "Datasheet" "~" (at 83.82 116.84 0)
+      (effects (font (size 1.27 1.27)) hide)
+    )
+    (pin "1")
+    (instances
+      (project "control_panel"
+        (path "/e63e39d7-6ac0-4ffd-8aa3-1841a4541b55/17827faa-2bd7-4315-b62a-454e8ea9e1b3"
+          (reference "TP6") (unit 1)
         )
       )
@@
     )
   )
+  (symbol (lib_id "Connector:TestPoint") (at 123.19 137.16 270) (unit 1)
+    (in_bom no) (on_board yes) (dnp no)
+    (property "Reference" "TP5" (at 128.27 137.16 90)
+      (effects (font (size 1.27 1.27)) (justify left))
+    )
+    (property "Value" "PD7" (at 133.35 137.16 90)
+      (effects (font (size 1.27 1.27)) (justify left))
+    )
+    (property "Footprint" "project_footprints:TestPoint_Pad_D1.5mm" (at 123.19 142.24 0)
+      (effects (font (size 1.27 1.27)) hide)
+    )
+    (property "Datasheet" "~" (at 123.19 142.24 0)
+      (effects (font (size 1.27 1.27)) hide)
+    )
+    (pin "1")
+    (instances
+      (project "control_panel"
+        (path "/e63e39d7-6ac0-4ffd-8aa3-1841a4541b55/17827faa-2bd7-4315-b62a-454e8ea9e1b3"
+          (reference "TP5") (unit 1)
+        )
+      )
+    )
+  )
   (symbol (lib_id "Device:R") (at 232.41 173.99 0) (unit 1)
     (in_bom yes) (on_board yes) (dnp no) (fields_autoplaced)
@@
         (path "/e63e39d7-6ac0-4ffd-8aa3-1841a4541b55/17827faa-2bd7-4315-b62a-454e8ea9e1b3"
           (reference "R30") (unit 1)
+        )
+      )
+    )
+  )
+  (symbol (lib_id "Connector:TestPoint") (at 123.19 134.62 270) (unit 1)
+    (in_bom no) (on_board yes) (dnp no)
+    (property "Reference" "TP4" (at 128.27 134.62 90)
+      (effects (font (size 1.27 1.27)) (justify left))
+    )
+    (property "Value" "PD6" (at 133.35 134.62 90)
+      (effects (font (size 1.27 1.27)) (justify left))
+    )
+    (property "Footprint" "project_footprints:TestPoint_Pad_D1.5mm" (at 123.19 139.7 0)
+      (effects (font (size 1.27 1.27)) hide)
+    )
+    (property "Datasheet" "~" (at 123.19 139.7 0)
+      (effects (font (size 1.27 1.27)) hide)
+    )
+    (pin "1")
+    (instances
+      (project "control_panel"
+        (path "/e63e39d7-6ac0-4ffd-8aa3-1841a4541b55/17827faa-2bd7-4315-b62a-454e8ea9e1b3"
+          (reference "TP4") (unit 1)
         )
       )
@@
         (path "/e63e39d7-6ac0-4ffd-8aa3-1841a4541b55/17827faa-2bd7-4315-b62a-454e8ea9e1b3"
           (reference "R40") (unit 1)
+        )
+      )
+    )
+  )
+  (symbol (lib_id "Connector:TestPoint") (at 123.19 132.08 270) (unit 1)
+    (in_bom no) (on_board yes) (dnp no)
+    (property "Reference" "TP3" (at 128.27 132.08 90)
+      (effects (font (size 1.27 1.27)) (justify left))
+    )
+    (property "Value" "PD5" (at 133.35 132.08 90)
+      (effects (font (size 1.27 1.27)) (justify left))
+    )
+    (property "Footprint" "project_footprints:TestPoint_Pad_D1.5mm" (at 123.19 137.16 0)
+      (effects (font (size 1.27 1.27)) hide)
+    )
+    (property "Datasheet" "~" (at 123.19 137.16 0)
+      (effects (font (size 1.27 1.27)) hide)
+    )
+    (pin "1")
+    (instances
+      (project "control_panel"
+        (path "/e63e39d7-6ac0-4ffd-8aa3-1841a4541b55/17827faa-2bd7-4315-b62a-454e8ea9e1b3"
+          (reference "TP3") (unit 1)
         )
       )
@@
     )
   )
+  (symbol (lib_id "Connector:TestPoint") (at 127 76.2 270) (unit 1)
+    (in_bom no) (on_board yes) (dnp no) (fields_autoplaced)
+    (property "Reference" "TP1" (at 132.08 74.93 90)
+      (effects (font (size 1.27 1.27)) (justify left))
+    )
+    (property "Value" "PB0" (at 132.08 77.47 90)
+      (effects (font (size 1.27 1.27)) (justify left))
+    )
+    (property "Footprint" "project_footprints:TestPoint_Pad_D1.5mm" (at 127 81.28 0)
+      (effects (font (size 1.27 1.27)) hide)
+    )
+    (property "Datasheet" "~" (at 127 81.28 0)
+      (effects (font (size 1.27 1.27)) hide)
+    )
+    (pin "1")
+    (instances
+      (project "control_panel"
+        (path "/e63e39d7-6ac0-4ffd-8aa3-1841a4541b55/17827faa-2bd7-4315-b62a-454e8ea9e1b3"
+          (reference "TP1") (unit 1)
+        )
+      )
+    )
+  )
   (symbol (lib_id "power:GND") (at 242.57 138.43 0) (unit 1)
     (in_bom yes) (on_board yes) (dnp no) (fields_autoplaced)
@@
       (effects (font (size 1.27 1.27)) (justify left))
     )
-    (property "Value" "Q_Dual_NMOS_S1G1D2S2G2D1" (at 246.38 134.62 0)
-      (effects (font (size 1.27 1.27)) (justify left))
-    )
+    (property "Value" "2N7002DW" (at 246.38 134.62 0)
+      (effects (font (size 1.27 1.27)) (justify left))
+    )
