File: hardware/repeater/CAN_XCVR.kicad_sch (KiCad schematic)
At the start: 11 parts, among them U6 TJA1051T-3

Commit message: completed repeater
Parts:
- added C8: 100n, Capacitor_SMD:C_0603_1608Metric, symbol Device:C
- added JP6, JP7: Jumper_2_Open, Jumper:SolderJumper-2_P1.3mm_Open_RoundedPad1.0x1.5mm, symbol Jumper:Jumper_2_Open
- C10: renamed from C15; now not fitted; now left out of the parts list
- C11: renamed from C14; value C -> 100nF 100V; LCSC (none) -> C28233
- C7: renamed from C2; now not fitted; now left out of the parts list
- C9: renamed from C26; LCSC (none) -> C14663
- D5: renamed from D6; value SM712_SOT23 -> NUP2105L; LCSC (none) -> C5180311
- L1: renamed from L4; now not fitted; now left out of the parts list
- R10: renamed from R15; value R -> 50; LCSC (none) -> C17720
- R11: renamed from R16; value R -> 50; LCSC (none) -> C17720
- R8: renamed from R14; value R -> 0; LCSC (none) -> C21189
- R9: renamed from R17; value R -> 0; LCSC (none) -> C21189
- U3: renamed from U6; LCSC (none) -> C51954344
Connections:
- net +5V: no longer U3.5 (VIO)
- net GND: now also C8.1
- net H: now also L1.1, R9.2
- net H_IN: now also JP7.2 (B); no longer R11.2
- net L: now also L1.4, R8.2
- net L_IN: now also JP6.1 (A); no longer R10.1
- new net: JP6.2 (B), R10.1
- new net: JP7.1 (A), R11.2
- new net VIO: C8.2, U3.5 (VIO)
Other:
- moved on the sheet: C11, R10, R11
