File: hardware/repeater/repeater.kicad_sch (KiCad schematic)
At the start: 20 parts, among them J1 Screw_Terminal_01x06, J2 Conn_01x08, J3 Screw_Terminal_01x06, U2 74LVC1G00, U3 74LVC2G74

Commit message: completed repeater
Parts:
- removed J1, J3: Screw_Terminal_01x06, Connector_Phoenix_MC:PhoenixContact_MCV_1,5_6-G-3.81_1x06_P3.81mm_Vertical, symbol Connector:Screw_Terminal_01x06
- removed J2: Conn_01x08, Connector_PinHeader_2.54mm:PinHeader_1x08_P2.54mm_Vertical, symbol Connector_Generic:Conn_01x08
- removed JP1: SolderJumper_2_Open, Jumper:SolderJumper-2_P1.3mm_Open_RoundedPad1.0x1.5mm, symbol Jumper:SolderJumper_2_Open
- added C4: 100n, Capacitor_SMD:C_0603_1608Metric, symbol Device:C
- added D4: LED_P, LED_SMD:LED_0603_1608Metric_Pad1.05x0.95mm_HandSolder, symbol Device:LED
- added H1, H2, H3, H4: MountingHole, MountingHole:ToolingHole_1.152mm, symbol Mechanical:MountingHole
- added J1: Screw_Terminal_01x02, Connector_Phoenix_MSTB:PhoenixContact_MSTBA_2,5_2-G_1x02_P5.00mm_Horizontal, symbol Connector:Screw_Terminal_01x02
- added J2, J3, J4, J5: Screw_Terminal_01x04, Connector_Phoenix_MC:PhoenixContact_MCV_1,5_4-G-3.81_1x04_P3.81mm_Vertical, symbol Connector:Screw_Terminal_01x04
- added J6: Conn_01x09, Connector_PinHeader_2.54mm:PinHeader_1x09_P2.54mm_Vertical, symbol Connector_Generic:Conn_01x09
- added J7: Conn_02x04_Odd_Even, Connector_PinHeader_2.54mm:PinHeader_2x04_P2.54mm_Vertical, symbol Connector_Generic:Conn_02x04_Odd_Even
- added JP1, JP2, JP3, JP4, JP5: Jumper_2_Open, Jumper:SolderJumper-2_P1.3mm_Open_RoundedPad1.0x1.5mm, symbol Jumper:Jumper_2_Open
- added R4: 0, Resistor_SMD:R_0603_1608Metric_Pad0.98x0.95mm_HandSolder, symbol Device:R
- added R7: 1k, Resistor_SMD:R_0603_1608Metric, symbol Device:R
- added TP1: TestPoint, TestPoint:TestPoint_Loop_D1.80mm_Drill1.0mm_Beaded, symbol Connector:TestPoint
- C1: value C -> 1nF 1kV; footprint Capacitor_SMD:C_0603_1608Metric_Pad1.08x0.95mm_HandSolder -> Capacitor_SMD:C_0805_2012Metric_Pad1.18x1.45mm_HandSolder; LCSC (none) -> C303890
- C2: renamed from C11; LCSC (none) -> C14663
- C3: footprint Capacitor_THT:CP_Radial_D5.0mm_P2.50mm -> Capacitor_THT:C_Disc_D3.0mm_W1.6mm_P2.50mm; now left out of the parts list
- C5: renamed from C12; value 5pF -> 10pF; LCSC (none) -> C1634
- C6: renamed from C13; value C -> C_CLK; footprint Capacitor_SMD:C_0603_1608Metric -> Capacitor_SMD:C_0603_1608Metric_Pad1.08x0.95mm_HandSolder; now not fitted; now left out of the parts list
- D1: value D_Zener -> SMAJ24A; LCSC (none) -> C19077541
- D2: renamed from D4; footprint LED_SMD:LED_0603_1608Metric -> LED_SMD:LED_0603_1608Metric_Pad1.05x0.95mm_HandSolder; now left out of the parts list
- D3: renamed from D5; footprint LED_SMD:LED_0603_1608Metric -> LED_SMD:LED_0603_1608Metric_Pad1.05x0.95mm_HandSolder; now left out of the parts list
- F1: LCSC (none) -> C41414042
- R1: renamed from R2; value R -> 10; LCSC (none) -> C22859
- R2: renamed from R3; value R -> 10; LCSC (none) -> C22859
- R3: renamed from R1; value R -> 1; LCSC (none) -> C25271
- R5: renamed from R4; value R -> 1k; LCSC (none) -> C21190
- R6: renamed from R5; value R -> 1k; LCSC (none) -> C21190
- U1: renamed from U2; LCSC (none) -> C2976658
- U2: renamed from U3; LCSC (none) -> C1850266
Connections:
- net +5VL is gone; now on net +5V: D2.2 (A), D3.2 (A)
- net +5V: now also C4.2, D4.2 (A), J6.3 (Pin_3), J7.2 (Pin_2), JP1.1 (A)
- net CLK: now also R4.2, TP1.1; no longer U1.4
- net GND: now also C4.1, J1.1 (Pin_1), J2.1 (Pin_1), J3.1 (Pin_1), J4.1 (Pin_1), J5.1 (Pin_1), J6.1 (Pin_1), J7.1 (Pin_1), R7.2
- net H_0: now also J2.3 (Pin_3), J4.3 (Pin_3)
- net H_1: now also J3.3 (Pin_3), J5.3 (Pin_3)
- net L_0: now also J2.2 (Pin_2), J4.2 (Pin_2)
- net L_1: now also J3.2 (Pin_2), J5.2 (Pin_2)
- net RX_0: now also R1.2, J6.4 (Pin_4), JP2.1 (A); no longer R1.1
- net RX_1: now also R2.2, J6.7 (Pin_7), JP3.1 (A); no longer R2.1
- net S_0: now also J6.6 (Pin_6), JP5.2 (B); no longer U2.3 (~{Q})
- net S_1: now also J6.9 (Pin_9), JP4.2 (B); no longer U2.5 (Q)
- net TX_0: now also J6.5 (Pin_5), JP3.2 (B); no longer R2.2
- net TX_1: now also J6.8 (Pin_8), JP2.2 (B); no longer R1.2
- net VBUS: now also J1.2 (Pin_2), J2.4 (Pin_4), J3.4 (Pin_4), J4.4 (Pin_4), J5.4 (Pin_4)
- new net: D4.1 (K), R7.1
- new net C: R4.1, U1.4
- new net Q: JP4.1 (A), U2.5 (Q)
- new net VIO: J6.2 (Pin_2), JP1.2 (B)
- new net XCVR0/RX_{CAN}: R1.1
- new net XCVR1/RX_{CAN}: R2.1
- new net ~{Q}: JP5.1 (A), U2.3 (~{Q})
Other:
- sheet XCVR renamed XCVR0
- sheet XCVR0 ports: added VIO; removed none
- sheet XCVR1 ports: added VIO; removed none
- note added: "fanout balancing"
- moved on the sheet: C2, R1, R2, U1
