File: hardware/repeater/vreg.kicad_sch (KiCad schematic)
At the start: 8 parts, among them U8 TD1465

Commit message: completed repeater
Parts:
- C17: renamed from C40; LCSC (none) -> C13585
- C18: renamed from C41; LCSC (none) -> C14663
- C19: renamed from C42; LCSC (none) -> C45783
- L3: renamed from L2; LCSC (none) -> C223225
- R16: renamed from R42; LCSC (none) -> C22935
- R17: renamed from R43; value 43k -> 39k; LCSC (none) -> C23153
- R18: renamed from R44; value 8k2 -> 7k5; LCSC (none) -> C23234
- U5: renamed from U8; LCSC (none) -> C2832208
Other:
- note added: "0.8V"
