File: hardware/knob/knob_top/LED.kicad_sch (KiCad schematic)
At the start: 36 parts

Commit message: various
Parts:
- D1: footprint project_lib:LED-APA102-2020 -> project_lib:LED-HD107S-2020_extPads
Changed lines of the file:
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@@
       (effects (font (size 1.27 1.27)) (justify left))
     )
-    (property "Footprint" "project_lib:LED-APA102-2020" (at 120.65 57.15 0)
+    (property "Footprint" "project_lib:LED-HD107S-2020_extPads" (at 120.65 57.15 0)
       (effects (font (size 1.27 1.27)) (justify left top) hide)
     )
@@
       (effects (font (size 1.27 1.27)) (justify left))
     )
-    (property "Footprint" "project_lib:LED-APA102-2020" (at 90.17 57.15 0)
+    (property "Footprint" "project_lib:LED-HD107S-2020_extPads" (at 90.17 57.15 0)
       (effects (font (size 1.27 1.27)) (justify left top) hide)
     )
@@
       (effects (font (size 1.27 1.27)) (justify left))
     )
-    (property "Footprint" "project_lib:LED-APA102-2020" (at 273.05 57.15 0)
+    (property "Footprint" "project_lib:LED-HD107S-2020_extPads" (at 273.05 57.15 0)
       (effects (font (size 1.27 1.27)) (justify left top) hide)
     )
@@
       (effects (font (size 1.27 1.27)) (justify left))
     )
-    (property "Footprint" "project_lib:LED-APA102-2020" (at 196.85 57.15 0)
+    (property "Footprint" "project_lib:LED-HD107S-2020_extPads" (at 196.85 57.15 0)
       (effects (font (size 1.27 1.27)) (justify left top) hide)
     )
@@
       (effects (font (size 1.27 1.27)) (justify left))
     )
-    (property "Footprint" "project_lib:LED-APA102-2020" (at 74.93 57.15 0)
+    (property "Footprint" "project_lib:LED-HD107S-2020_extPads" (at 74.93 57.15 0)
       (effects (font (size 1.27 1.27)) (justify left top) hide)
     )
@@
       (effects (font (size 1.27 1.27)) (justify left))
     )
-    (property "Footprint" "project_lib:LED-APA102-2020" (at 105.41 57.15 0)
+    (property "Footprint" "project_lib:LED-HD107S-2020_extPads" (at 105.41 57.15 0)
       (effects (font (size 1.27 1.27)) (justify left top) hide)
     )
@@
       (effects (font (size 1.27 1.27)) (justify left))
     )
-    (property "Footprint" "project_lib:LED-APA102-2020" (at 257.81 57.15 0)
+    (property "Footprint" "project_lib:LED-HD107S-2020_extPads" (at 257.81 57.15 0)
       (effects (font (size 1.27 1.27)) (justify left top) hide)
     )
@@
       (effects (font (size 1.27 1.27)) (justify left))
     )
-    (property "Footprint" "project_lib:LED-APA102-2020" (at 44.45 57.15 0)
+    (property "Footprint" "project_lib:LED-HD107S-2020_extPads" (at 44.45 57.15 0)
       (effects (font (size 1.27 1.27)) (justify left top) hide)
     )
@@
       (effects (font (size 1.27 1.27)) (justify left))
     )
-    (property "Footprint" "project_lib:LED-APA102-2020" (at 212.09 57.15 0)
+    (property "Footprint" "project_lib:LED-HD107S-2020_extPads" (at 212.09 57.15 0)
       (effects (font (size 1.27 1.27)) (justify left top) hide)
     )
@@
       (effects (font (size 1.27 1.27)) (justify left))
     )
-    (property "Footprint" "project_lib:LED-APA102-2020" (at 135.89 57.15 0)
+    (property "Footprint" "project_lib:LED-HD107S-2020_extPads" (at 135.89 57.15 0)
       (effects (font (size 1.27 1.27)) (justify left top) hide)
     )
@@
       (effects (font (size 1.27 1.27)) (justify left))
     )
-    (property "Footprint" "project_lib:LED-APA102-2020" (at 59.69 57.15 0)
+    (property "Footprint" "project_lib:LED-HD107S-2020_extPads" (at 59.69 57.15 0)
       (effects (font (size 1.27 1.27)) (justify left top) hide)
     )
@@
       (effects (font (size 1.27 1.27)) (justify left))
     )
-    (property "Footprint" "project_lib:LED-APA102-2020" (at 242.57 57.15 0)
+    (property "Footprint" "project_lib:LED-HD107S-2020_extPads" (at 242.57 57.15 0)
       (effects (font (size 1.27 1.27)) (justify left top) hide)
     )
@@
       (effects (font (size 1.27 1.27)) (justify left))
     )
-    (property "Footprint" "project_lib:LED-APA102-2020" (at 166.37 57.15 0)
+    (property "Footprint" "project_lib:LED-HD107S-2020_extPads" (at 166.37 57.15 0)
       (effects (font (size 1.27 1.27)) (justify left top) hide)
     )
@@
       (effects (font (size 1.27 1.27)) (justify left))
     )
-    (property "Footprint" "project_lib:LED-APA102-2020" (at 181.61 57.15 0)
+    (property "Footprint" "project_lib:LED-HD107S-2020_extPads" (at 181.61 57.15 0)
       (effects (font (size 1.27 1.27)) (justify left top) hide)
     )
@@
       (effects (font (size 1.27 1.27)) (justify left))
     )
-    (property "Footprint" "project_lib:LED-APA102-2020" (at 227.33 57.15 0)
+    (property "Footprint" "project_lib:LED-HD107S-2020_extPads" (at 227.33 57.15 0)
       (effects (font (size 1.27 1.27)) (justify left top) hide)
     )
@@
       (effects (font (size 1.27 1.27)) (justify left))
     )
-    (property "Footprint" "project_lib:LED-APA102-2020" (at 151.13 57.15 0)
+    (property "Footprint" "project_lib:LED-HD107S-2020_extPads" (at 151.13 57.15 0)
       (effects (font (size 1.27 1.27)) (justify left top) hide)
     )
@@
       (effects (font (size 1.27 1.27)) (justify left))
     )
-    (property "Footprint" "project_lib:LED-APA102-2020" (at 288.29 57.15 0)
+    (property "Footprint" "project_lib:LED-HD107S-2020_extPads" (at 288.29 57.15 0)
       (effects (font (size 1.27 1.27)) (justify left top) hide)
     )
@@
       (effects (font (size 1.27 1.27)) (justify left))
     )
-    (property "Footprint" "project_lib:LED-APA102-2020" (at 29.21 57.15 0)
-      (effects (font (size 1.27 1.27)) (justify left top) hide)
-    )
+    (property "Footprint" "project_lib:LED-HD107S-2020_extPads" (at 29.21 57.15 0)
+      (effects (font (size 1.27 1.27)) (justify left top) hide)
+    )
