File: hardware/knob/knob_top/knob_top.kicad_pcb (KiCad board)
At the start: 2 copper layers, 25 x 25 mm, 41 parts, among them J1 Conn_02x05_Odd_Even, SW1 SW_Push

Commit message: various
Parts:
- D1, D10, D11, D12, D13, D14, D15, D16, D17, D18, D2, D3, D4, D5, D6, D7, D8, D9: footprint project_lib:LED-APA102-2020 -> project_lib:LED-HD107S-2020_extPads
- moved C1 130.9 mm to (0.00, -7.75)
- moved C10 130.9 mm to (0.00, 7.75)
- moved C11 130.9 mm to (-2.65, 7.28)
- moved C12 130.9 mm to (-4.98, 5.94)
- moved C13 130.9 mm to (-6.71, 3.88)
- moved C14 130.9 mm to (-7.63, 1.35)
- moved C15 130.9 mm to (-7.63, -1.35)
- moved C16 130.9 mm to (-6.71, -3.88)
- moved C17 130.9 mm to (-4.98, -5.94)
- moved C18 130.9 mm to (-2.65, -7.28)
- moved C19 130.9 mm to (-2.00, 4.50)
- moved C2 130.9 mm to (2.65, -7.28)
- moved C3 130.9 mm to (4.98, -5.94)
- moved C4 130.9 mm to (6.71, -3.88)
- moved C5 130.9 mm to (7.63, -1.35)
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Routing:
- net +5V: track 110.7 -> 95.0 mm
- net Net-(D15-SDO): track 3.09 -> 0.00 mm
- net Net-(D6-SDO): track 3.09 -> 0.00 mm
- net Net-(D14-SDO): track 3.09 -> 0.00 mm
- net Net-(D7-SDO): track 3.09 -> 0.00 mm
- net Net-(D16-SDO): track 3.09 -> 0.00 mm
- net Net-(D13-SDO): track 3.09 -> 0.00 mm
- net Net-(D4-SDO): track 3.09 -> 0.00 mm
- net Net-(D17-SDO): track 3.09 -> 0.00 mm
- net Net-(D11-SDO): track 3.09 -> 0.00 mm
- net Net-(D2-SDO): track 3.09 -> 0.00 mm
- net Net-(D10-SDI): track 3.09 -> 0.00 mm
- net Net-(D12-SDO): track 3.09 -> 0.00 mm
- net Net-(D3-SDO): track 3.09 -> 0.00 mm
- net Net-(D8-SDO): track 3.09 -> 0.00 mm
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