File: hardware/generic_node/MCU.kicad_sch (KiCad schematic)
At the start: 17 parts, among them J10 AVR-ISP-6, SW4 SW_Push, U3 ATmega328PB-A, Y1 Crystal_GND24

Commit message: hw layout
Parts:
- removed D1: LED, LED_SMD:LED_0603_1608Metric, symbol Device:LED
- removed R7: R, Resistor_SMD:R_0603_1608Metric, symbol Device:R
- removed U3: ATmega328PB-A, Package_QFP:TQFP-32_7x7mm_P0.8mm, symbol MCU_Microchip_ATmega:ATmega328PB-A
- added U2: ATmega328PB-M, Package_DFN_QFN:QFN-32-1EP_5x5mm_P0.5mm_EP3.1x3.1mm, symbol MCU_Microchip_ATmega:ATmega328PB-M
- C1, C2, C3, C4, C5, C6, C7: footprint Capacitor_SMD:C_0603_1608Metric -> Capacitor_SMD:C_0402_1005Metric
- D2: footprint LED_SMD:LED_0603_1608Metric -> LED_SMD:LED_0402_1005Metric
- FB1: footprint Inductor_SMD:L_0603_1608Metric -> Inductor_SMD:L_0402_1005Metric
- R13, R8: footprint Resistor_SMD:R_0603_1608Metric -> Resistor_SMD:R_0402_1005Metric
- Y1: footprint Crystal:Crystal_SMD_3225-4Pin_3.2x2.5mm -> Crystal:Crystal_SMD_2520-4Pin_2.5x2.0mm
Connections:
- net +5V: now also U2.4 (VCC)
- net +5VA: now also U2.18 (AVCC)
- net CD: now also U2.32 (PD2)
- net GND: now also U2.21 (GND), U2.33 (GND), U2.5 (GND)
- net RXD: now also U2.30 (PD0)
- net TXD: now also U2.31 (PD1)
- net XTAL1: now also U2.7 (XTAL1/PB6)
- net XTAL2: now also U2.8 (XTAL2/PB7)
- net AREF renamed REF
- net REF: now also U2.20 (AREF)
- net ISP_SCK renamed D13
- net D13: now also U2.17 (PB5)
- net RXD1 renamed D12
- net D12: now also U2.16 (PB4)
- net TXD1 renamed D11
- net D11: now also U2.15 (PB3)
- net ~{ISP_RST} renamed ~{RST}
- net ~{RST}: now also U2.29 (~{RESET}/PC6)
- new net A0: U2.23 (PC0)
- new net A1: U2.24 (PC1)
- new net A2: U2.25 (PC2)
- new net A3: U2.26 (PC3)
- new net A4: U2.27 (PC4)
- new net A5: U2.28 (PC5)
- new net A6: U2.19 (PE2)
- new net A7: U2.22 (PE3)
- new net D10: U2.14 (PB2)
- new net D23: U2.3 (PE0)
- new net D24: U2.6 (PE1)
- new net D3: U2.1 (PD3)
- new net D4: U2.2 (PD4)
- new net D5: U2.9 (PD5)
- new net D6: U2.10 (PD6)
- new net D7: U2.11 (PD7)
- new net D8: U2.12 (PB0)
- new net D9: U2.13 (PB1)

Commit message: working
Parts:
- J10: footprint project_lib:Tag-Connect_TC2030-IDC-NL_2x03_P1.27mm_Vertical -> Connector_PinHeader_2.54mm:PinHeader_2x03_P2.54mm_Vertical
