File: hardware/generic_node/generic_node.kicad_pcb (KiCad board)
At the start: 2 copper layers, 17.8 x 48.7 mm, 49 parts, among them J1 Conn_01x15, J10 AVR-ISP-6, J11 Screw_Terminal_01x04, J2 Conn_01x15, SW4 SW_Push, U3 ATmega328PB-A, U4 74LVC1G57, U5 TD1465, U6 TJA1051T-3, Y1 Crystal_GND24

Commit message: hw layout
Parts:
- removed D1: LED, LED_SMD:LED_0603_1608Metric
- removed R7: R, Resistor_SMD:R_0603_1608Metric
- removed U3: ATmega328PB-A, Package_QFP:TQFP-32_7x7mm_P0.8mm
- removed U6: TJA1051T-3, Package_SO:SOIC-8_3.9x4.9mm_P1.27mm
- added U1: TJA1051TK-3, Package_DFN_QFN:DFN-8-1EP_3x3mm_P0.65mm_EP1.55x2.4mm, F.Cu at (212.8, 94.0)
- added U2: ATmega328PB-M, Package_DFN_QFN:QFN-32-1EP_5x5mm_P0.5mm_EP3.1x3.1mm, F.Cu at (191.8, 97.0)
- C1, C15, C17, C18, C19, C2, C3, C4, C5, C6, C7: footprint Capacitor_SMD:C_0603_1608Metric -> Capacitor_SMD:C_0402_1005Metric
- C11: footprint Capacitor_THT:CP_Radial_D6.3mm_P2.50mm -> Capacitor_THT:C_Disc_D3.0mm_W1.6mm_P2.50mm
- D2: footprint LED_SMD:LED_0603_1608Metric -> LED_SMD:LED_0402_1005Metric
- FB1: footprint Inductor_SMD:L_0603_1608Metric -> Inductor_SMD:L_0402_1005Metric
- R13, R19, R20, R21, R22, R8: footprint Resistor_SMD:R_0603_1608Metric -> Resistor_SMD:R_0402_1005Metric
- Y1: footprint Crystal:Crystal_SMD_3225-4Pin_3.2x2.5mm -> Crystal:Crystal_SMD_2520-4Pin_2.5x2.0mm
- moved C10 59.8 mm to (213.8, 99.2), turned to -90 degrees
- moved F1 58.1 mm to (212.0, 99.5), turned to -90 degrees
- moved R14 56.5 mm to (212.8, 102.5), turned to 180 degrees
- moved D2 44.5 mm to (185.2, 100.2)
- moved J10 43.5 mm to (182.2, 94.2), turned to -90 degrees
- moved R8 41.7 mm to (185.2, 101.2), turned to 0 degrees
- moved SW4 41.1 mm to (182.3, 100.2), turned to -90 degrees
- moved R13 35.7 mm to (185.2, 99.2), turned to 180 degrees
- moved C1 35.4 mm to (187.2, 96.8), turned to 180 degrees
- moved C5 34.6 mm to (187.2, 95.8), turned to 180 degrees
- moved FB1 34.0 mm to (187.2, 94.8), turned to 0 degrees
- moved C4 33.5 mm to (187.2, 93.7), turned to 0 degrees
- moved R16 25.5 mm to (227.5, 99.0), turned to 0 degrees
- moved C13 24.4 mm to (227.5, 97.0), turned to 180 degrees
- moved J11 24.3 mm to (223.8, 102.7), turned to 90 degrees
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Connections:
- C1 pad 1: /MCU/AREF -> /REF
- D5 pad 1: /MCU/TXD -> /D1
- J1 pad 1: unconnected-(J1-Pin_1-Pad1) -> /D1
- J1 pad 2: unconnected-(J1-Pin_2-Pad2) -> /D0
- J1 pad 3: unconnected-(J1-Pin_3-Pad3) -> /D24
- J10 pad 1: /RX1 -> /D12
- J10 pad 3: /MCU/ISP_SCK -> /D13
- J10 pad 4: /TX1 -> /D11
- J10 pad 5: /MCU/~{ISP_RST} -> /~{RST}
- J2 pad 14: unconnected-(J2-Pin_14-Pad14) -> /~{RST}
- J2 pad 3: unconnected-(J2-Pin_3-Pad3) -> /D23
- R13 pad 2: /MCU/~{ISP_RST} -> /~{RST}
- R19 pad 2: /MCU/TXD -> /D1
- R8 pad 2: /MCU/ISP_SCK -> /D13
- SW4 pad 1: /MCU/~{ISP_RST} -> /~{RST}
- U4 pad 1: /MCU/RXD -> /D0
- U4 pad 4: /MCU/CD -> /D2
Routing:
- net /D1: track 0.00 -> 40.8 mm, vias 0 -> 2
- net /D2: track 0.00 -> 39.9 mm, vias 0 -> 1
- net /D0: track 0.00 -> 39.8 mm, vias 0 -> 2
- net VBUS: track 2.63 -> 34.9 mm
- net /D13: track 0.00 -> 30.8 mm
- net /A7: track 0.00 -> 26.2 mm, vias 0 -> 2
- net /A6: track 0.00 -> 25.6 mm, vias 0 -> 2
- net /D23: track 0.00 -> 24.4 mm, vias 0 -> 2
- net GND: track 0.00 -> 24.4 mm, vias 0 -> 98
- net /D24: track 0.00 -> 23.3 mm, vias 0 -> 2
- net /D3: track 0.00 -> 21.7 mm
- net /~{RST}: track 0.00 -> 20.0 mm, vias 0 -> 2
- net /D4: track 0.00 -> 19.1 mm
- net /A5: track 0.00 -> 16.7 mm
- net +5V: track 5.11 -> 21.2 mm, vias 0 -> 6
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- added copper zone on In2.Cu, net +5V
- added copper zone on In1.Cu, net GND
Other:
- board size 17.8 x 48.7 mm -> 48.9 x 17.8 mm
- copper layers 2 -> 4
- board text added: "5V"
- board text added: "A0"
- board text added: "A1"
- board text added: "A2"
- board text added: "A3"
- board text added: "A4"
- board text added: "A5"
- board text added: "A6"
- board text added: "A7"
- board text added: "AREF"
- board text added: "D0"
- board text added: "D1"
- board text added: "D10"
- board text added: "D11"
- board text added: "D12"
- board text added: "D13"
- board text added: "D2"
- board text added: "D23"
- board text added: "D24"
- board text added: "D3"
- board text added: "D4"
- board text added: "D5"
- board text added: "D6"
- board text added: "D7"
- board text added: "D8"
- board text added: "D9"
- board text added: "GND"
- board text added: "H"
- board text added: "L"
- board text added: "Vin"
- board text added: "~{RST}"

Commit message: working
Parts:
- J10: footprint project_lib:Tag-Connect_TC2030-IDC-NL_2x03_P1.27mm_Vertical -> Connector_PinHeader_2.54mm:PinHeader_2x03_P2.54mm_Vertical
- moved J10 7.28 mm to (175.0, 94.0), turned to 0 degrees
Routing:
- net +24V: track 12.5 -> 11.6 mm
