File: hardware/generic_node/generic_node.kicad_sch (KiCad schematic)
At the start: 2 parts, among them J1 Conn_01x15, J2 Conn_01x15

Commit message: hw layout
Connections:
- net D0: now also J1.2 (Pin_2)
- net D1: now also J1.1 (Pin_1)
- net D24: now reaches J1.3 (Pin_3)
- net ~{RST}: now reaches J2.14 (Pin_14)
- net D23: now reaches J2.3 (Pin_3)
Other:
- sheet MCU ports: added REF, {A[0..7]}, {D[0..24]}, ~{RST}; removed ALS, ENC_A, ENC_B, ENC_P0, ENC_P1, MISO1, MOSI1, RXD1, SCK1, SCL, SDA, SS1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
