File: hardware/generic_node/input.kicad_sch (KiCad schematic)
At the start: 30 parts, among them J11 Screw_Terminal_01x04, U4 74LVC1G57, U5 TD1465, U6 TJA1051T-3

Commit message: hw layout
Parts:
- removed U6: TJA1051T-3, Package_SO:SOIC-8_3.9x4.9mm_P1.27mm, symbol Interface_CAN_LIN:TJA1051T-3
- added U1: TJA1051TK-3, Package_DFN_QFN:DFN-8-1EP_3x3mm_P0.65mm_EP1.55x2.4mm, symbol Interface_CAN_LIN:TJA1051TK-3
- C11: footprint Capacitor_THT:CP_Radial_D6.3mm_P2.50mm -> Capacitor_THT:C_Disc_D3.0mm_W1.6mm_P2.50mm
- C15, C17, C18, C19: footprint Capacitor_SMD:C_0603_1608Metric -> Capacitor_SMD:C_0402_1005Metric
- R19, R20, R21, R22: footprint Resistor_SMD:R_0603_1608Metric -> Resistor_SMD:R_0402_1005Metric
Connections:
- net +5V: now also U1.3 (VCC), U1.5 (VIO)
- net CAN_N: now also U1.6 (CANL)
- net CAN_P: now also U1.7 (CANH)
- net GND: now also U1.2 (GND), U1.8 (S), U1.9 (GND)
- net RX: now also U1.4 (RXD)
- net TX: now also U1.1 (TXD)
