File: hardware/knob/knob_base/MCU.kicad_sch (KiCad schematic)
At the start: 33 parts, among them J10 AVR-ISP-6, SW2 SW_Push, SW3 SW_Push, SW4 SW_Push, U3 ATmega328PB-A, Y1 Crystal_GND24

Commit message: working
Parts:
- J10: now left out of the parts list
