File: hardware/knob/knob_base/input.kicad_sch (KiCad schematic)
At the start: 30 parts, among them J11 Screw_Terminal_01x04, U4 74LVC1G57, U5 TD1465, U6 TJA1051T-3

Commit message: working
Parts:
- C11, C13, J11, R16, R17: now left out of the parts list
- U4: footprint Package_TO_SOT_SMD:SOT-563 -> Package_TO_SOT_SMD:SOT-363_SC-70-6
