File: hardware/knob/knob_base/knob_base.kicad_pcb (KiCad board)
At the start: 2 copper layers, 44 x 40.5 mm, 76 parts, among them J1 Conn_01x05, J10 AVR-ISP-6, J11 Screw_Terminal_01x04, J3 Conn_02x05_Odd_Even, J4 Conn_01x04, J5 Conn_01x04, J6 Conn_01x04, SW1 RotaryEncoder, SW2 SW_Push, SW3 SW_Push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

Commit message: working
Parts:
- removed C23: C, Capacitor_SMD:C_0603_1608Metric
- removed D6: D_Photo, LED_THT:LED_D3.0mm_Clear
- removed R1: R, Resistor_SMD:R_0603_1608Metric
- removed U1: LMV321, Package_TO_SOT_SMD:SOT-23-5
- added Q1: ALS-PDIC144-6C/L378, LED_THT:LED_D3.0mm_FlatTop, B.Cu at (134.4, 118.6)
- U4: footprint Package_TO_SOT_SMD:SOT-563 -> Package_TO_SOT_SMD:SOT-363_SC-70-6
- moved C25 4.87 mm to (137.0, 119.8), turned to 90 degrees
- moved R2 4.87 mm to (138.5, 119.8)
- moved C24 2.39 mm to (140.0, 119.8), turned to 90 degrees
- moved C15 0.40 mm to (133.8, 87.9)
- moved R19 0.40 mm to (133.8, 89.4)
- moved D5 0.35 mm to (133.8, 90.8)
- moved C18 0.25 mm to (136.2, 85.8)
- moved U4 0.25 mm to (133.8, 85.8)
Connections:
- R2 pad 1: /light sensor/PTout -> GND
Routing:
- net /light sensor/PTout: track 9.04 -> 0.00 mm
- net /LS: track 19.6 -> 27.1 mm
- net /light sensor/PT-: track 5.93 -> 0.00 mm
- net +5VA: track 25.0 -> 30.6 mm
- net +5V: track 162.8 -> 167.6 mm
- net GND: track 11.5 -> 12.3 mm, vias 83 -> 185
Other:
- board text added: "+5V"
- board text added: "+5V SCL SDA GND"
- board text added: "+5V TXD RXD GND"
- board text added: "GND"
- board text added: "GND 0 1 +5V"
- board text added: "GND CANL CANH VBUS"
- board text added: "MISO"
- board text added: "MOSI"
- board text added: "P0"
- board text added: "P1"
- board text added: "SCK"
- board text added: "SCL"
- board text added: "SDA"
- board text added: "SS"
- board text added: "VBUS 3 2 GND"
