File: hardware/knob/knob_base/knob_base.kicad_sch (KiCad schematic)
At the start: 6 parts, among them J1 Conn_01x05, J3 Conn_02x05_Odd_Even, J4 Conn_01x04, J5 Conn_01x04, J6 Conn_01x04, SW1 RotaryEncoder

Commit message: working
Parts:
- J1, J3, J4, J5, J6, SW1: now left out of the parts list
Other:
- removed sheet LED_out
