File: hardware/led_balance/led_balance.kicad_sch (KiCad schematic)
At the start: 30 parts, among them J1 Screw_Terminal_01x04, J2 Screw_Terminal_01x02, J3 Screw_Terminal_01x04, J4 Screw_Terminal_01x04, J5 Screw_Terminal_01x04, J6 Screw_Terminal_01x02, J7 Screw_Terminal_01x02, J8 Screw_Terminal_01x02

Commit message: led balance and corridor ready
Parts:
- TH1, TH2, TH3, TH4: footprint TestPoint:TestPoint_2Pads_Pitch2.54mm_Drill0.8mm -> Package_TO_SOT_THT:TO-220-2_Horizontal_TabUp
Changed lines of the file:
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@@
       (effects (font (size 1.27 1.27)))
     )
-    (property "Footprint" "TestPoint:TestPoint_2Pads_Pitch2.54mm_Drill0.8mm" (at 22.86 119.38 0)
+    (property "Footprint" "Package_TO_SOT_THT:TO-220-2_Horizontal_TabUp" (at 22.86 119.38 0)
       (effects (font (size 1.27 1.27)) hide)
     )
@@
       (effects (font (size 1.27 1.27)))
     )
-    (property "Footprint" "TestPoint:TestPoint_2Pads_Pitch2.54mm_Drill0.8mm" (at 22.86 106.68 0)
+    (property "Footprint" "Package_TO_SOT_THT:TO-220-2_Horizontal_TabUp" (at 22.86 106.68 0)
       (effects (font (size 1.27 1.27)) hide)
     )
@@
       (effects (font (size 1.27 1.27)))
     )
-    (property "Footprint" "TestPoint:TestPoint_2Pads_Pitch2.54mm_Drill0.8mm" (at 21.59 54.61 0)
+    (property "Footprint" "Package_TO_SOT_THT:TO-220-2_Horizontal_TabUp" (at 21.59 54.61 0)
       (effects (font (size 1.27 1.27)) hide)
     )
@@
       (effects (font (size 1.27 1.27)))
     )
-    (property "Footprint" "TestPoint:TestPoint_2Pads_Pitch2.54mm_Drill0.8mm" (at 21.59 67.31 0)
+    (property "Footprint" "Package_TO_SOT_THT:TO-220-2_Horizontal_TabUp" (at 21.59 67.31 0)
       (effects (font (size 1.27 1.27)) hide)
     )
