File: hardware/led_balance/mirror_unit.kicad_sch (KiCad schematic)
At the start: 11 parts, among them Q1 Q_NMOS_GDS, Q17 Q_NPN_BEC, Q18 Q_PNP_BEC

Commit message: led balance and corridor ready
Parts:
- added D20: 1N5333B, Diode_THT:D_DO-27_P12.70mm_Horizontal, symbol Diode:1N53xxB
Connections:
- net SINK: now also D20.1 (K); no longer D1.1 (K), Q1.2 (D), R1.1
- new net: D1.1 (K), D20.2 (A), Q1.2 (D), R1.1
Changed lines of the file:
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@@
+    (stroke (width 0) (type default))
+  )
+  (wire (pts (xy 142.24 95.25) (xy 142.24 97.79))
     (stroke (width 0) (type default))
   )
@@
     (stroke (width 0) (type default))
   )
+  (wire (pts (xy 142.24 82.55) (xy 142.24 87.63))
+    (stroke (width 0) (type default))
+  )
   (wire (pts (xy 142.24 134.62) (xy 142.24 137.16))
     (stroke (width 0) (type default))
@@
   )
   (wire (pts (xy 119.38 124.46) (xy 119.38 127))
-    (stroke (width 0) (type default))
-  )
-  (wire (pts (xy 142.24 82.55) (xy 142.24 97.79))
     (stroke (width 0) (type default))
   )
@@
         )
       )
+    )
+  )
+  (symbol (lib_id "Diode:1N53xxB") (at 142.24 91.44 270) (unit 1)
+    (in_bom yes) (on_board yes) (dnp no) (fields_autoplaced)
+    (property "Reference" "D20" (at 144.78 90.17 90)
+      (effects (font (size 1.27 1.27)) (justify left))
+    )
+    (property "Value" "1N5333B" (at 144.78 92.71 90)
+      (effects (font (size 1.27 1.27)) (justify left))
+    )
+    (property "Footprint" "Diode_THT:D_DO-27_P12.70mm_Horizontal" (at 137.795 91.44 0)
+      (effects (font (size 1.27 1.27)) hide)
+    )
+    (property "Datasheet" "https://diotec.com/tl_files/diotec/files/pdf/datasheets/1n5345b.pdf" (at 142.24 91.44 0)
+      (effects (font (size 1.27 1.27)) hide)
+    )
+    (pin "1")
+    (pin "2")
+    (instances
+      (project "led_balance"
+        (path "/f283858f-5dca-4ed2-8697-33202af53f49/b83b4677-bf25-48e0-9434-d0dad3c291f7"
+          (reference "D20") (unit 1)
+        )
+        (path "/f283858f-5dca-4ed2-8697-33202af53f49/9a41cbb6-3e7d-4a02-b827-429543edfb52"
+          (reference "D21") (unit 1)
+        )
+        (path "/f283858f-5dca-4ed2-8697-33202af53f49/a32f99c4-e2a2-491b-aacc-d753c29a5e22"
+          (reference "D23") (unit 1)
+        )
+        (path "/f283858f-5dca-4ed2-8697-33202af53f49/d8e3ac6b-a41e-4658-8daa-61761a230bac"
+          (reference "D24") (unit 1)
+        )
+        (path "/f283858f-5dca-4ed2-8697-33202af53f49/40e7225f-e3db-4b1b-902f-0b3839ba321d"
+          (reference "D25") (unit 1)
+        )
+        (path "/f283858f-5dca-4ed2-8697-33202af53f49/dc898c80-ffd1-4edd-b90e-bb15c2cb461e"
+          (reference "D26") (unit 1)
+        )
+        (path "/f283858f-5dca-4ed2-8697-33202af53f49/3044f107-1044-4a5d-ae3e-419c69b1b824"
+          (reference "D27") (unit 1)
+        )
+        (path "/f283858f-5dca-4ed2-8697-33202af53f49/fb5e80ca-f886-458f-9950-758bf69fafd9"
+          (reference "D28") (unit 1)
+        )
+      )

Commit message: various
Parts:
- Q17: value Q_NPN_BEC -> MMBT3904
- Q18: value Q_PNP_BEC -> MMBT3906
- R1: value R -> 10k
- R2: value R -> 2.2
- R3, R6: value R -> 1k
Changed lines of the file:
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@@
   (symbol (lib_id "Device:R") (at 119.38 120.65 0) (unit 1)
     (in_bom yes) (on_board yes) (dnp no) (fields_autoplaced)
-    (property "Reference" "R3" (at 121.158 119.8153 0)
-      (effects (font (size 1.27 1.27)) (justify left))
-    )
-    (property "Value" "R" (at 121.158 122.3522 0)
+    (property "Reference" "R3" (at 121.92 119.38 0)
+      (effects (font (size 1.27 1.27)) (justify left))
+    )
+    (property "Value" "1k" (at 121.92 121.92 0)
       (effects (font (size 1.27 1.27)) (justify left))
     )
@@
   (symbol (lib_id "Device:Q_NPN_BEC") (at 121.92 134.62 0) (mirror y) (unit 1)
     (in_bom yes) (on_board yes) (dnp no) (fields_autoplaced)
-    (property "Reference" "Q17" (at 117.0687 133.7853 0)
-      (effects (font (size 1.27 1.27)) (justify left))
-    )
-    (property "Value" "Q_NPN_BEC" (at 117.0687 136.3222 0)
+    (property "Reference" "Q17" (at 116.84 133.35 0)
+      (effects (font (size 1.27 1.27)) (justify left))
+    )
+    (property "Value" "MMBT3904" (at 116.84 135.89 0)
       (effects (font (size 1.27 1.27)) (justify left))
     )
@@
   )
   (symbol (lib_id "Device:R") (at 135.89 106.68 270) (unit 1)
-    (in_bom yes) (on_board yes) (dnp no) (fields_autoplaced)
-    (property "Reference" "R1" (at 135.89 101.9642 90)
-      (effects (font (size 1.27 1.27)))
-    )
-    (property "Value" "R" (at 135.89 104.5011 90)
+    (in_bom yes) (on_board yes) (dnp no)
+    (property "Reference" "R1" (at 135.89 104.14 90)
+      (effects (font (size 1.27 1.27)))
+    )
+    (property "Value" "10k" (at 135.89 106.68 90)
       (effects (font (size 1.27 1.27)))
     )
@@
   (symbol (lib_id "Device:R") (at 142.24 140.97 0) (unit 1)
     (in_bom yes) (on_board yes) (dnp no) (fields_autoplaced)
-    (property "Reference" "R2" (at 144.018 140.1353 0)
-      (effects (font (size 1.27 1.27)) (justify left))
-    )
-    (property "Value" "R" (at 144.018 142.6722 0)
+    (property "Reference" "R2" (at 144.78 139.7 0)
+      (effects (font (size 1.27 1.27)) (justify left))
+    )
+    (property "Value" "2.2" (at 144.78 142.24 0)
       (effects (font (size 1.27 1.27)) (justify left))
     )
@@
   )
   (symbol (lib_id "Device:R") (at 135.89 134.62 270) (unit 1)
-    (in_bom yes) (on_board yes) (dnp no) (fields_autoplaced)
-    (property "Reference" "R6" (at 135.89 129.9042 90)
-      (effects (font (size 1.27 1.27)))
-    )
-    (property "Value" "R" (at 135.89 132.4411 90)
+    (in_bom yes) (on_board yes) (dnp no)
+    (property "Reference" "R6" (at 135.89 132.08 90)
+      (effects (font (size 1.27 1.27)))
+    )
+    (property "Value" "1k" (at 135.89 134.62 90)
       (effects (font (size 1.27 1.27)))
     )
@@
   (symbol (lib_id "Device:Q_PNP_BEC") (at 127 127 0) (mirror x) (unit 1)
     (in_bom yes) (on_board yes) (dnp no) (fields_autoplaced)
-    (property "Reference" "Q18" (at 131.8514 126.1653 0)
-      (effects (font (size 1.27 1.27)) (justify left))
-    )
-    (property "Value" "Q_PNP_BEC" (at 131.8514 128.7022 0)
-      (effects (font (size 1.27 1.27)) (justify left))
-    )
+    (property "Reference" "Q18" (at 132.08 125.73 0)
+      (effects (font (size 1.27 1.27)) (justify left))
+    )
+    (property "Value" "MMBT3906" (at 132.08 128.27 0)
+      (effects (font (size 1.27 1.27)) (justify left))
+    )
