File: hardware/room_hub/MCU.kicad_sch (KiCad schematic)
At the start: 33 parts, among them J10 AVR-ISP-6, SW2 SW_Push, SW3 SW_Push, SW4 SW_Push, U3 ATmega328PB-A, Y1 Crystal_GND24

Commit message: hw layout
Parts:
- removed C21, C22: C, Capacitor_SMD:C_0603_1608Metric, symbol Device:C
- removed R23, R24, R25, R26: R, Resistor_SMD:R_0603_1608Metric, symbol Device:R
- J10: footprint project_lib:Tag-Connect_TC2030-IDC-NL_2x03_P1.27mm_Vertical -> Connector_PinHeader_2.54mm:PinHeader_2x03_P2.54mm_Vertical
Connections:
- net ALS: no longer names the net of U3.27 (PC4)
- net ENC_P0 renamed INT1
- net ENC_P1: no longer names the net of U3.28 (PC5)
- net OUT0 renamed DIM0
- net OUT1 renamed DIM1
- net OUT2 renamed DIM2
- net OUT3 renamed DIM3
- net SS1: no longer names the net of U3.19 (PE2)
- net _ENC_A: no longer names the net of U3.26 (PC3)
- net _ENC_B: no longer names the net of U3.25 (PC2)

Commit message: working
Connections:
- net MISO1 is gone; now on net A_EN: U3.23 (PC0)
- net SCK1 is gone; now on net B_EN: U3.24 (PC1)
- net A_FB: now also U3.27 (PC4)
- net B_FB: now also U3.28 (PC5)
- net CLS: now also U3.26 (PC3)
- net OPN: now also U3.25 (PC2)
- net ALS: now reaches U3.19 (PE2)
- net MOSI1: no longer names the net of U3.22 (PE3)
