File: hardware/room_hub/damp.kicad_sch (KiCad schematic)
At the start: 23 parts, among them J11 Screw_Terminal_01x04, Q2 2N7002K, Q3 2N7002K, Q4 BSS83P, Q5 BSS83P, Q6 2N7002DW, U8 LM393A

Commit message: working
Parts:
- J2: renamed from J11; footprint Connector_Phoenix_MC:PhoenixContact_MCV_1,5_4-G-3.5_1x04_P3.50mm_Vertical -> Connector_Phoenix_MC:PhoenixContact_MC_1,5_4-G-3.5_1x04_P3.50mm_Horizontal
- renumbered C9 to C23, C9 to C24, C9 to C25, C9 to C37, R18 to R1, R18 to R2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
