File: hardware/room_hub/input.kicad_sch (KiCad schematic)
At the start: 30 parts, among them J11 Screw_Terminal_01x04, U4 74LVC1G57, U5 TD1465, U6 TJA1051T-3

Commit message: hw layout
Parts:
- U4: footprint Package_TO_SOT_SMD:SOT-563 -> Package_TO_SOT_SMD:SOT-363_SC-70-6
Connections:
- net +24V: now also F1.2, R14.1; no longer C11.1, C16.2, R14.2, R20.2, U5.5 (VIN)
- net +5V: now also C11.1, C16.2, R14.2, R20.2, U5.5 (VIN)

Commit message: working
Parts:
- removed J11: Screw_Terminal_01x04, Connector_Phoenix_MC:PhoenixContact_MCV_1,5_4-G-3.81_1x04_P3.81mm_Vertical, symbol Connector:Screw_Terminal_01x04
- added J1, J3: Screw_Terminal_01x02, Connector_Phoenix_MC:PhoenixContact_MC_1,5_2-G-3.81_1x02_P3.81mm_Horizontal, symbol Connector:Screw_Terminal_01x02
- added J6: Screw_Terminal_01x02, Connector_Phoenix_MSTB:PhoenixContact_MSTBA_2,5_2-G_1x02_P5.00mm_Horizontal, symbol Connector:Screw_Terminal_01x02
Connections:
- net +5V: no longer C11.1, C16.2, R14.2, R20.2, U5.5 (VIN)
- net CAN+: now also J3.2 (Pin_2)
- net CAN-: now also J3.1 (Pin_1)
- net GND: now also J1.1 (Pin_1), J6.1 (Pin_1)
- net VBUS: now also J1.2 (Pin_2), J6.2 (Pin_2)
- new net VCCQ: C11.1, C16.2, R14.2, R20.2, U5.5 (VIN)
