File: hardware/room_hub/out.kicad_sch (KiCad schematic)
At the start: 28 parts, among them J3 Screw_Terminal_01x05, U1 UCC27517, U3 UCC27517, U4 UCC27517, U5 UCC27517, U6 L78L12_SOT89

Commit message: working
Parts:
- J4: renamed from J3; footprint Connector_Phoenix_MC:PhoenixContact_MCV_1,5_5-G-3.81_1x05_P3.81mm_Vertical -> Connector_Phoenix_MC:PhoenixContact_MC_1,5_5-G-3.81_1x05_P3.81mm_Horizontal
- renumbered C1 to C21, C1 to C22, C2 to C28, C4 to C29, C5 to C30, C6 to C31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
