File: hardware/room_hub/radar.kicad_sch (KiCad schematic)
At the start: 7 parts, among them M1 HLK-LD2410C, Q1 BSS138, U2 TXB0102DCT, U7 APE8865N-33-HF-3

Commit message: working
Parts:
- renumbered C18 to C26, C18 to C27, R18 to R3
