File: hardware/room_hub/room_hub.kicad_pcb (KiCad board)
At the start: 2 copper layers, 44 x 40.5 mm, 76 parts, among them J1 Conn_01x05, J10 AVR-ISP-6, J11 Screw_Terminal_01x04, J3 Conn_02x05_Odd_Even, J4 Conn_01x04, J5 Conn_01x04, J6 Conn_01x04, SW1 RotaryEncoder, SW2 SW_Push, SW3 SW_Push, SW4 SW_Push, U1 LMV321, U3 ATmega328PB-A, U4 74LVC1G57, U5 TD1465, U6 TJA1051T-3, Y1 Crystal_GND24

Commit message: hw layout
Parts:
- removed D6: D_Photo, LED_THT:LED_D3.0mm_Clear
- removed J1: Conn_01x05, Connector_PinSocket_2.54mm:PinSocket_1x05_P2.54mm_Vertical
- removed J3: Conn_02x05_Odd_Even, Connector_PinSocket_2.54mm:PinSocket_2x05_P2.54mm_Vertical_SMD
- removed J6: Conn_01x04, Connector_JST:JST_PH_B4B-PH-K_1x04_P2.00mm_Vertical
- removed SW1: RotaryEncoder, project_lib:EC35A0930401
- removed U1: LMV321, Package_TO_SOT_SMD:SOT-23-5
- added C26: 100n, Capacitor_SMD:C_0603_1608Metric, F.Cu at (198.5, 147.2)
- added C27: 100n, Capacitor_SMD:C_0603_1608Metric, F.Cu at (193.0, 147.2)
- added C28: C, Capacitor_SMD:C_0805_2012Metric, F.Cu at (173.7, 31.6)
- added C29: C, Capacitor_SMD:C_0603_1608Metric, F.Cu at (161.2, 31.8)
- added C30: C, Capacitor_SMD:C_0603_1608Metric, F.Cu at (160.4, 29.6)
- added C31: C, Capacitor_SMD:C_0603_1608Metric, F.Cu at (164.7, 31.8)
- added C32: C, Capacitor_SMD:C_0603_1608Metric, F.Cu at (163.9, 29.6)
- added C33: C, Capacitor_SMD:C_0603_1608Metric, F.Cu at (171.7, 31.8)
- added C34: C, Capacitor_SMD:C_0603_1608Metric, F.Cu at (167.4, 29.6)
- added C35: C, Capacitor_SMD:C_0603_1608Metric, F.Cu at (168.2, 31.8)
- added C36: C, Capacitor_SMD:C_0603_1608Metric, F.Cu at (170.9, 29.6)
- added C37: C, Capacitor_SMD:C_0603_1608Metric, F.Cu at (182.4, 28.5)
- added D7: ~, Package_TO_SOT_SMD:SOT-23_Handsoldering, F.Cu at (110.0, 142.4)
- added D8: ~, Package_TO_SOT_SMD:SOT-23_Handsoldering, F.Cu at (110.0, 147.0)
- added FB10: FerriteBead, Inductor_SMD:L_0603_1608Metric, F.Cu at (170.2, 31.8)
- added FB6: FerriteBead, Inductor_SMD:L_1206_3216Metric, F.Cu at (176.6, 25.8)
- added FB7: FerriteBead, Inductor_SMD:L_0603_1608Metric, F.Cu at (159.7, 31.8)
- added FB8: FerriteBead, Inductor_SMD:L_0603_1608Metric, F.Cu at (163.2, 31.8)
- added FB9: FerriteBead, Inductor_SMD:L_0603_1608Metric, F.Cu at (166.7, 31.8)
- added H1: MountingHole, MountingHole:MountingHole_3.2mm_M3, F.Cu at (155.5, 18.0)
- added H2: MountingHole, MountingHole:MountingHole_3.2mm_M3, F.Cu at (199.5, 18.0)
- added H3: MountingHole, MountingHole:MountingHole_3.2mm_M3, F.Cu at (199.5, 72.0)
- added H4: MountingHole, MountingHole:MountingHole_3.2mm_M3, F.Cu at (155.5, 72.0)
- added J2: Screw_Terminal_01x04, Connector_Phoenix_MC:PhoenixContact_MCV_1,5_4-G-3.5_1x04_P3.50mm_Vertical, F.Cu at (193.4, 18.2)
- added M1: HLK-LD2410C, project_lib:HLK-LD2410C, B.Cu at (177.5, 31.8)
- added Q1: BSS138, Package_TO_SOT_SMD:SOT-23, F.Cu at (190.8, 135.2)
- added Q2: 2N7002K, Package_TO_SOT_SMD:SOT-23, F.Cu at (182.9, 25.0)
- added Q3: 2N7002K, Package_TO_SOT_SMD:SOT-23, F.Cu at (186.4, 25.0)
- added Q4: BSS83P, Package_TO_SOT_SMD:SOT-23, F.Cu at (193.4, 26.5)
- added Q5: BSS83P, Package_TO_SOT_SMD:SOT-23, F.Cu at (189.9, 26.5)
- added Q6: 2N7002DW, Package_TO_SOT_SMD:SOT-363_SC-70-6, F.Cu at (191.6, 31.5)
- added R29: 1, Resistor_SMD:R_0603_1608Metric, F.Cu at (189.9, 23.8)
- added R3: R, Resistor_SMD:R_0603_1608Metric, F.Cu at (193.5, 135.2)
- added R30: 200, Resistor_SMD:R_0603_1608Metric, F.Cu at (160.5, 23.9)
- added R31: 200, Resistor_SMD:R_0603_1608Metric, F.Cu at (167.5, 23.9)
- added R32: 200, Resistor_SMD:R_0603_1608Metric, F.Cu at (164.0, 23.9)
- added R33: 200, Resistor_SMD:R_0603_1608Metric, F.Cu at (171.0, 23.9)
- added R34: R, Resistor_SMD:R_0603_1608Metric, F.Cu at (185.4, 28.5)
- added R35: R, Resistor_SMD:R_0603_1608Metric, F.Cu at (183.9, 28.5)
- added R4: R, Resistor_SMD:R_0603_1608Metric, F.Cu at (189.9, 29.2)
- added R5: R, Resistor_SMD:R_0603_1608Metric, F.Cu at (193.4, 29.2)
- added R6: R, Resistor_SMD:R_0603_1608Metric, F.Cu at (194.4, 31.5)
- added U10: UCC27517, Package_TO_SOT_SMD:SOT-23-5, F.Cu at (160.6, 26.8)
- added U11: UCC27517, Package_TO_SOT_SMD:SOT-23-5, F.Cu at (167.6, 26.8)
- added U12: UCC27517, Package_TO_SOT_SMD:SOT-23-5, F.Cu at (164.1, 26.8)
- added U13: UCC27517, Package_TO_SOT_SMD:SOT-23-5, F.Cu at (171.1, 26.8)
- added U2: TXB0102DCT, Package_SO:TSSOP-8_3x3mm_P0.65mm, F.Cu at (195.8, 143.8)
- added U7: APE8865N-33-HF-3, Package_TO_SOT_SMD:SOT-23, F.Cu at (195.8, 147.2)
- added U8: LM393A, Package_SO:VSSOP-8_3.0x3.0mm_P0.65mm, F.Cu at (184.6, 31.8)
- added U9: L78L12_SOT89, Package_TO_SOT_SMD:SOT-89-3, F.Cu at (177.6, 30.5)
- C21, C22: footprint Capacitor_SMD:C_0603_1608Metric -> Capacitor_SMD:C_1206_3216Metric
- J10: footprint project_lib:Tag-Connect_TC2030-IDC-NL_2x03_P1.27mm_Vertical -> Connector_PinHeader_2.54mm:PinHeader_2x03_P2.54mm_Vertical
- J4: value Conn_01x04 -> Screw_Terminal_01x05; footprint Connector_PinSocket_2.54mm:PinSocket_1x04_P2.54mm_Vertical -> Connector_Phoenix_MC:PhoenixContact_MCV_1,5_5-G-3.81_1x05_P3.81mm_Vertical
- R26: value R -> 1
- U4: footprint Package_TO_SOT_SMD:SOT-563 -> Package_TO_SOT_SMD:SOT-363_SC-70-6
- moved J4 110.9 mm to (177.1, 18.2)
- moved C25 103.4 mm to (186.9, 28.5), turned to 90 degrees
- moved C23 100.0 mm to (185.4, 35.0)
- moved R1 98.5 mm to (183.9, 35.0), turned to 90 degrees
- moved R2 96.9 mm to (186.9, 35.0), turned to -90 degrees
- moved C24 93.2 mm to (182.4, 35.0), turned to -90 degrees
- moved R26 86.5 mm to (193.4, 23.8), turned to 0 degrees
- moved R23 80.4 mm to (188.9, 31.5), turned to 90 degrees
- moved C22 80.2 mm to (179.1, 25.8), turned to -90 degrees
- moved C21 79.9 mm to (174.1, 25.8), turned to 90 degrees
- moved R25 63.7 mm to (172.5, 45.0)
- moved R24 59.7 mm to (167.5, 43.2)
- moved C1 55.1 mm to (141.0, 161.4)
- moved C2 55.1 mm to (125.5, 160.6)
- moved C3 55.1 mm to (125.5, 159.0)
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Connections:
- net /RX1 renamed /MCU/ISP_MISO
- net /TX1 renamed /MCU/ISP_MOSI
- C11 pad 1: +24V -> +5V
- C16 pad 2: +24V -> +5V
- C21 pad 1: /MCU/_ENC_B -> GND
- C21 pad 2: GND -> +24V
- C22 pad 1: /MCU/_ENC_A -> GND
- C22 pad 2: GND -> Net-(U9-IN)
- C23 pad 1: /light sensor/PT- -> /damp/VREF
- C23 pad 2: /light sensor/PTout -> GND
- C24 pad 1: GND -> +24V
- C24 pad 2: /LS -> GND
- C25 pad 1: GND -> Net-(U8A-+)
- C25 pad 2: +5VA -> GND
- F1 pad 2: Net-(F1-Pad2) -> +24V
- J4 pad 2: /OUT0 -> /out/OUT3
- J4 pad 3: /OUT1 -> /out/OUT2
- J4 pad 4: +5V -> /out/OUT1
- R1 pad 1: /light sensor/PT- -> +24V
- R1 pad 2: /light sensor/PTout -> /damp/VREF
- R14 pad 1: Net-(F1-Pad2) -> +24V
- R14 pad 2: +24V -> +5V
- R2 pad 1: /light sensor/PTout -> /damp/VREF
- R2 pad 2: /LS -> GND
- R20 pad 2: +24V -> +5V
- R23 pad 1: /MCU/_ENC_B -> /MCU/A_EN
- R23 pad 2: /ENC_B -> GND
- R24 pad 1: /MCU/_ENC_A -> +5V
- R24 pad 2: /ENC_A -> /MCU/A_FB
- R25 pad 2: /ENC_B -> /MCU/B_FB
- R26 pad 1: +5V -> /damp/A+
- R26 pad 2: /ENC_A -> Net-(Q4-D)
- U3 pad 1: /P0 -> /MCU/INT1
- U3 pad 10: /OUT0 -> /DIM0
- U3 pad 13: /OUT2 -> /DIM2
- U3 pad 14: /OUT3 -> /DIM3
- U3 pad 19: /SS -> unconnected-(U3-PE2-Pad19)
- U3 pad 25: /MCU/_ENC_B -> unconnected-(U3-PC2-Pad25)
- U3 pad 26: /MCU/_ENC_A -> unconnected-(U3-PC3-Pad26)
- U3 pad 27: /LS -> unconnected-(U3-PC4-Pad27)
- U3 pad 28: /P1 -> unconnected-(U3-PC5-Pad28)
- U3 pad 9: /OUT1 -> /DIM1
- U5 pad 5: +24V -> +5V
Routing:
- net +5V: track 162.8 -> 28.0 mm, vias 8 -> 0
- net /MCU/ISP_MOSI: track 56.5 -> 0.00 mm
- net /MCU/ISP_MISO: track 46.4 -> 0.00 mm
- net /SDA: track 38.1 -> 0.00 mm, vias 1 -> 0
- net /SCL: track 38.1 -> 0.00 mm, vias 1 -> 0
- net VBUS: track 36.3 -> 0.00 mm
- net /MCU/~{ISP_RST}: track 34.9 -> 0.00 mm, vias 2 -> 0
- net /ENC_A: track 31.9 -> 0.00 mm, vias 2 -> 0
- net /MCU/CD: track 31.1 -> 0.00 mm
- net /ENC_B: track 28.0 -> 0.00 mm, vias 2 -> 0
- net /MCU/RXD: track 28.3 -> 3.34 mm
- net /OUT3: track 23.9 -> 0.00 mm, vias 2 -> 0
- net /OUT2: track 23.5 -> 0.00 mm, vias 2 -> 0
- net +5VA: track 25.0 -> 4.23 mm, vias 2 -> 0
- net /OUT1: track 20.6 -> 0.00 mm
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Other:
- board size 44 x 40.5 mm -> 50 x 60 mm

Commit message: working
Parts:
- removed J11: Screw_Terminal_01x04, Connector_Phoenix_MC:PhoenixContact_MCV_1,5_4-G-3.81_1x04_P3.81mm_Vertical
- added C38: C, Capacitor_SMD:C_0603_1608Metric, F.Cu at (90.9, 129.0)
- added J1: Screw_Terminal_01x02, Connector_Phoenix_MC:PhoenixContact_MC_1,5_2-G-3.81_1x02_P3.81mm_Horizontal, F.Cu at (187.9, 60.3)
- added J3: Screw_Terminal_01x02, Connector_Phoenix_MC:PhoenixContact_MC_1,5_2-G-3.81_1x02_P3.81mm_Horizontal, F.Cu at (163.4, 60.3)
- added J6: Screw_Terminal_01x02, Connector_Phoenix_MSTB:PhoenixContact_MSTBA_2,5_2-G_1x02_P5.00mm_Horizontal, F.Cu at (175.0, 58.2)
- added Q7: Q_Photo_NPN, LED_THT:LED_D3.0mm_Clear, F.Cu at (84.7, 130.5)
- added R36: R, Resistor_SMD:R_0603_1608Metric, F.Cu at (90.9, 131.5)
- J2: footprint Connector_Phoenix_MC:PhoenixContact_MCV_1,5_4-G-3.5_1x04_P3.50mm_Vertical -> Connector_Phoenix_MC:PhoenixContact_MC_1,5_4-G-3.5_1x04_P3.50mm_Horizontal
- J4: footprint Connector_Phoenix_MC:PhoenixContact_MCV_1,5_5-G-3.81_1x05_P3.81mm_Vertical -> Connector_Phoenix_MC:PhoenixContact_MC_1,5_5-G-3.81_1x05_P3.81mm_Horizontal
- moved C4 140.9 mm to (197.7, 37.0), turned to -90 degrees
- moved FB1 139.0 mm to (196.2, 37.0), turned to -90 degrees
- moved C7 137.7 mm to (200.0, 52.5), turned to -90 degrees
- moved C5 137.0 mm to (194.8, 37.0), turned to 90 degrees
- moved C1 134.9 mm to (193.2, 37.0), turned to 90 degrees
- moved Y1 133.5 mm to (197.0, 52.5), turned to 0 degrees
- moved U3 130.6 mm to (192.8, 44.8), turned to 90 degrees
- moved C6 129.4 mm to (194.0, 52.5), turned to 90 degrees
- moved C2 127.1 mm to (192.3, 52.5), turned to 90 degrees
- moved C3 124.9 mm to (190.8, 52.5), turned to 90 degrees
- moved R28 122.1 mm to (188.5, 51.8), turned to 180 degrees
- moved R27 121.6 mm to (188.5, 53.2), turned to 180 degrees
- moved C17 48.6 mm to (159.0, 41.7), turned to 0 degrees
- moved C18 44.0 mm to (154.8, 41.8), turned to 180 degrees
- moved U6 41.7 mm to (159.0, 46.2), turned to -90 degrees
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Connections:
- C11 pad 1: +5V -> VCCQ
- C16 pad 2: +5V -> VCCQ
- R14 pad 2: +5V -> VCCQ
- R20 pad 2: +5V -> VCCQ
- U3 pad 19: unconnected-(U3-PE2-Pad19) -> /ALS
- U3 pad 22: /MOSI -> unconnected-(U3-PE3-Pad22)
- U3 pad 23: /MISO -> /MCU/A_EN
- U3 pad 24: /SCK -> /MCU/B_EN
- U3 pad 25: unconnected-(U3-PC2-Pad25) -> /MCU/OPN
- U3 pad 26: unconnected-(U3-PC3-Pad26) -> /MCU/CLS
- U3 pad 27: unconnected-(U3-PC4-Pad27) -> /MCU/A_FB
- U3 pad 28: unconnected-(U3-PC5-Pad28) -> /MCU/B_FB
- U5 pad 5: +5V -> VCCQ
Routing:
- net VBUS: track 0.00 -> 18.1 mm
- net +12V: track 16.5 -> 28.0 mm
- net /damp/O-: track 4.56 -> 9.43 mm
- net /damp/B+: track 11.9 -> 16.2 mm
- net +5V: track 28.0 -> 23.8 mm
- net /DIM3: track 0.00 -> 2.84 mm
- net /DIM2: track 0.00 -> 2.84 mm
- net /DIM1: track 0.00 -> 2.84 mm
- net /DIM0: track 0.00 -> 2.84 mm
- net /out/OUT0: track 5.86 -> 7.69 mm
- net /damp/C-: track 4.56 -> 6.01 mm
- net /damp/A+: track 14.1 -> 15.6 mm
- net Net-(U8B-+): track 3.04 -> 4.16 mm
- net /out/OUT2: track 6.11 -> 5.39 mm
- net /out/OUT1: track 5.99 -> 6.50 mm
Other:
- board size 50 x 60 mm -> 50 x 50 mm
