File: hardware/room_hub/room_hub.kicad_sch (KiCad schematic)
At the start: 6 parts, among them J1 Conn_01x05, J3 Conn_02x05_Odd_Even, J4 Conn_01x04, J5 Conn_01x04, J6 Conn_01x04, SW1 RotaryEncoder

Commit message: hw layout
Parts:
- removed J1: Conn_01x05, Connector_PinSocket_2.54mm:PinSocket_1x05_P2.54mm_Vertical, symbol Connector_Generic:Conn_01x05
- removed J3: Conn_02x05_Odd_Even, Connector_PinSocket_2.54mm:PinSocket_2x05_P2.54mm_Vertical_SMD, symbol Connector_Generic:Conn_02x05_Odd_Even
- removed J4: Conn_01x04, Connector_PinSocket_2.54mm:PinSocket_1x04_P2.54mm_Vertical, symbol Connector_Generic:Conn_01x04
- removed J6: Conn_01x04, Connector_JST:JST_PH_B4B-PH-K_1x04_P2.00mm_Vertical, symbol Connector_Generic:Conn_01x04
- removed SW1: RotaryEncoder, project_lib:EC35A0930401, symbol Device:RotaryEncoder
- added H1, H2, H3, H4: MountingHole, MountingHole:MountingHole_3.2mm_M3, symbol Mechanical:MountingHole
Other:
- removed sheet LED_out
- removed sheet light sensor
- added sheet damp (damp.kicad_sch)
- added sheet out (out.kicad_sch)
- added sheet radar (radar.kicad_sch)
- sheet MCU ports: added A_EN, A_FB, B_EN, B_FB, CLS, INT1, OPN, {DIM[0..3]}; removed ALS, ENC_A, ENC_B, ENC_P0, ENC_P1, SS1, {OUT[0..3]}
- note removed: "38,5mm apart"

Commit message: working
Parts:
- added C38: C, Capacitor_SMD:C_0603_1608Metric, symbol Device:C
- added Q7: Q_Photo_NPN, LED_THT:LED_D3.0mm_Clear, symbol Device:Q_Photo_NPN
- added R36: R, Resistor_SMD:R_0603_1608Metric, symbol Device:R
Connections:
- net +5V: now also Q7.1 (C)
- net GND: now also C38.2, R36.2
- new net ALS: C38.1, Q7.2 (E), R36.1
Other:
- sheet MCU ports: added ALS; removed none
