File: hardware/corridor_distribution/IO.kicad_sch (KiCad schematic)
At the start: 4 parts, among them U4 TCA9554PW

Commit message: led balance and corridor ready
Parts:
- added C12, C13: 100n 50V, Capacitor_SMD:C_0603_1608Metric, symbol Device:C
- added JP4: IO7, Jumper:SolderJumper-2_P1.3mm_Open_RoundedPad1.0x1.5mm, symbol Jumper:SolderJumper_2_Open
- added R1: 4.7k, Resistor_SMD:R_0603_1608Metric, symbol Device:R
- added R1: 100k, Resistor_SMD:R_0603_1608Metric, symbol Device:R
- added U7: 74LVC1G17, Package_TO_SOT_SMD:SOT-353_SC-70-5, symbol 74xGxx:74LVC1G17
- C6: value C -> 100n 50V; LCSC Part # (none) -> C14663; Total quantity (none) -> 30
- RN4: value R_Pack04_Split -> 4.7k; LCSC Part # (none) -> C700514; Total quantity (none) -> 10
- U4: value TCA9554PW -> TCA9554APW; LCSC Part # (none) -> C2863976; Total quantity (none) -> 5
Connections:
- net +5V: now also C12.1, R1.2, U7.5 (VCC)
- net GND: now also C12.2, C13.2, U7.3 (GND)
- net IO7: now also JP4.2 (B), R1.1, R1.1; no longer RN4.5 (R4.2), U4.12 (P7)
- new net IO7F: C13.1, R1.2, U7.2
- new net IO7S: JP4.1 (A), RN4.5 (R4.2), U4.12 (P7), U7.4
Other:
- note added: "Address (non A ver) = 0 1 0 0 A2 A1 A0 (0x20) Address (A version) = 0 1 1 1 A2 A1 A0 (0x38)"
- note added: "R_{SER} > 10*R_{PU}"
- note removed: "Address = 0 1 0 0 A2 A1 A0"
- moved on the sheet: C6, RN4A, RN4B, RN4C, RN4D, U4

Commit message: Night Light firmware
Parts:
- renumbered JP4 to JP1, R1 to R12, R1 to R13
Other:
- note added: "Address (non A ver) = _ 0 1 0 0 A2 A1 A0 (0x20) Address (A version) = _ 0 1 1 1 A2 A1 A0 (0x38) <-- mounted"
- note removed: "Address (non A ver) = 0 1 0 0 A2 A1 A0 (0x20) Address (A version) = 0 1 1 1 A2 A1 A0 (0x38)"
