File: hardware/corridor_distribution/corridor_distribution.kicad_sch (KiCad schematic)
At the start: 2 parts

Commit message: led balance and corridor ready
Parts:
- H1, H2: now left out of the parts list
Changed lines of the file:
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@@
   )
   (symbol (lib_id "Mechanical:MountingHole") (at 38.1 38.1 0) (unit 1)
-    (in_bom yes) (on_board yes) (dnp no) (fields_autoplaced)
+    (in_bom no) (on_board yes) (dnp no) (fields_autoplaced)
     (property "Reference" "H1" (at 40.64 37.2653 0)
       (effects (font (size 1.27 1.27)) (justify left))
@@
       (effects (font (size 1.27 1.27)) hide)
     )
+    (property "LCSC Part #" "" (at 38.1 38.1 0)
+      (effects (font (size 1.27 1.27)) hide)
+    )
+    (property "Total quantity" "" (at 38.1 38.1 0)
+      (effects (font (size 1.27 1.27)) hide)
+    )
     (instances
-      (project "multi_led_driver"
+      (project "corridor_distribution"
         (path "/d4c2f312-ca5d-462b-a371-0fb5d5a0cf93"
           (reference "H1") (unit 1)
@@
   )
   (symbol (lib_id "Mechanical:MountingHole") (at 38.1 44.45 0) (unit 1)
-    (in_bom yes) (on_board yes) (dnp no) (fields_autoplaced)
+    (in_bom no) (on_board yes) (dnp no) (fields_autoplaced)
     (property "Reference" "H2" (at 40.64 43.6153 0)
       (effects (font (size 1.27 1.27)) (justify left))
@@
       (effects (font (size 1.27 1.27)) hide)
     )
+    (property "LCSC Part #" "" (at 38.1 44.45 0)
+      (effects (font (size 1.27 1.27)) hide)
+    )
+    (property "Total quantity" "" (at 38.1 44.45 0)
+      (effects (font (size 1.27 1.27)) hide)
+    )
     (instances
-      (project "multi_led_driver"
+      (project "corridor_distribution"
         (path "/d4c2f312-ca5d-462b-a371-0fb5d5a0cf93"
           (reference "H2") (unit 1)
@@
     )
     (instances
-      (project "multi_led_driver"
+      (project "corridor_distribution"
         (path "/d4c2f312-ca5d-462b-a371-0fb5d5a0cf93" (page "37"))
       )
@@
     )
     (instances
-      (project "multi_led_driver"
+      (project "corridor_distribution"
         (path "/d4c2f312-ca5d-462b-a371-0fb5d5a0cf93" (page "7"))
       )
@@
     )
     (instances
-      (project "multi_led_driver"
+      (project "corridor_distribution"
         (path "/d4c2f312-ca5d-462b-a371-0fb5d5a0cf93" (page "39"))
       )
@@
     )
     (instances
-      (project "multi_led_driver"
+      (project "corridor_distribution"
         (path "/d4c2f312-ca5d-462b-a371-0fb5d5a0cf93" (page "40"))
       )
@@
     )
     (instances
-      (project "multi_led_driver"
+      (project "corridor_distribution"
         (path "/d4c2f312-ca5d-462b-a371-0fb5d5a0cf93" (page "38"))
       )
@@
     )
     (instances
-      (project "multi_led_driver"
+      (project "corridor_distribution"
         (path "/d4c2f312-ca5d-462b-a371-0fb5d5a0cf93" (page "36"))
       )

Commit message: various
Other:
- sheet power_in ports: added CS; removed none
Changed lines of the file:
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@@
+    (stroke (width 0) (type default))
+  )
+  (wire (pts (xy 127 107.95) (xy 128.27 107.95))
     (stroke (width 0) (type default))
   )
@@
   (label "{ADR}" (at 111.76 60.96 180) (fields_autoplaced)
     (effects (font (size 1.27 1.27)) (justify right bottom))
+  )
+  (label "CS" (at 128.27 107.95 0) (fields_autoplaced)
+    (effects (font (size 1.27 1.27)) (justify left bottom))
   )
   (label "{ADR}" (at 180.34 111.76 0) (fields_autoplaced)
@@
       (effects (font (size 1.27 1.27)) (justify left top))
     )
-    (instances
+    (pin "CS" output (at 127 107.95 0)
+      (effects (font (size 1.27 1.27)) (justify right))
+    )
+    (instances
