File: hardware/corridor_distribution/node_conn.kicad_sch (KiCad schematic)
At the start: 3 parts, among them J6 Screw_Terminal_01x06

Commit message: led balance and corridor ready
Parts:
- D14, D6: value D -> SM05; LCSC Part # (none) -> C460613; Total quantity (none) -> 100
- J6: now left out of the parts list
Changed lines of the file:
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@@
       (effects (font (size 1.27 1.27)))
     )
-    (property "Value" "D" (at 69.85 60.96 0)
+    (property "Value" "SM05" (at 69.85 60.96 0)
       (effects (font (size 1.27 1.27)))
     )
@@
     )
     (property "Datasheet" "https://www.littelfuse.com/~/media/electronics/datasheets/tvs_diode_arrays/littelfuse_tvs_diode_array_sm712_datasheet.pdf.pdf" (at 73.66 63.5 0)
+      (effects (font (size 1.27 1.27)) hide)
+    )
+    (property "LCSC Part #" "C460613" (at 69.85 63.5 0)
+      (effects (font (size 1.27 1.27)) hide)
+    )
+    (property "Total quantity" "100" (at 69.85 63.5 0)
       (effects (font (size 1.27 1.27)) hide)
     )
@@
     (pin "3")
     (instances
-      (project "multi_led_driver"
+      (project "corridor_distribution"
         (path "/d4c2f312-ca5d-462b-a371-0fb5d5a0cf93/1aca686d-2447-4f34-be8b-d923e9c8fa6d/a73f9a82-c47b-4816-a401-331a91601895"
           (reference "D6") (unit 1)
@@
   )
   (symbol (lib_id "Connector:Screw_Terminal_01x06") (at 127 78.74 0) (mirror x) (unit 1)
-    (in_bom yes) (on_board yes) (dnp no) (fields_autoplaced)
+    (in_bom no) (on_board yes) (dnp no) (fields_autoplaced)
     (property "Reference" "J6" (at 127 66.1502 0)
       (effects (font (size 1.27 1.27)))
@@
     )
     (property "Datasheet" "~" (at 127 78.74 0)
+      (effects (font (size 1.27 1.27)) hide)
+    )
+    (property "LCSC Part #" "" (at 127 78.74 0)
+      (effects (font (size 1.27 1.27)) hide)
+    )
+    (property "Total quantity" "" (at 127 78.74 0)
       (effects (font (size 1.27 1.27)) hide)
     )
@@
     (pin "6")
     (instances
-      (project "multi_led_driver"
+      (project "corridor_distribution"
         (path "/d4c2f312-ca5d-462b-a371-0fb5d5a0cf93/1aca686d-2447-4f34-be8b-d923e9c8fa6d/f09d4f16-a43e-4d70-add6-2630777eb0c8"
           (reference "J6") (unit 1)
@@
       (effects (font (size 1.27 1.27)))
     )
-    (property "Value" "D" (at 69.85 80.01 0)
+    (property "Value" "SM05" (at 69.85 80.01 0)
       (effects (font (size 1.27 1.27)))
     )
@@
     )
     (property "Datasheet" "https://www.littelfuse.com/~/media/electronics/datasheets/tvs_diode_arrays/littelfuse_tvs_diode_array_sm712_datasheet.pdf.pdf" (at 66.04 82.55 0)
+      (effects (font (size 1.27 1.27)) hide)
+    )
+    (property "LCSC Part #" "C460613" (at 69.85 82.55 0)
+      (effects (font (size 1.27 1.27)) hide)
+    )
+    (property "Total quantity" "100" (at 69.85 82.55 0)
       (effects (font (size 1.27 1.27)) hide)
     )
@@
     (pin "3")
     (instances
-      (project "multi_led_driver"
+      (project "corridor_distribution"
         (path "/d4c2f312-ca5d-462b-a371-0fb5d5a0cf93/1aca686d-2447-4f34-be8b-d923e9c8fa6d/a73f9a82-c47b-4816-a401-331a91601895"
           (reference "D14") (unit 1)
@@
     (pin "1")
     (instances
-      (project "multi_led_driver"
+      (project "corridor_distribution"
         (path "/d4c2f312-ca5d-462b-a371-0fb5d5a0cf93/1aca686d-2447-4f34-be8b-d923e9c8fa6d/f09d4f16-a43e-4d70-add6-2630777eb0c8"
           (reference "#PWR0112") (unit 1)
@@
     (pin "1")
     (instances
-      (project "multi_led_driver"
+      (project "corridor_distribution"
         (path "/d4c2f312-ca5d-462b-a371-0fb5d5a0cf93/1aca686d-2447-4f34-be8b-d923e9c8fa6d/f09d4f16-a43e-4d70-add6-2630777eb0c8"
           (reference "#PWR048") (unit 1)
@@
     (pin "1")
     (instances
-      (project "multi_led_driver"
+      (project "corridor_distribution"
         (path "/d4c2f312-ca5d-462b-a371-0fb5d5a0cf93/1aca686d-2447-4f34-be8b-d923e9c8fa6d/f09d4f16-a43e-4d70-add6-2630777eb0c8"
           (reference "#PWR0111") (unit 1)
@@
     (pin "1")
     (instances
-      (project "multi_led_driver"
+      (project "corridor_distribution"
         (path "/d4c2f312-ca5d-462b-a371-0fb5d5a0cf93/1aca686d-2447-4f34-be8b-d923e9c8fa6d/f09d4f16-a43e-4d70-add6-2630777eb0c8"
           (reference "#PWR056") (unit 1)

Commit message: Night Light firmware
Parts:
- renumbered D6 to D10, D14 to D18, J6 to J5
