File: hardware/corridor_distribution/nodes.kicad_sch (KiCad schematic)
At the start: 0 parts

Commit message: various
Parts:
- added R44 (x2): 330, Resistor_SMD:R_0603_1608Metric_Pad0.98x0.95mm_HandSolder, symbol Device:R
Connections:
- net PW14: now also R44.1
- net PW15: now also R44.1
- new net node conn 7/LED_C: R44.2
- new net node conn 7/LED_W: R44.2
Changed lines of the file:
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@@
     (stroke (width 0) (type default))
   )
-  (wire (pts (xy 158.75 130.81) (xy 161.29 130.81))
+  (wire (pts (xy 177.8 130.81) (xy 180.34 130.81))
     (stroke (width 0) (type default))
   )
@@
     (stroke (width 0) (type default))
   )
-  (wire (pts (xy 158.75 135.89) (xy 161.29 135.89))
+  (wire (pts (xy 177.8 135.89) (xy 180.34 135.89))
     (stroke (width 0) (type default))
   )
@@
     (stroke (width 0) (type default))
   )
-  (wire (pts (xy 137.16 130.81) (xy 139.7 130.81))
+  (wire (pts (xy 156.21 130.81) (xy 158.75 130.81))
     (stroke (width 0) (type default))
   )
@@
     (stroke (width 0) (type default))
   )
-  (wire (pts (xy 137.16 135.89) (xy 139.7 135.89))
+  (wire (pts (xy 156.21 135.89) (xy 158.75 135.89))
     (stroke (width 0) (type default))
   )
@@
     (effects (font (size 1.27 1.27)) (justify left bottom))
   )
-  (label "PW15" (at 137.16 135.89 180) (fields_autoplaced)
+  (label "PW15" (at 148.59 135.89 180) (fields_autoplaced)
     (effects (font (size 1.27 1.27)) (justify right bottom))
   )
@@
     (effects (font (size 1.27 1.27)) (justify left bottom))
   )
-  (label "PW14" (at 137.16 130.81 180) (fields_autoplaced)
+  (label "PW14" (at 148.59 130.81 180) (fields_autoplaced)
     (effects (font (size 1.27 1.27)) (justify right bottom))
   )
@@
     (effects (font (size 1.27 1.27)) (justify right bottom))
   )
-  (label "IO7" (at 161.29 135.89 0) (fields_autoplaced)
+  (label "IO7" (at 180.34 135.89 0) (fields_autoplaced)
     (effects (font (size 1.27 1.27)) (justify left bottom))
   )
@@
     (effects (font (size 1.27 1.27)) (justify right bottom))
   )
-  (label "AD7" (at 161.29 130.81 0) (fields_autoplaced)
+  (label "AD7" (at 180.34 130.81 0) (fields_autoplaced)
     (effects (font (size 1.27 1.27)) (justify left bottom))
   )
@@
   (hierarchical_label "AD[0..7]" (shape output) (at 215.9 83.82 0) (fields_autoplaced)
     (effects (font (size 1.27 1.27)) (justify left))
+  )
+  (symbol (lib_id "Device:R") (at 152.4 130.81 90) (unit 1)
+    (in_bom yes) (on_board yes) (dnp no)
+    (property "Reference" "R44" (at 152.4 133.35 90)
+      (effects (font (size 1.27 1.27)))
+    )
+    (property "Value" "330" (at 152.4 130.81 90)
+      (effects (font (size 1.27 1.27)))
+    )
+    (property "Footprint" "Resistor_SMD:R_0603_1608Metric_Pad0.98x0.95mm_HandSolder" (at 152.4 132.588 90)
+      (effects (font (size 1.27 1.27)) hide)
+    )
+    (property "Datasheet" "~" (at 152.4 130.81 0)
+      (effects (font (size 1.27 1.27)) hide)
+    )
+    (property "LCSC Part #" "C98220" (at 152.4 130.81 0)
+      (effects (font (size 1.27 1.27)) hide)
+    )
+    (property "Total quantity" "10" (at 152.4 130.81 0)
+      (effects (font (size 1.27 1.27)) hide)
+    )
+    (pin "1")
+    (pin "2")
+    (instances
+      (project "myWindow"
+        (path "/0e851ea5-1f1c-40d5-bf47-393077fa2f9e/18c72d34-702e-4a55-b186-6bdbdd75298d"
+          (reference "R44") (unit 1)
+        )
+      )
+      (project "corridor_distribution"
+        (path "/d4c2f312-ca5d-462b-a371-0fb5d5a0cf93/01427d6a-2fed-4662-9fee-1ada565cb5a0"
+          (reference "R9") (unit 1)
+        )
+        (path "/d4c2f312-ca5d-462b-a371-0fb5d5a0cf93/2321c199-a07b-4723-8fa0-97a4bbc3bc1c"
+          (reference "R9") (unit 1)
+        )
+        (path "/d4c2f312-ca5d-462b-a371-0fb5d5a0cf93/1aca686d-2447-4f34-be8b-d923e9c8fa6d"
+          (reference "R15") (unit 1)
+        )
+      )
+      (project "control_panel"
+        (path "/e63e39d7-6ac0-4ffd-8aa3-1841a4541b55/8ca9797e-e63e-4e59-a184-ef2a887eb814"
+          (reference "R26") (unit 1)
+        )
+      )
+    )
+  )
+  (symbol (lib_id "Device:R") (at 152.4 135.89 90) (unit 1)
+    (in_bom yes) (on_board yes) (dnp no)
+    (property "Reference" "R44" (at 152.4 138.43 90)
+      (effects (font (size 1.27 1.27)))
+    )
+    (property "Value" "330" (at 152.4 135.89 90)
+      (effects (font (size 1.27 1.27)))
+    )
+    (property "Footprint" "Resistor_SMD:R_0603_1608Metric_Pad0.98x0.95mm_HandSolder" (at 152.4 137.668 90)
+      (effects (font (size 1.27 1.27)) hide)
+    )
+    (property "Datasheet" "~" (at 152.4 135.89 0)
+      (effects (font (size 1.27 1.27)) hide)
+    )
+    (property "LCSC Part #" "C98220" (at 152.4 135.89 0)
+      (effects (font (size 1.27 1.27)) hide)
+    )
+    (property "Total quantity" "10" (at 152.4 135.89 0)
+      (effects (font (size 1.27 1.27)) hide)
+    )
+    (pin "1")
+    (pin "2")
+    (instances
+      (project "myWindow"
+        (path "/0e851ea5-1f1c-40d5-bf47-393077fa2f9e/18c72d34-702e-4a55-b186-6bdbdd75298d"
+          (reference "R44") (unit 1)
+        )
+      )
+      (project "corridor_distribution"
+        (path "/d4c2f312-ca5d-462b-a371-0fb5d5a0cf93/01427d6a-2fed-4662-9fee-1ada565cb5a0"
+          (reference "R9") (unit 1)
+        )
+        (path "/d4c2f312-ca5d-462b-a371-0fb5d5a0cf93/2321c199-a07b-4723-8fa0-97a4bbc3bc1c"
+          (reference "R9") (unit 1)
+        )
+        (path "/d4c2f312-ca5d-462b-a371-0fb5d5a0cf93/1aca686d-2447-4f34-be8b-d923e9c8fa6d"
+          (reference "R14") (unit 1)
+        )
+      )
+      (project "control_panel"
+        (path "/e63e39d7-6ac0-4ffd-8aa3-1841a4541b55/8ca9797e-e63e-4e59-a184-ef2a887eb814"
+          (reference "R26") (unit 1)
+        )
+      )
+    )
   )
   (sheet (at 139.7 76.2) (size 19.05 12.7) (fields_autoplaced)
@@
     )
   )
-  (sheet (at 139.7 127) (size 19.05 12.7) (fields_autoplaced)
+  (sheet (at 158.75 127) (size 19.05 12.7) (fields_autoplaced)
     (stroke (width 0.1524) (type solid))
     (fill (color 0 0 0 0.0000))
-    (property "Sheetname" "node conn 7" (at 139.7 126.2884 0)
+    (property "Sheetname" "node conn 7" (at 158.75 126.2884 0)
       (effects (font (size 1.27 1.27)) (justify left bottom))
     )
-    (property "Sheetfile" "node_conn.kicad_sch" (at 139.7 140.2846 0)
+    (property "Sheetfile" "node_conn.kicad_sch" (at 158.75 140.2846 0)
       (effects (font (size 1.27 1.27)) (justify left top))
     )
-    (pin "SEN_L" output (at 158.75 130.81 0)
-      (effects (font (size 1.27 1.27)) (justify right))
-    )
-    (pin "SEN_M" output (at 158.75 135.89 0)
-      (effects (font (size 1.27 1.27)) (justify right))
-    )
-    (pin "LED_C" input (at 139.7 130.81 180)
-      (effects (font (size 1.27 1.27)) (justify left))
-    )
-    (pin "LED_W" input (at 139.7 135.89 180)
-      (effects (font (size 1.27 1.27)) (justify left))
-    )
+    (pin "SEN_L" output (at 177.8 130.81 0)
+      (effects (font (size 1.27 1.27)) (justify right))
+    )
+    (pin "SEN_M" output (at 177.8 135.89 0)
+      (effects (font (size 1.27 1.27)) (justify right))
+    )
+    (pin "LED_C" input (at 158.75 130.81 180)
+      (effects (font (size 1.27 1.27)) (justify left))
+    )
+    (pin "LED_W" input (at 158.75 135.89 180)
+      (effects (font (size 1.27 1.27)) (justify left))
+    )
