File: hardware/corridor_distribution/pwm.kicad_sch (KiCad schematic)
At the start: 6 parts, among them U3 PCA9685PW

Commit message: led balance and corridor ready
Parts:
- added U2: PCA9635, Package_SO:TSSOP-28_4.4x9.7mm_P0.65mm, symbol Driver_LED:PCA9635
- C5: value C -> 100n 50V; LCSC Part # (none) -> C14663; Total quantity (none) -> 30
- RN1, RN2, RN3, RN4: value R_Pack04 -> 100; LCSC Part # (none) -> C136838; Total quantity (none) -> 20
- U3: LCSC Part # (none) -> C2678753; Total quantity (none) -> 5
Other:
- note added: "Address (PCA9685) = 1 A5 A4 A3 A2 A1 A0 -> 1 0 0 0 0 A1 A0"
- note removed: "Address = 0 1 0 0 A2 A1 A0"
- note removed: "Address = 1 A5 A4 A3 A2 A1 A0"

Commit message: various
Parts:
- added JP2, JP5: SolderJumper_2_Open, Jumper:SolderJumper-2_P1.3mm_Open_RoundedPad1.0x1.5mm, symbol Jumper:SolderJumper_2_Open
Connections:
- net GND: now also JP2.1 (A), JP5.2 (B); no longer U3.25 (EXTCLK)
- net ~{OE}: now also JP5.1 (A)
- new net: JP2.2 (B), U3.25 (EXTCLK)
Changed lines of the file:
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@@
-    (stroke (width 0) (type default))
-  )
-  (wire (pts (xy 116.84 86.36) (xy 107.95 86.36))
     (stroke (width 0) (type default))
   )
@@
     (stroke (width 0) (type default))
   )
+  (wire (pts (xy 101.6 86.36) (xy 116.84 86.36))
+    (stroke (width 0) (type default))
+  )
+  (wire (pts (xy 91.44 86.36) (xy 93.98 86.36))
+    (stroke (width 0) (type default))
+  )
   (wire (pts (xy 187.96 83.82) (xy 195.58 83.82))
     (stroke (width 0) (type default))
@@
     (stroke (width 0) (type default))
   )
+  (wire (pts (xy 91.44 88.9) (xy 91.44 86.36))
+    (stroke (width 0) (type default))
+  )
   (bus (pts (xy 198.12 124.46) (xy 198.12 127))
     (stroke (width 0) (type default))
@@
   )
   (wire (pts (xy 114.3 114.3) (xy 116.84 114.3))
-    (stroke (width 0) (type default))
-  )
-  (wire (pts (xy 107.95 86.36) (xy 107.95 91.44))
     (stroke (width 0) (type default))
   )
@@
   (label "PW10" (at 189.23 116.84 0) (fields_autoplaced)
     (effects (font (size 1.27 1.27)) (justify left bottom))
+  )
+  (label "~{OE}" (at 80.01 91.44 180) (fields_autoplaced)
+    (effects (font (size 1.27 1.27)) (justify right bottom))
   )
   (label "_PW6" (at 175.26 101.6 180) (fields_autoplaced)
@@
         (path "/d4c2f312-ca5d-462b-a371-0fb5d5a0cf93/cbc143e2-a435-47df-91fd-d639c7126821"
           (reference "#PWR0136") (unit 1)
+        )
+      )
+    )
+  )
+  (symbol (lib_id "Jumper:SolderJumper_2_Open") (at 97.79 86.36 0) (unit 1)
+    (in_bom yes) (on_board yes) (dnp no) (fields_autoplaced)
+    (property "Reference" "JP2" (at 97.79 80.01 0)
+      (effects (font (size 1.27 1.27)))
+    )
+    (property "Value" "SolderJumper_2_Open" (at 97.79 82.55 0)
+      (effects (font (size 1.27 1.27)))
+    )
+    (property "Footprint" "Jumper:SolderJumper-2_P1.3mm_Open_RoundedPad1.0x1.5mm" (at 97.79 86.36 0)
+      (effects (font (size 1.27 1.27)) hide)
+    )
+    (property "Datasheet" "~" (at 97.79 86.36 0)
+      (effects (font (size 1.27 1.27)) hide)
+    )
+    (pin "1")
+    (pin "2")
+    (instances
+      (project "corridor_distribution"
+        (path "/d4c2f312-ca5d-462b-a371-0fb5d5a0cf93/cbc143e2-a435-47df-91fd-d639c7126821"
+          (reference "JP2") (unit 1)
         )
       )
@@
     )
   )
+  (symbol (lib_id "Jumper:SolderJumper_2_Open") (at 80.01 95.25 270) (unit 1)
+    (in_bom yes) (on_board yes) (dnp no) (fields_autoplaced)
+    (property "Reference" "JP5" (at 82.55 93.98 90)
+      (effects (font (size 1.27 1.27)) (justify left))
+    )
+    (property "Value" "SolderJumper_2_Open" (at 82.55 96.52 90)
+      (effects (font (size 1.27 1.27)) (justify left))
+    )
+    (property "Footprint" "Jumper:SolderJumper-2_P1.3mm_Open_RoundedPad1.0x1.5mm" (at 80.01 95.25 0)
+      (effects (font (size 1.27 1.27)) hide)
+    )
+    (property "Datasheet" "~" (at 80.01 95.25 0)
+      (effects (font (size 1.27 1.27)) hide)
+    )
+    (pin "1")
+    (pin "2")
+    (instances
+      (project "corridor_distribution"
+        (path "/d4c2f312-ca5d-462b-a371-0fb5d5a0cf93/cbc143e2-a435-47df-91fd-d639c7126821"
+          (reference "JP5") (unit 1)
+        )
+      )
+    )
+  )
   (symbol (lib_id "power:GND") (at 134.62 127 0) (unit 1)
     (in_bom yes) (on_board yes) (dnp no) (fields_autoplaced)
@@
     )
   )
-  (symbol (lib_id "power:GND") (at 107.95 91.44 0) (unit 1)
-    (in_bom yes) (on_board yes) (dnp no) (fields_autoplaced)
-    (property "Reference" "#PWR0140" (at 107.95 97.79 0)
-      (effects (font (size 1.27 1.27)) hide)
-    )
-    (property "Value" "GND" (at 107.95 95.8834 0)
-      (effects (font (size 1.27 1.27)))
-    )
-    (property "Footprint" "" (at 107.95 91.44 0)
-      (effects (font (size 1.27 1.27)) hide)
-    )
-    (property "Datasheet" "" (at 107.95 91.44 0)
-      (effects (font (size 1.27 1.27)) hide)
-    )
+  (symbol (lib_id "power:GND") (at 80.01 99.06 0) (unit 1)
+    (in_bom yes) (on_board yes) (dnp no) (fields_autoplaced)
+    (property "Reference" "#PWR075" (at 80.01 105.41 0)
+      (effects (font (size 1.27 1.27)) hide)
+    )
+    (property "Value" "GND" (at 80.01 103.5034 0)
+      (effects (font (size 1.27 1.27)))
+    )
+    (property "Footprint" "" (at 80.01 99.06 0)
+      (effects (font (size 1.27 1.27)) hide)
+    )
+    (property "Datasheet" "" (at 80.01 99.06 0)
+      (effects (font (size 1.27 1.27)) hide)
+    )
+    (pin "1")
+    (instances
+      (project "corridor_distribution"
+        (path "/d4c2f312-ca5d-462b-a371-0fb5d5a0cf93/cbc143e2-a435-47df-91fd-d639c7126821"
+          (reference "#PWR075") (unit 1)
+        )
+      )
+    )
+  )
+  (symbol (lib_id "power:GND") (at 91.44 88.9 0) (unit 1)
+    (in_bom yes) (on_board yes) (dnp no) (fields_autoplaced)
+    (property "Reference" "#PWR0140" (at 91.44 95.25 0)
+      (effects (font (size 1.27 1.27)) hide)
+    )
+    (property "Value" "GND" (at 91.44 93.3434 0)
+      (effects (font (size 1.27 1.27)))
+    )
+    (property "Footprint" "" (at 91.44 88.9 0)
+      (effects (font (size 1.27 1.27)) hide)
+    )
+    (property "Datasheet" "" (at 91.44 88.9 0)
+      (effects (font (size 1.27 1.27)) hide)
+    )

Commit message: Night Light firmware
Other:
- note added: "Address (PCA9685) = 1 A5 A4 A3 A2 A1 A0 -> _ 1 0 0 0 0 A1 A0 (0x40)"
- note removed: "Address (PCA9685) = 1 A5 A4 A3 A2 A1 A0 -> 1 0 0 0 0 A1 A0"
