File: hardware/night_light/LED.kicad_sch (KiCad schematic)
At the start: 9 parts, among them U2 MT9284CS6

Commit message: night light ready
Parts:
- C5: value C -> 22u 10V
- C6: value C -> 10u 16V
- D2: value 6V-150mA -> 6V 150mA
- D3: value D_Schottky -> RB161VAM-20TR
- L2: value 22u -> CBC3225T220KR; L (none) -> 22u
- R4: value 2 -> 0.7
- U2: value MT9284CS6 -> MT9284-28J
Other:
- note added: "10u actual"
- note added: "4u actual"
- note added: "Order Part Number Package Remark Top Marking MT9284-28J SOT23-6 VFB=104mV B11G8W MT9284AS6 SOT23-6 VFB=104mV B1A8DC MT9284BS6 SOT23-6 VFB=250mV B1B8DC MT9284CS6 SOT23-6 VFB=300mV B1C8DC"
Changed lines of the file:
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@@
     (stroke (width 0) (type default))
+  )
+  (text "Order Part Number	Package		Remark		Top Marking\nMT9284-28J			SOT23-6		VFB=104mV	B11G8W\nMT9284AS6			SOT23-6		VFB=104mV	B1A8DC\nMT9284BS6			SOT23-6		VFB=250mV	B1B8DC\nMT9284CS6			SOT23-6		VFB=300mV	B1C8DC"
+    (at 38.1 31.75 0)
+    (effects (font (size 1.27 1.27)) (justify left bottom))
   )
   (text "V_out=6V\nI_L=250mA\nDelta_I_L=10%\nL=22uH\nI_peak=200mA"
@@
     (effects (font (size 1.27 1.27)) (justify left bottom))
   )
+  (text "10u actual" (at 58.42 125.73 0)
+    (effects (font (size 1.27 1.27)) (justify left bottom))
+  )
+  (text "4u actual" (at 114.3 124.46 0)
+    (effects (font (size 1.27 1.27)) (justify left bottom))
+  )
   (text "Part Number		VFB		Top Marking\nMT9284-28J		104mV	B11G8W\nMT9284AS6		104mV	B1A8DC\nMT9284BS6		250mV	B1B8DC\nMT9284CS6		300mV	B1C8DC"
     (at 234.95 55.88 0)
@@
   (symbol (lib_id "Device:R") (at 135.89 125.73 0) (unit 1)
     (in_bom yes) (on_board yes) (dnp no) (fields_autoplaced)
-    (property "Reference" "R4" (at 137.668 124.8953 0)
-      (effects (font (size 1.27 1.27)) (justify left))
-    )
-    (property "Value" "2" (at 137.668 127.4322 0)
+    (property "Reference" "R4" (at 138.43 124.46 0)
+      (effects (font (size 1.27 1.27)) (justify left))
+    )
+    (property "Value" "0.7" (at 138.43 127 0)
       (effects (font (size 1.27 1.27)) (justify left))
     )
@@
       (effects (font (size 1.27 1.27)) hide)
     )
+    (property "LCSC Part #" "" (at 135.89 125.73 0)
+      (effects (font (size 1.27 1.27)) hide)
+    )
     (pin "1")
     (pin "2")
@@
   (symbol (lib_id "Device:C") (at 63.5 113.03 0) (unit 1)
     (in_bom yes) (on_board yes) (dnp no) (fields_autoplaced)
-    (property "Reference" "C5" (at 66.421 112.1953 0)
-      (effects (font (size 1.27 1.27)) (justify left))
-    )
-    (property "Value" "C" (at 66.421 114.7322 0)
+    (property "Reference" "C5" (at 67.31 111.76 0)
+      (effects (font (size 1.27 1.27)) (justify left))
+    )
+    (property "Value" "22u 10V" (at 67.31 114.3 0)
       (effects (font (size 1.27 1.27)) (justify left))
     )
@@
       (effects (font (size 1.27 1.27)) hide)
     )
+    (property "LCSC Part #" "" (at 63.5 113.03 0)
+      (effects (font (size 1.27 1.27)) hide)
+    )
     (pin "1")
     (pin "2")
@@
   )
   (symbol (lib_id "Device:L") (at 88.9 96.52 90) (unit 1)
-    (in_bom yes) (on_board yes) (dnp no) (fields_autoplaced)
+    (in_bom yes) (on_board yes) (dnp no)
     (property "Reference" "L2" (at 88.9 92.3122 90)
       (effects (font (size 1.27 1.27)))
     )
-    (property "Value" "22u" (at 88.9 94.8491 90)
+    (property "Value" "CBC3225T220KR" (at 88.9 94.8491 90)
       (effects (font (size 1.27 1.27)))
     )
@@
       (effects (font (size 1.27 1.27)) hide)
     )
+    (property "LCSC Part #" "" (at 88.9 96.52 0)
+      (effects (font (size 1.27 1.27)) hide)
+    )
+    (property "L" "22u" (at 88.9 97.79 90) (show_name)
+      (effects (font (size 1.27 1.27)))
+    )
     (pin "1")
     (pin "2")
@@
   (symbol (lib_id "Device:LED") (at 135.89 113.03 90) (unit 1)
     (in_bom yes) (on_board yes) (dnp no) (fields_autoplaced)
-    (property "Reference" "D2" (at 138.811 113.7828 90)
+    (property "Reference" "D2" (at 139.7 113.3475 90)
       (effects (font (size 1.27 1.27)) (justify right))
     )
-    (property "Value" "6V-150mA" (at 138.811 116.3197 90)
+    (property "Value" "6V 150mA" (at 139.7 115.8875 90)
       (effects (font (size 1.27 1.27)) (justify right))
     )
@@
       (effects (font (size 1.27 1.27)) hide)
     )
+    (property "LCSC Part #" "" (at 135.89 113.03 0)
+      (effects (font (size 1.27 1.27)) hide)
+    )
     (pin "1")
     (pin "2")
@@
       (effects (font (size 1.27 1.27)) hide)
     )
+    (property "LCSC Part #" "" (at 138.43 119.38 0)
+      (effects (font (size 1.27 1.27)) hide)
+    )
     (pin "1")
     (instances
@@
       (effects (font (size 1.27 1.27)) hide)
     )
+    (property "LCSC Part #" "" (at 135.89 104.14 0)
+      (effects (font (size 1.27 1.27)) hide)
+    )
     (pin "1")
     (instances
@@
   )
   (symbol (lib_id "Driver_LED:LT3465") (at 88.9 114.3 0) (unit 1)
-    (in_bom yes) (on_board yes) (dnp no) (fields_autoplaced)
-    (property "Reference" "U2" (at 88.9 100.4402 0)
-      (effects (font (size 1.27 1.27)))
-    )
-    (property "Value" "MT9284CS6" (at 88.9 102.9771 0)
+    (in_bom yes) (on_board yes) (dnp no)
+    (property "Reference" "U2" (at 88.9 110.49 0)
+      (effects (font (size 1.27 1.27)))
+    )
+    (property "Value" "MT9284-28J" (at 88.9 101.6 0)
       (effects (font (size 1.27 1.27)))
     )
@@
       (effects (font (size 1.27 1.27) italic) (justify left) hide)
     )
-    (property "Datasheet" "https://www.analog.com/media/en/technical-documentation/data-sheets/3465fa.pdf" (at 90.17 127 0)
+    (property "Datasheet" "https://datasheet.lcsc.com/lcsc/1806141217_XI-AN-Aerosemi-Tech-MT9284BS6_C181740.pdf" (at 90.17 127 0)
+      (effects (font (size 1.27 1.27)) hide)
+    )
+    (property "LCSC Part #" "" (at 88.9 114.3 0)
       (effects (font (size 1.27 1.27)) hide)
     )
@@
   (symbol (lib_id "Device:D_Schottky") (at 107.95 106.68 180) (unit 1)
     (in_bom yes) (on_board yes) (dnp no) (fields_autoplaced)
-    (property "Reference" "D3" (at 108.2675 101.7102 0)
-      (effects (font (size 1.27 1.27)))
-    )
-    (property "Value" "D_Schottky" (at 108.2675 104.2471 0)
+    (property "Reference" "D3" (at 108.2675 100.33 0)
+      (effects (font (size 1.27 1.27)))
+    )
+    (property "Value" "RB161VAM-20TR" (at 108.2675 102.87 0)
       (effects (font (size 1.27 1.27)))
     )
@@
       (effects (font (size 1.27 1.27)) hide)
     )
+    (property "LCSC Part #" "" (at 107.95 106.68 0)
+      (effects (font (size 1.27 1.27)) hide)
+    )
     (pin "1")
     (pin "2")
@@
   (symbol (lib_id "Device:C") (at 119.38 113.03 0) (unit 1)
     (in_bom yes) (on_board yes) (dnp no) (fields_autoplaced)
-    (property "Reference" "C6" (at 122.301 112.1953 0)
-      (effects (font (size 1.27 1.27)) (justify left))
-    )
-    (property "Value" "C" (at 122.301 114.7322 0)
+    (property "Reference" "C6" (at 123.19 111.76 0)
+      (effects (font (size 1.27 1.27)) (justify left))
+    )
+    (property "Value" "10u 16V" (at 123.19 114.3 0)
       (effects (font (size 1.27 1.27)) (justify left))
     )
@@
       (effects (font (size 1.27 1.27)) hide)
     )
+    (property "LCSC Part #" "" (at 119.38 113.03 0)
+      (effects (font (size 1.27 1.27)) hide)
+    )

Commit message: various
Parts:
- C5: LCSC (none) -> C29277
- C6: LCSC (none) -> C1713
- D3: LCSC (none) -> C308725
- L2: LCSC (none) -> C223225
- R4: LCSC (none) -> C175718
- U2: LCSC (none) -> C181780
Other:
- note added: "Compatible diode packages: - TUMD2M - Power-DI-323 - SOD-323HE"
- note removed: "Part Number VFB Top Marking MT9284-28J 104mV B11G8W MT9284AS6 104mV B1A8DC MT9284BS6 250mV B1B8DC MT9284CS6 300mV B1C8DC"
Changed lines of the file:
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@@
+    (effects (font (size 1.27 1.27)) (justify left bottom))
+  )
+  (text "Compatible diode packages:\n- TUMD2M\n- Power-DI-323\n- SOD-323HE"
+    (at 106.68 92.71 0)
     (effects (font (size 1.27 1.27)) (justify left bottom))
   )
@@
     (effects (font (size 1.27 1.27)) (justify left bottom))
   )
-  (text "Part Number		VFB		Top Marking\nMT9284-28J		104mV	B11G8W\nMT9284AS6		104mV	B1A8DC\nMT9284BS6		250mV	B1B8DC\nMT9284CS6		300mV	B1C8DC"
-    (at 234.95 55.88 0)
-    (effects (font (size 1.27 1.27)) (justify left bottom))
-  )
   (label "LED-" (at 128.27 119.38 0) (fields_autoplaced)
     (effects (font (size 1.27 1.27)) (justify left bottom))
@@
       (effects (font (size 1.27 1.27)) hide)
     )
+    (property "LCSC" "C175718" (at 138.43 124.46 0)
+      (effects (font (size 1.27 1.27)) hide)
+    )
     (pin "1")
     (pin "2")
@@
     )
     (property "LCSC Part #" "" (at 63.5 113.03 0)
+      (effects (font (size 1.27 1.27)) hide)
+    )
+    (property "LCSC" "C29277" (at 67.31 111.76 0)
       (effects (font (size 1.27 1.27)) hide)
     )
@@
       (effects (font (size 1.27 1.27)))
     )
+    (property "LCSC" "C223225" (at 88.9 92.3122 0)
+      (effects (font (size 1.27 1.27)) hide)
+    )
     (pin "1")
     (pin "2")
@@
     )
     (property "LCSC Part #" "" (at 88.9 114.3 0)
+      (effects (font (size 1.27 1.27)) hide)
+    )
+    (property "LCSC" "C181780" (at 88.9 110.49 0)
       (effects (font (size 1.27 1.27)) hide)
     )
@@
       (effects (font (size 1.27 1.27)) hide)
     )
+    (property "LCSC" "C308725" (at 108.2675 100.33 0)
+      (effects (font (size 1.27 1.27)) hide)
+    )
     (pin "1")
     (pin "2")
@@
       (effects (font (size 1.27 1.27)) hide)
     )
+    (property "LCSC" "C1713" (at 123.19 111.76 0)
+      (effects (font (size 1.27 1.27)) hide)
+    )

Commit message: Night Light firmware
Changed lines of the file:
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@@
 (kicad_sch
-	(version 20231120)
+	(version 20250114)
 	(generator "eeschema")
-	(generator_version "8.0")
+	(generator_version "9.0")
 	(paper "A4")
+	(text "Order Part Number	Package		Remark		Top Marking\nMT9284-28J			SOT23-6		VFB=104mV	B11G8W\nMT9284AS6			SOT23-6		VFB=104mV	B1A8DC\nMT9284BS6			SOT23-6		VFB=250mV	B1B8DC\nMT9284CS6			SOT23-6		VFB=300mV	B1C8DC"
+		(exclude_from_sim no)
+		(at 38.1 31.75 0)
+		(effects
+			(font
+				(size 1.27 1.27)
+			)
+			(justify left bottom)
+		)
+	)
+	(text "Compatible diode packages:\n- TUMD2M\n- Power-DI-323\n- SOD-323HE"
+		(exclude_from_sim no)
+		(at 106.68 92.71 0)
+		(effects
+			(font
+				(size 1.27 1.27)
+			)
+			(justify left bottom)
+		)
+	)
+	(text "V_out=6V\nI_L=250mA\nDelta_I_L=10%\nL=22uH\nI_peak=200mA"
+		(exclude_from_sim no)
+		(at 93.98 76.2 0)
+		(effects
+			(font
+				(size 1.27 1.27)
+			)
+			(justify left bottom)
+		)
+	)
+	(text "10u actual"
+		(exclude_from_sim no)
+		(at 58.42 125.73 0)
+		(effects
+			(font
+				(size 1.27 1.27)
+			)
+			(justify left bottom)
+		)
+	)
+	(text "4u actual"
+		(exclude_from_sim no)
+		(at 114.3 124.46 0)
+		(effects
+			(font
+				(size 1.27 1.27)
+			)
+			(justify left bottom)
+		)
+	)
 	(junction
 		(at 135.89 119.38)
@@
 			(width 0)
 			(type default)
-		)
-	)
-	(text "Order Part Number	Package		Remark		Top Marking\nMT9284-28J			SOT23-6		VFB=104mV	B11G8W\nMT9284AS6			SOT23-6		VFB=104mV	B1A8DC\nMT9284BS6			SOT23-6		VFB=250mV	B1B8DC\nMT9284CS6			SOT23-6		VFB=300mV	B1C8DC"
-		(exclude_from_sim no)
-		(at 38.1 31.75 0)
-		(effects
-			(font
-				(size 1.27 1.27)
-			)
-			(justify left bottom)
-		)
-	)
-	(text "Compatible diode packages:\n- TUMD2M\n- Power-DI-323\n- SOD-323HE"
-		(exclude_from_sim no)
-		(at 106.68 92.71 0)
-		(effects
-			(font
-				(size 1.27 1.27)
-			)
-			(justify left bottom)
-		)
-	)
-	(text "V_out=6V\nI_L=250mA\nDelta_I_L=10%\nL=22uH\nI_peak=200mA"
-		(exclude_from_sim no)
-		(at 93.98 76.2 0)
-		(effects
-			(font
-				(size 1.27 1.27)
-			)
-			(justify left bottom)
-		)
-	)
-	(text "10u actual"
-		(exclude_from_sim no)
-		(at 58.42 125.73 0)
-		(effects
-			(font
-				(size 1.27 1.27)
-			)
-			(justify left bottom)
-		)
-	)
-	(text "4u actual"
-		(exclude_from_sim no)
-		(at 114.3 124.46 0)
-		(effects
-			(font
-				(size 1.27 1.27)
-			)
-			(justify left bottom)
 		)
 	)
 	(label "LED-"
 		(at 128.27 119.38 0)
-		(fields_autoplaced yes)
 		(effects
 			(font
@@
 	(label "LED+"
 		(at 124.46 106.68 0)
-		(fields_autoplaced yes)
 		(effects
 			(font
@@
 	(label "SW"
 		(at 99.06 96.52 0)
-		(fields_autoplaced yes)
 		(effects
 			(font
@@
 		(shape input)
 		(at 76.2 116.84 180)
-		(fields_autoplaced yes)
-		(effects
-			(font
+		(effects
+			(font
