File: hardware/night_light/battery.kicad_sch (KiCad schematic)
At the start: 15 parts, among them J3 Conn_01x02_Male, Q1 Q_PMOS_GSD, U3 MCP73832-2-OT

Commit message: night light ready
Parts:
- C11: value C_Polarized -> 220u 6.3V
- C16: value C -> 100n 50V
- C7, C8, C9: value C -> 4.7u 16V
- D5: value D_Schottky -> RB161VAM-20TR
- J3: value Conn_01x02_Male -> JST PH
- Q1: value Q_PMOS_GSD -> AO3401A
- R5: value R -> 3.9k
- R6: value R -> 2.2k
- R7: value R -> 2.43k
- R8: value R -> 1k
Other:
- note added: "1.1V reference (1.0V min / 1.2V max) 4.5V input 100mV margin = 1.3V"
- note added: "Actual 2.7uF"
- note added: "I_chg=~250mA"
- moved on the sheet: C11, C7, J3

Commit message: various
Parts:
- removed C11: 220u 6.3V, Capacitor_SMD:CP_Elec_6.3x5.7, symbol Device:C_Polarized
- added C18: 100uF 6.3V, Capacitor_Tantalum_SMD:CP_EIA-3528-15_AVX-H, symbol Device:C_Polarized
- C16: LCSC (none) -> C14663
- C7, C8, C9: LCSC (none) -> C19666
- D5: LCSC (none) -> C308725
- J3: LCSC Part # (none) -> C722767
- Q1: LCSC (none) -> C15127
- R5: LCSC (none) -> C23018
- R6: value 2.2k -> 22k; LCSC (none) -> C4190
- R7: LCSC (none) -> C22906
- R8: LCSC (none) -> C21190
- U3: LCSC (none) -> C38066
Connections:
- net GND: now also C18.2
- net VCC: now also C18.1
Other:
- note added: "Compatible diode packages: - TUMD2M - Power-DI-323 - SOD-323HE"
Changed lines of the file:
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@@
     (stroke (width 0) (type default))
+  )
+  (text "Compatible diode packages:\n- TUMD2M\n- Power-DI-323\n- SOD-323HE"
+    (at 193.04 64.77 0)
+    (effects (font (size 1.27 1.27)) (justify left bottom))
   )
   (text "Actual 2.7uF" (at 34.29 81.28 0)
@@
       (effects (font (size 1.27 1.27)) hide)
     )
+    (property "LCSC" "C14663" (at 189.23 116.84 0)
+      (effects (font (size 1.27 1.27)) hide)
+    )
     (pin "1")
     (pin "2")
@@
       (effects (font (size 1.27 1.27)) hide)
     )
+    (property "LCSC" "C15127" (at 201.93 85.09 0)
+      (effects (font (size 1.27 1.27)) hide)
+    )
     (pin "1")
     (pin "2")
@@
       (effects (font (size 1.27 1.27)) hide)
     )
+    (property "LCSC" "C19666" (at 74.93 78.74 0)
+      (effects (font (size 1.27 1.27)) hide)
+    )
     (pin "1")
     (pin "2")
@@
       (effects (font (size 1.27 1.27)) hide)
     )
+    (property "LCSC" "C19666" (at 57.15 78.74 0)
+      (effects (font (size 1.27 1.27)) hide)
+    )
     (pin "1")
     (pin "2")
@@
     )
   )
+  (symbol (lib_id "Device:C_Polarized") (at 250.19 93.98 0) (unit 1)
+    (in_bom yes) (on_board yes) (dnp no) (fields_autoplaced)
+    (property "Reference" "C18" (at 254 91.821 0)
+      (effects (font (size 1.27 1.27)) (justify left))
+    )
+    (property "Value" "100uF 6.3V" (at 254 94.361 0)
+      (effects (font (size 1.27 1.27)) (justify left))
+    )
+    (property "Footprint" "Capacitor_Tantalum_SMD:CP_EIA-3528-15_AVX-H" (at 251.1552 97.79 0)
+      (effects (font (size 1.27 1.27)) hide)
+    )
+    (property "Datasheet" "~" (at 250.19 93.98 0)
+      (effects (font (size 1.27 1.27)) hide)
+    )
+    (property "LCSC" "C16133" (at 250.19 93.98 0)
+      (effects (font (size 1.27 1.27)) hide)
+    )
+    (pin "1")
+    (pin "2")
+    (instances
+      (project "night_light"
+        (path "/c8bb3ba9-1daa-4665-ae97-22c9ddbf6eee/c446dc9c-d1fa-44b7-bcc3-f2a9c3c4127e"
+          (reference "C18") (unit 1)
+        )
+      )
+    )
+  )
   (symbol (lib_id "Device:R") (at 201.93 118.11 0) (unit 1)
     (in_bom yes) (on_board yes) (dnp no) (fields_autoplaced)
@@
     )
     (property "LCSC Part #" "" (at 201.93 118.11 0)
+      (effects (font (size 1.27 1.27)) hide)
+    )
+    (property "LCSC" "C21190" (at 204.47 116.84 0)
       (effects (font (size 1.27 1.27)) hide)
     )
@@
     )
     (property "LCSC Part #" "" (at 125.73 77.47 0)
+      (effects (font (size 1.27 1.27)) hide)
+    )
+    (property "LCSC" "C38066" (at 127.7494 68.6902 0)
       (effects (font (size 1.27 1.27)) hide)
     )
@@
     )
   )
-  (symbol (lib_id "Device:C_Polarized") (at 250.19 93.98 0) (unit 1)
-    (in_bom yes) (on_board yes) (dnp no) (fields_autoplaced)
-    (property "Reference" "C11" (at 254 91.821 0)
-      (effects (font (size 1.27 1.27)) (justify left))
-    )
-    (property "Value" "220u 6.3V" (at 254 94.361 0)
-      (effects (font (size 1.27 1.27)) (justify left))
-    )
-    (property "Footprint" "Capacitor_SMD:CP_Elec_6.3x5.7" (at 251.1552 97.79 0)
-      (effects (font (size 1.27 1.27)) hide)
-    )
-    (property "Datasheet" "~" (at 250.19 93.98 0)
-      (effects (font (size 1.27 1.27)) hide)
-    )
-    (property "LCSC Part #" "" (at 250.19 93.98 0)
-      (effects (font (size 1.27 1.27)) hide)
-    )
-    (pin "1")
-    (pin "2")
-    (instances
-      (project "night_light"
-        (path "/c8bb3ba9-1daa-4665-ae97-22c9ddbf6eee/c446dc9c-d1fa-44b7-bcc3-f2a9c3c4127e"
-          (reference "C11") (unit 1)
-        )
-      )
-    )
-  )
   (symbol (lib_id "power:GND") (at 250.19 97.79 0) (unit 1)
     (in_bom yes) (on_board yes) (dnp no) (fields_autoplaced)
@@
       (effects (font (size 1.27 1.27)) hide)
     )
+    (property "LCSC" "C19666" (at 234.95 92.71 0)
+      (effects (font (size 1.27 1.27)) hide)
+    )
     (pin "1")
     (pin "2")
@@
       (effects (font (size 1.27 1.27)) hide)
     )
+    (property "LCSC" "C308725" (at 203.5175 74.93 0)
+      (effects (font (size 1.27 1.27)) hide)
+    )
     (pin "1")
     (pin "2")
@@
       (effects (font (size 1.27 1.27)))
     )
-    (property "Value" "2.2k" (at 149.86 76.2 90)
+    (property "Value" "22k" (at 149.86 76.2 90)
       (effects (font (size 1.27 1.27)))
     )
@@
       (effects (font (size 1.27 1.27)) hide)
     )
+    (property "LCSC" "C4190" (at 149.86 73.66 0)
+      (effects (font (size 1.27 1.27)) hide)
+    )
     (pin "1")
     (pin "2")
@@
       (effects (font (size 1.27 1.27)) hide)
     )
-    (property "LCSC Part #" "" (at 93.98 81.28 0)
+    (property "LCSC Part #" "C722767" (at 93.98 81.28 0)
       (effects (font (size 1.27 1.27)) hide)
     )
@@
       (effects (font (size 1.27 1.27)) hide)
     )
+    (property "LCSC" "C23018" (at 115.57 85.09 0)
+      (effects (font (size 1.27 1.27)) hide)
+    )
     (pin "1")
     (pin "2")
@@
       (effects (font (size 1.27 1.27)) hide)
     )
+    (property "LCSC" "C22906" (at 204.47 104.14 0)
+      (effects (font (size 1.27 1.27)) hide)
+    )

Commit message: working
Other:
- note removed: "1.1V reference (1.0V min / 1.2V max) 4.5V input 100mV margin = 1.3V"

Commit message: Night Light firmware
Parts:
- U3: value MCP73832-2-OT -> MCP73832T-2ACI/OT
Changed lines of the file:
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@@
 (kicad_sch
-	(version 20231120)
+	(version 20250114)
 	(generator "eeschema")
-	(generator_version "8.0")
+	(generator_version "9.0")
 	(paper "A4")
+	(text "Compatible diode packages:\n- TUMD2M\n- Power-DI-323\n- SOD-323HE"
+		(exclude_from_sim no)
+		(at 193.04 64.77 0)
+		(effects
+			(font
+				(size 1.27 1.27)
+			)
+			(justify left bottom)
+		)
+	)
+	(text "Actual 2.7uF"
+		(exclude_from_sim no)
+		(at 34.29 81.28 0)
+		(effects
+			(font
+				(size 1.27 1.27)
+			)
+			(justify left bottom)
+		)
+	)
+	(text "I_chg=~250mA"
+		(exclude_from_sim no)
+		(at 110.49 99.06 0)
+		(effects
+			(font
+				(size 1.27 1.27)
+			)
+			(justify left bottom)
+		)
+	)
+	(text "heatsink on source"
+		(exclude_from_sim no)
+		(at 207.01 97.79 0)
+		(effects
+			(font
+				(size 1.27 1.27)
+			)
+			(justify left bottom)
+		)
+	)
+	(text_box "If using the analog comparator:\n	1.1V reference (1.0V min / 1.2V max)\n	4.5V input\n	100mV margin\n	= 1.3V\nIf using the ADC:\n	\n\n75uA reverse corrent through D5 -> 75mV"
+		(exclude_from_sim no)
+		(at 215.9 127 0)
+		(size 50.8 25.4)
+		(margins 0.9525 0.9525 0.9525 0.9525)
+		(stroke
+			(width 0)
+			(type default)
+		)
+		(fill
+			(type none)
+		)
+		(effects
+			(font
+				(size 1.27 1.27)
+			)
+			(justify left top)
+		)
+	)
+	(text_box "Device:\n	MCP73831:	Single-Cell Charge Controller\n	MCP73831T:	Single-Cell Charge Controller (Tape and Reel)\n	MCP73832:	Single-Cell Charge Controller\n	MCP73832T:	Single-Cell Charge Controller (Tape and Reel)\n\n(MCP73832 is open drain. MCP73831 is push-pull.)\n\nRegulation Voltage:\n	Code	V_{REG}\n	2		4.20V\n	3		4.35V\n	4		4.40V\n	5		4.50V\n\nOptions:\n	Code	I_{PREG}/I_{REG}	V_{PTH}/V_{REG}	I_{TERM}/I_{REG}	V_{RTH}/V_{REG}\n	AC		10			66.5		7.5			96.5\n	AD		10			66.5		7.5			94\n	AT		10			71.5		20			94\n	DC		100			x			7.5			96.5\n\nTemperature Range:\n	I = -40°C to +85°C (Industrial)\n\nPackage:\n	MC = Dual-Flat, No-Lead (2x3 mm body), 8-Lead\n	OT = Small Outline Transistor (SOT23), 5-Lead"
+		(exclude_from_sim no)
+		(at 25.4 114.3 0)
+		(size 86.36 58.42)
+		(margins 0.9525 0.9525 0.9525 0.9525)
+		(stroke
+			(width 0)
+			(type solid)
+		)
+		(fill
+			(type none)
+		)
+		(effects
+			(font
+				(face "KiCad Font")
+				(size 1.27 1.27)
+			)
+			(justify left top)
+		)
+	)
 	(junction
 		(at 209.55 81.28)
@@
 		)
 	)
-	(text_box "If using the analog comparator:\n	1.1V reference (1.0V min / 1.2V max)\n	4.5V input\n	100mV margin\n	= 1.3V\nIf using the ADC:\n	\n\n75uA reverse corrent through D5 -> 75mV"
-		(exclude_from_sim no)
-		(at 215.9 127 0)
-		(size 50.8 25.4)
-		(stroke
-			(width 0)
-			(type default)
-		)
-		(fill
-			(type none)
-		)
+	(label "PROG"
+		(at 113.03 80.01 180)
 		(effects
 			(font
 				(size 1.27 1.27)
 			)
-			(justify left top)
-		)
-	)
-	(text "Compatible diode packages:\n- TUMD2M\n- Power-DI-323\n- SOD-323HE"
-		(exclude_from_sim no)
-		(at 193.04 64.77 0)
+			(justify right bottom)
+		)
+	)
+	(hierarchical_label "V_{SEN}"
+		(shape output)
+		(at 214.63 111.76 0)
 		(effects
 			(font
 				(size 1.27 1.27)
 			)
-			(justify left bottom)
-		)
-	)
-	(text "Actual 2.7uF"
-		(exclude_from_sim no)
-		(at 34.29 81.28 0)
-		(effects
-			(font
-				(size 1.27 1.27)
-			)
-			(justify left bottom)
-		)
-	)
-	(text "I_chg=~250mA"
-		(exclude_from_sim no)
-		(at 110.49 99.06 0)
-		(effects
-			(font
-				(size 1.27 1.27)
-			)
-			(justify left bottom)
-		)
-	)
-	(text "heatsink on source"
-		(exclude_from_sim no)
-		(at 207.01 97.79 0)
-		(effects
-			(font
-				(size 1.27 1.27)
-			)
-			(justify left bottom)
-		)
-	)
-	(label "PROG"
-		(at 113.03 80.01 180)
-		(fields_autoplaced yes)
-		(effects
-			(font
-				(size 1.27 1.27)
-			)
-			(justify right bottom)
-		)
-	)
-	(hierarchical_label "V_{SEN}"
-		(shape output)
-		(at 214.63 111.76 0)
-		(fields_autoplaced yes)
-		(effects
-			(font
-				(size 1.27 1.27)
-			)
 			(justify left)
 		)
@@
 		(shape output)
 		(at 140.97 86.36 0)
-		(fields_autoplaced yes)
 		(effects
 			(font
@@
 		(on_board yes)
 		(dnp no)
-		(fields_autoplaced yes)
 		(property "Reference" "U3"
-			(at 127.7494 68.6902 0)
+			(at 127.8733 67.31 0)
 			(effects
 				(font
@@
 			)
 		)
-		(property "Value" "MCP73832-2-OT"
-			(at 127.7494 71.2271 0)
-			(effects
-				(font
+		(property "Value" "MCP73832T-2ACI/OT"
+			(at 116.078 63.5 0)
+			(effects
+				(font
