File: hardware/night_light/input.kicad_sch (KiCad schematic)
At the start: 5 parts, among them J2 Screw_Terminal_01x02

Commit message: night light ready
Parts:
- added C10: 1n 1kV, Capacitor_SMD:C_0603_1608Metric, symbol Device:C
- D1: value D_Zener -> SMAJ40A
- F1: value Fuse -> 0468.500NRHF
Connections:
- net +24V: no longer D1.1 (K)
- net GND: now also C10.2
- net Vin: now reaches F1.1, J2.2 (Pin_2), TP1.1
- net Vin: now also D1.1 (K), C10.1
Other:
- moved on the sheet: D1, F1, TP1, TP2

Commit message: various
Parts:
- removed TP1: V_{IN}, prj_lib:TestPoint_THTPad_D1.0mm_Drill0.5mm, symbol Connector:TestPoint
- removed TP2: V_{FS}, prj_lib:TestPoint_THTPad_D1.0mm_Drill0.5mm, symbol Connector:TestPoint
- added C11: C_Polarized, Capacitor_THT:C_Disc_D3.0mm_W1.6mm_P2.50mm, symbol Device:C_Polarized
- C10: LCSC (none) -> C14663
- D1: LCSC (none) -> C134985
Connections:
- net +24V: now also C11.1
- net GND: now also C11.2
Changed lines of the file:
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@@
 (kicad_sch (version 20230121) (generator eeschema)
   (paper "A4")
-  (junction (at 140.97 80.01) (diameter 0) (color 0 0 0 0)
+  (junction (at 157.48 80.01) (diameter 0) (color 0 0 0 0)
   )
   (junction (at 116.84 80.01) (diameter 0) (color 0 0 0 0)
@@
   (junction (at 128.27 80.01) (diameter 0) (color 0 0 0 0)
   )
-  (wire (pts (xy 140.97 74.93) (xy 140.97 80.01))
-    (stroke (width 0) (type default))
-  )
-  (wire (pts (xy 157.48 80.01) (xy 140.97 80.01))
+  (wire (pts (xy 138.43 80.01) (xy 157.48 80.01))
     (stroke (width 0) (type default))
   )
@@
     (stroke (width 0) (type default))
   )
+  (wire (pts (xy 157.48 80.01) (xy 157.48 82.55))
+    (stroke (width 0) (type default))
+  )
   (wire (pts (xy 116.84 82.55) (xy 116.84 80.01))
     (stroke (width 0) (type default))
   )
   (wire (pts (xy 111.76 82.55) (xy 109.22 82.55))
-    (stroke (width 0) (type default))
-  )
-  (wire (pts (xy 116.84 74.93) (xy 116.84 80.01))
-    (stroke (width 0) (type default))
-  )
-  (wire (pts (xy 138.43 80.01) (xy 140.97 80.01))
     (stroke (width 0) (type default))
   )
@@
     (effects (font (size 1.27 1.27)) (justify left bottom))
   )
+  (symbol (lib_id "Device:C_Polarized") (at 157.48 86.36 0) (unit 1)
+    (in_bom yes) (on_board yes) (dnp no) (fields_autoplaced)
+    (property "Reference" "C11" (at 161.29 84.201 0)
+      (effects (font (size 1.27 1.27)) (justify left))
+    )
+    (property "Value" "C_Polarized" (at 161.29 86.741 0)
+      (effects (font (size 1.27 1.27)) (justify left))
+    )
+    (property "Footprint" "Capacitor_THT:C_Disc_D3.0mm_W1.6mm_P2.50mm" (at 158.4452 90.17 0)
+      (effects (font (size 1.27 1.27)) hide)
+    )
+    (property "Datasheet" "~" (at 157.48 86.36 0)
+      (effects (font (size 1.27 1.27)) hide)
+    )
+    (pin "1")
+    (pin "2")
+    (instances
+      (project "night_light"
+        (path "/c8bb3ba9-1daa-4665-ae97-22c9ddbf6eee/eed5a22c-e790-43f8-b267-77806927c9e9"
+          (reference "C11") (unit 1)
+        )
+      )
+    )
+  )
   (symbol (lib_id "Device:D_Zener") (at 116.84 86.36 270) (unit 1)
     (in_bom yes) (on_board yes) (dnp no) (fields_autoplaced)
@@
       (effects (font (size 1.27 1.27)) hide)
     )
+    (property "LCSC" "C134985" (at 119.38 85.09 0)
+      (effects (font (size 1.27 1.27)) hide)
+    )
     (pin "1")
     (pin "2")
@@
     )
   )
-  (symbol (lib_id "Connector:TestPoint") (at 116.84 74.93 0) (unit 1)
-    (in_bom yes) (on_board yes) (dnp no) (fields_autoplaced)
-    (property "Reference" "TP1" (at 118.237 70.7933 0)
-      (effects (font (size 1.27 1.27)) (justify left))
-    )
-    (property "Value" "V_{IN}" (at 118.237 73.3302 0)
-      (effects (font (size 1.27 1.27)) (justify left))
-    )
-    (property "Footprint" "prj_lib:TestPoint_THTPad_D1.0mm_Drill0.5mm" (at 121.92 74.93 0)
-      (effects (font (size 1.27 1.27)) hide)
-    )
-    (property "Datasheet" "~" (at 121.92 74.93 0)
-      (effects (font (size 1.27 1.27)) hide)
-    )
-    (property "LCSC Part #" "" (at 116.84 74.93 0)
-      (effects (font (size 1.27 1.27)) hide)
-    )
-    (pin "1")
-    (instances
-      (project "night_light"
-        (path "/c8bb3ba9-1daa-4665-ae97-22c9ddbf6eee/eed5a22c-e790-43f8-b267-77806927c9e9"
-          (reference "TP1") (unit 1)
-        )
-      )
-    )
-  )
-  (symbol (lib_id "Connector:TestPoint") (at 140.97 74.93 0) (unit 1)
-    (in_bom yes) (on_board yes) (dnp no) (fields_autoplaced)
-    (property "Reference" "TP2" (at 142.367 70.7933 0)
-      (effects (font (size 1.27 1.27)) (justify left))
-    )
-    (property "Value" "V_{FS}" (at 142.367 73.3302 0)
-      (effects (font (size 1.27 1.27)) (justify left))
-    )
-    (property "Footprint" "prj_lib:TestPoint_THTPad_D1.0mm_Drill0.5mm" (at 146.05 74.93 0)
-      (effects (font (size 1.27 1.27)) hide)
-    )
-    (property "Datasheet" "~" (at 146.05 74.93 0)
-      (effects (font (size 1.27 1.27)) hide)
-    )
-    (property "LCSC Part #" "" (at 140.97 74.93 0)
-      (effects (font (size 1.27 1.27)) hide)
-    )
-    (pin "1")
-    (instances
-      (project "night_light"
-        (path "/c8bb3ba9-1daa-4665-ae97-22c9ddbf6eee/eed5a22c-e790-43f8-b267-77806927c9e9"
-          (reference "TP2") (unit 1)
-        )
-      )
-    )
-  )
   (symbol (lib_id "power:GND") (at 116.84 90.17 0) (unit 1)
     (in_bom yes) (on_board yes) (dnp no) (fields_autoplaced)
@@
     )
   )
+  (symbol (lib_id "power:GND") (at 157.48 90.17 0) (unit 1)
+    (in_bom yes) (on_board yes) (dnp no) (fields_autoplaced)
+    (property "Reference" "#PWR014" (at 157.48 96.52 0)
+      (effects (font (size 1.27 1.27)) hide)
+    )
+    (property "Value" "GND" (at 157.48 94.6134 0)
+      (effects (font (size 1.27 1.27)))
+    )
+    (property "Footprint" "" (at 157.48 90.17 0)
+      (effects (font (size 1.27 1.27)) hide)
+    )
+    (property "Datasheet" "" (at 157.48 90.17 0)
+      (effects (font (size 1.27 1.27)) hide)
+    )
+    (pin "1")
+    (instances
+      (project "night_light"
+        (path "/c8bb3ba9-1daa-4665-ae97-22c9ddbf6eee/eed5a22c-e790-43f8-b267-77806927c9e9"
+          (reference "#PWR014") (unit 1)
+        )
+      )
+    )
+  )
   (symbol (lib_id "power:GND") (at 128.27 90.17 0) (unit 1)
     (in_bom yes) (on_board yes) (dnp no) (fields_autoplaced)
@@
       (effects (font (size 1.27 1.27)) hide)
     )
+    (property "LCSC" "C14663" (at 132.08 85.09 0)
+      (effects (font (size 1.27 1.27)) hide)
+    )

Commit message: working
Parts:
- renumbered C10 to C4
