File: hardware/night_light/mcu.kicad_sch (KiCad schematic)
At the start: 9 parts, among them J4 AVR-ISP-6, SW1 TS-1088, U5 ATtiny13A-SS

Commit message: various
Parts:
- C15, C17: LCSC (none) -> C14663
- R10: LCSC (none) -> C25804
- R13, R14: LCSC (none) -> C21190
- R9: LCSC (none) -> C25803
- SW1: LCSC (none) -> C455280
- U5: LCSC (none) -> C14075
Connections:
- net PB1: now also R14.1; no longer R13.1
- net PB2: now also R13.1; no longer R14.1
Changed lines of the file:
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@@
     (effects (font (size 1.27 1.27)) (justify left bottom))
   )
-  (label "PB1" (at 162.56 76.2 180) (fields_autoplaced)
+  (label "PB1" (at 162.56 85.09 180) (fields_autoplaced)
     (effects (font (size 1.27 1.27)) (justify right bottom))
   )
@@
     (effects (font (size 1.27 1.27)) (justify right bottom))
   )
-  (label "PB2" (at 162.56 85.09 180) (fields_autoplaced)
+  (label "PB2" (at 162.56 76.2 180) (fields_autoplaced)
     (effects (font (size 1.27 1.27)) (justify right bottom))
   )
@@
       (effects (font (size 1.27 1.27)) hide)
     )
+    (property "LCSC" "C25804" (at 147.32 30.48 0)
+      (effects (font (size 1.27 1.27)) hide)
+    )
     (pin "1")
     (pin "2")
@@
     )
     (property "LCSC Part #" "" (at 190.5 38.1 0)
+      (effects (font (size 1.27 1.27)) hide)
+    )
+    (property "LCSC" "C14663" (at 194.31 36.83 0)
       (effects (font (size 1.27 1.27)) hide)
     )
@@
       (effects (font (size 1.27 1.27)) hide)
     )
+    (property "LCSC" "C25803" (at 151.13 44.45 0)
+      (effects (font (size 1.27 1.27)) hide)
+    )
     (pin "1")
     (pin "2")
@@
       (effects (font (size 1.27 1.27)) hide)
     )
+    (property "LCSC" "C14663" (at 161.29 43.18 0)
+      (effects (font (size 1.27 1.27)) hide)
+    )
     (pin "1")
     (pin "2")
@@
       (effects (font (size 1.27 1.27)) hide)
     )
+    (property "LCSC" "C21190" (at 168.91 78.74 0)
+      (effects (font (size 1.27 1.27)) hide)
+    )
     (pin "1")
     (pin "2")
@@
     )
     (property "LCSC Part #" "" (at 168.91 76.2 0)
+      (effects (font (size 1.27 1.27)) hide)
+    )
+    (property "LCSC" "C21190" (at 168.91 69.85 0)
       (effects (font (size 1.27 1.27)) hide)
     )
@@
     )
     (property "LCSC Part #" "" (at 123.19 83.82 0)
+      (effects (font (size 1.27 1.27)) hide)
+    )
+    (property "LCSC" "C14075" (at 109.728 82.9853 0)
       (effects (font (size 1.27 1.27)) hide)
     )
@@
       (effects (font (size 1.27 1.27)) hide)
     )
+    (property "LCSC" "C455280" (at 137.16 30.48 0)
+      (effects (font (size 1.27 1.27)) hide)
+    )
