File: hardware/night_light/vreg.kicad_sch (KiCad schematic)
At the start: 9 parts, among them U1 TD1465

Commit message: night light ready
Parts:
- C1: value 10u -> 10u 50V
- C2: value 100n -> 100n 50V
- C3: value 22u -> 22u 10V
- L1: value 22u -> CBC3225T220KR; L (none) -> 22u
- R2: value 47k -> 100k
- R3: value 10k -> 22k
- U1: value TD1465 -> TD1469
Other:
- note added: "FB=0,812V Vout=4,5V"
- note removed: "FB=0,8V Vout=4,56V"
Changed lines of the file:
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@@
     (stroke (width 0) (type default))
   )
-  (text "FB=0,8V\nVout=4,56V" (at 106.68 120.65 0)
+  (text "FB=0,812V\nVout=4,5V" (at 106.68 120.65 0)
     (effects (font (size 1.27 1.27)) (justify left bottom))
   )
@@
   (symbol (lib_id "Device:C") (at 50.8 114.3 180) (unit 1)
     (in_bom yes) (on_board yes) (dnp no) (fields_autoplaced)
-    (property "Reference" "C1" (at 53.721 113.4653 0)
+    (property "Reference" "C1" (at 54.61 113.03 0)
       (effects (font (size 1.27 1.27)) (justify right))
     )
-    (property "Value" "10u" (at 53.721 116.0022 0)
+    (property "Value" "10u 50V" (at 54.61 115.57 0)
       (effects (font (size 1.27 1.27)) (justify right))
     )
@@
       (effects (font (size 1.27 1.27)) hide)
     )
+    (property "LCSC Part #" "" (at 50.8 114.3 0)
+      (effects (font (size 1.27 1.27)) hide)
+    )
     (pin "1")
     (pin "2")
@@
   (symbol (lib_id "Device:R") (at 127 132.08 0) (unit 1)
     (in_bom yes) (on_board yes) (dnp no) (fields_autoplaced)
-    (property "Reference" "R3" (at 128.778 131.2453 0)
-      (effects (font (size 1.27 1.27)) (justify left))
-    )
-    (property "Value" "10k" (at 128.778 133.7822 0)
+    (property "Reference" "R3" (at 129.54 130.81 0)
+      (effects (font (size 1.27 1.27)) (justify left))
+    )
+    (property "Value" "22k" (at 129.54 133.35 0)
       (effects (font (size 1.27 1.27)) (justify left))
     )
@@
       (effects (font (size 1.27 1.27)) hide)
     )
+    (property "LCSC Part #" "" (at 127 132.08 0)
+      (effects (font (size 1.27 1.27)) hide)
+    )
     (pin "1")
     (pin "2")
@@
   (symbol (lib_id "Device:R") (at 127 121.92 0) (unit 1)
     (in_bom yes) (on_board yes) (dnp no) (fields_autoplaced)
-    (property "Reference" "R2" (at 128.778 121.0853 0)
-      (effects (font (size 1.27 1.27)) (justify left))
-    )
-    (property "Value" "47k" (at 128.778 123.6222 0)
+    (property "Reference" "R2" (at 129.54 120.65 0)
+      (effects (font (size 1.27 1.27)) (justify left))
+    )
+    (property "Value" "100k" (at 129.54 123.19 0)
       (effects (font (size 1.27 1.27)) (justify left))
     )
@@
       (effects (font (size 1.27 1.27)) hide)
     )
+    (property "LCSC Part #" "" (at 127 121.92 0)
+      (effects (font (size 1.27 1.27)) hide)
+    )
     (pin "1")
     (pin "2")
@@
   (symbol (lib_id "Device:C") (at 137.16 106.68 180) (unit 1)
     (in_bom yes) (on_board yes) (dnp no) (fields_autoplaced)
-    (property "Reference" "C3" (at 140.081 105.8453 0)
+    (property "Reference" "C3" (at 140.97 105.41 0)
       (effects (font (size 1.27 1.27)) (justify right))
     )
-    (property "Value" "22u" (at 140.081 108.3822 0)
+    (property "Value" "22u 10V" (at 140.97 107.95 0)
       (effects (font (size 1.27 1.27)) (justify right))
     )
@@
       (effects (font (size 1.27 1.27)) hide)
     )
+    (property "LCSC Part #" "" (at 137.16 106.68 0)
+      (effects (font (size 1.27 1.27)) hide)
+    )
     (pin "1")
     (pin "2")
@@
   (symbol (lib_id "Device:C") (at 118.11 100.33 90) (unit 1)
     (in_bom yes) (on_board yes) (dnp no) (fields_autoplaced)
-    (property "Reference" "C2" (at 118.11 94.4712 90)
-      (effects (font (size 1.27 1.27)))
-    )
-    (property "Value" "100n" (at 118.11 97.0081 90)
+    (property "Reference" "C2" (at 118.11 92.71 90)
+      (effects (font (size 1.27 1.27)))
+    )
+    (property "Value" "100n 50V" (at 118.11 95.25 90)
       (effects (font (size 1.27 1.27)))
     )
@@
       (effects (font (size 1.27 1.27)) hide)
     )
+    (property "LCSC Part #" "" (at 118.11 100.33 0)
+      (effects (font (size 1.27 1.27)) hide)
+    )
     (pin "1")
     (pin "2")
@@
       (effects (font (size 1.27 1.27)) hide)
     )
+    (property "LCSC Part #" "" (at 139.7 100.33 0)
+      (effects (font (size 1.27 1.27)) hide)
+    )
     (pin "1")
     (instances
@@
   )
   (symbol (lib_id "Device:L") (at 130.81 100.33 90) (unit 1)
-    (in_bom yes) (on_board yes) (dnp no) (fields_autoplaced)
-    (property "Reference" "L1" (at 130.81 96.1222 90)
-      (effects (font (size 1.27 1.27)))
-    )
-    (property "Value" "22u" (at 130.81 98.6591 90)
+    (in_bom yes) (on_board yes) (dnp no)
+    (property "Reference" "L1" (at 130.81 95.25 90)
+      (effects (font (size 1.27 1.27)))
+    )
+    (property "Value" "CBC3225T220KR" (at 130.81 97.79 90)
       (effects (font (size 1.27 1.27)))
     )
@@
       (effects (font (size 1.27 1.27)) hide)
     )
+    (property "LCSC Part #" "" (at 130.81 100.33 0)
+      (effects (font (size 1.27 1.27)) hide)
+    )
+    (property "L" "22u" (at 130.81 102.87 90) (show_name)
+      (effects (font (size 1.27 1.27)))
+    )
     (pin "1")
     (pin "2")
@@
     )
     (property "Datasheet" "~" (at 80.01 109.22 0)
+      (effects (font (size 1.27 1.27)) hide)
+    )
+    (property "LCSC Part #" "" (at 80.01 109.22 0)
       (effects (font (size 1.27 1.27)) hide)
     )
@@
       (effects (font (size 1.27 1.27)))
     )
-    (property "Value" "TD1465" (at 99.06 101.6 0)
+    (property "Value" "TD1469" (at 99.06 101.6 0)
       (effects (font (size 1.27 1.27)))
     )
@@
       (effects (font (size 1.27 1.27)) hide)
     )
+    (property "LCSC Part #" "" (at 99.06 109.22 0)
+      (effects (font (size 1.27 1.27)) hide)
+    )

Commit message: various
Parts:
- added C12: 22u 10V, Capacitor_SMD:C_0805_2012Metric, symbol Device:C
- C1: LCSC (none) -> C13585
- C2: LCSC (none) -> C14663
- C3: LCSC (none) -> C29277
- L1: LCSC (none) -> C223225
- R1: LCSC (none) -> C22935
- R2: LCSC (none) -> C25803
- R3: LCSC (none) -> C31850
- U1: LCSC (none) -> C2832208
Connections:
- net +5V: now also C12.2
- net GND: now also C12.1
Changed lines of the file:
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@@
+      (effects (font (size 1.27 1.27)) hide)
+    )
+    (property "LCSC" "C13585" (at 54.61 113.03 0)
       (effects (font (size 1.27 1.27)) hide)
     )
@@
       (effects (font (size 1.27 1.27)) hide)
     )
+    (property "LCSC" "C31850" (at 129.54 130.81 0)
+      (effects (font (size 1.27 1.27)) hide)
+    )
     (pin "1")
     (pin "2")
@@
     )
     (property "LCSC Part #" "" (at 127 121.92 0)
+      (effects (font (size 1.27 1.27)) hide)
+    )
+    (property "LCSC" "C25803" (at 129.54 120.65 0)
       (effects (font (size 1.27 1.27)) hide)
     )
@@
       (effects (font (size 1.27 1.27)) hide)
     )
+    (property "LCSC" "C29277" (at 140.97 105.41 0)
+      (effects (font (size 1.27 1.27)) hide)
+    )
     (pin "1")
     (pin "2")
@@
     )
   )
+  (symbol (lib_id "Device:C") (at 153.67 106.68 180) (unit 1)
+    (in_bom yes) (on_board yes) (dnp no) (fields_autoplaced)
+    (property "Reference" "C12" (at 157.48 105.41 0)
+      (effects (font (size 1.27 1.27)) (justify right))
+    )
+    (property "Value" "22u 10V" (at 157.48 107.95 0)
+      (effects (font (size 1.27 1.27)) (justify right))
+    )
+    (property "Footprint" "Capacitor_SMD:C_0805_2012Metric" (at 152.7048 102.87 0)
+      (effects (font (size 1.27 1.27)) hide)
+    )
+    (property "Datasheet" "~" (at 153.67 106.68 0)
+      (effects (font (size 1.27 1.27)) hide)
+    )
+    (property "LCSC Part #" "" (at 153.67 106.68 0)
+      (effects (font (size 1.27 1.27)) hide)
+    )
+    (property "LCSC" "C29277" (at 157.48 105.41 0)
+      (effects (font (size 1.27 1.27)) hide)
+    )
+    (pin "1")
+    (pin "2")
+    (instances
+      (project "night_light"
+        (path "/c8bb3ba9-1daa-4665-ae97-22c9ddbf6eee/54bb5b8e-b8b2-4417-ae30-f2c2986dc27a"
+          (reference "C12") (unit 1)
+        )
+      )
+    )
+  )
   (symbol (lib_id "Device:C") (at 118.11 100.33 90) (unit 1)
     (in_bom yes) (on_board yes) (dnp no) (fields_autoplaced)
@@
     )
     (property "LCSC Part #" "" (at 118.11 100.33 0)
+      (effects (font (size 1.27 1.27)) hide)
+    )
+    (property "LCSC" "C14663" (at 118.11 92.71 0)
       (effects (font (size 1.27 1.27)) hide)
     )
@@
       (effects (font (size 1.27 1.27)))
     )
+    (property "LCSC" "C223225" (at 130.81 95.25 0)
+      (effects (font (size 1.27 1.27)) hide)
+    )
     (pin "1")
     (pin "2")
@@
       (effects (font (size 1.27 1.27)) hide)
     )
+    (property "LCSC" "C22935" (at 80.01 104.5042 0)
+      (effects (font (size 1.27 1.27)) hide)
+    )
     (pin "1")
     (pin "2")
@@
         (path "/c8bb3ba9-1daa-4665-ae97-22c9ddbf6eee/54bb5b8e-b8b2-4417-ae30-f2c2986dc27a"
           (reference "#PWR08") (unit 1)
+        )
+      )
+    )
+  )
+  (symbol (lib_id "power:+5V") (at 153.67 102.87 0) (unit 1)
+    (in_bom yes) (on_board yes) (dnp no) (fields_autoplaced)
+    (property "Reference" "#PWR015" (at 153.67 106.68 0)
+      (effects (font (size 1.27 1.27)) hide)
+    )
+    (property "Value" "+5V" (at 153.67 99.2942 0)
+      (effects (font (size 1.27 1.27)))
+    )
+    (property "Footprint" "" (at 153.67 102.87 0)
+      (effects (font (size 1.27 1.27)) hide)
+    )
+    (property "Datasheet" "" (at 153.67 102.87 0)
+      (effects (font (size 1.27 1.27)) hide)
+    )
+    (pin "1")
+    (instances
+      (project "night_light"
+        (path "/c8bb3ba9-1daa-4665-ae97-22c9ddbf6eee/54bb5b8e-b8b2-4417-ae30-f2c2986dc27a"
+          (reference "#PWR015") (unit 1)
         )
       )
@@
     )
     (property "LCSC Part #" "" (at 99.06 109.22 0)
+      (effects (font (size 1.27 1.27)) hide)
+    )
+    (property "LCSC" "C2832208" (at 99.06 99.06 0)
       (effects (font (size 1.27 1.27)) hide)
     )
@@
         )
       )
+    )
+  )
+  (symbol (lib_id "power:GND") (at 153.67 110.49 0) (unit 1)
+    (in_bom yes) (on_board yes) (dnp no) (fields_autoplaced)
+    (property "Reference" "#PWR013" (at 153.67 116.84 0)
+      (effects (font (size 1.27 1.27)) hide)
+    )
+    (property "Value" "GND" (at 153.67 114.9334 0)
+      (effects (font (size 1.27 1.27)))
+    )
+    (property "Footprint" "" (at 153.67 110.49 0)
+      (effects (font (size 1.27 1.27)) hide)
+    )
+    (property "Datasheet" "" (at 153.67 110.49 0)
+      (effects (font (size 1.27 1.27)) hide)
+    )
+    (pin "1")
+    (instances
+      (project "night_light"
+        (path "/c8bb3ba9-1daa-4665-ae97-22c9ddbf6eee/54bb5b8e-b8b2-4417-ae30-f2c2986dc27a"
+          (reference "#PWR013") (unit 1)
+        )
+      )

Commit message: working
Other:
- note added: "UVLO: 5.5V / 6V"
