File: hardware/night_light/night_light.kicad_pcb (KiCad board)
At the start: 2 copper layers, 22 x 40 mm, 59 parts, among them J1 RDB223, J2 Screw_Terminal_01x02, J3 Conn_01x02_Male, J4 AVR-ISP-6, Q1 Q_PMOS_GSD, SW1 SW_Push, U1 TD1465, U2 MT9284CS6, U3 MCP73832-2-OT, U4 LMV321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

Commit message: night light ready
Parts:
- added C4: 1n 1kV, Capacitor_SMD:C_0603_1608Metric, F.Cu at (117.0, 107.0)
- C1: value 10u -> 10u 50V
- C10, C12, C13, C14, C15, C16, C17: value C -> 100n 50V
- C11: value C_Polarized -> 220u 6.3V
- C2: value 100n -> 100n 50V
- C3: value 22u -> 22u 10V
- C5: value C -> 22u 10V
- C6: value C -> 10u 16V
- C7, C8, C9: value C -> 4.7u 16V
- D1: value D_Zener -> SMAJ40A
- D2: value 6V-150mA -> 6V 150mA
- D3, D5: value D_Schottky -> RB161VAM-20TR
- D6: value D_Photo -> TEPT5700
- F1: value Fuse -> 500mA
- J3: value Conn_01x02_Male -> JST PH
- L1, L2: value 22u -> CBC3225T220KR
- Q1: value Q_PMOS_GSD -> AO3401A
- R10: value R -> 10k
- R11: value R -> 1M
- R12: value R -> 68k
- R13, R14, R8: value R -> 1k
- R2: value 47k -> 100k
- R3: value 10k -> 22k
- R4: value 2 -> 0.7
- R5: value R -> 3.9k
- R6: value R -> 2.2k
- R7: value R -> 2.43k
- R9: value R -> 100k
- SW1: value SW_Push -> TS-1088
- U1: value TD1465 -> TD1469
- U2: value MT9284CS6 -> MT9284-28J
- U4: value LMV321 -> LMV321A
Connections:
- D1 pad 1: +24V -> /Input/Vin
- F1 pad 1: Net-(J2-Pin_2) -> /Input/Vin
- J2 pad 2: Net-(J2-Pin_2) -> /Input/Vin
- TP1 pad 1: Net-(J2-Pin_2) -> /Input/Vin
Routing:
- net Net-(J2-Pin_2): track 11.2 -> 0.00 mm
- net /Input/Vin: track 0.00 -> 6.05 mm
- net VCC: track 71.6 -> 68.8 mm
- net +5V: track 42.8 -> 42.3 mm
- added copper zone on F.Cu, net /Input/Vin

Commit message: various
Parts:
- removed R12: 68k, Resistor_SMD:R_0603_1608Metric
- removed TP1: V_{IN}, prj_lib:TestPoint_THTPad_D1.0mm_Drill0.5mm
- removed TP2: V_{FS}, prj_lib:TestPoint_THTPad_D1.0mm_Drill0.5mm
- removed TP7: PT_{OUT}, prj_lib:TestPoint_THTPad_D1.0mm_Drill0.5mm
- removed U4: LMV321A, Package_TO_SOT_SMD:SOT-23-5
- added C18: 100uF 6.3V, Capacitor_Tantalum_SMD:CP_EIA-3528-15_AVX-H, F.Cu at (123.2, 127.2)
- C11: value 220u 6.3V -> C_Polarized; footprint Capacitor_SMD:CP_Elec_6.3x5.7 -> Capacitor_THT:C_Disc_D3.0mm_W1.6mm_P2.50mm
- C12: value 100n 50V -> 22u 10V; footprint Capacitor_SMD:C_0603_1608Metric -> Capacitor_SMD:C_0805_2012Metric
- D6: footprint LED_THT:LED_D3.0mm_Clear -> LED_THT:LED_D3.0mm_FlatTop
- F1: value 500mA -> 0468.500NRHF
- R11: value 1M -> 1.83k
- R6: value 2.2k -> 22k
- moved C11 25.1 mm to (113.8, 107.0)
- moved C12 12.0 mm to (125.0, 106.0), turned to 180 degrees
- moved C4 10.4 mm to (118.8, 117.2), turned to -90 degrees
- moved D1 9.12 mm to (121.5, 114.0), turned to 0 degrees
- moved C15 3.85 mm to (125.8, 119.4), turned to -90 degrees
- moved C14 3.71 mm to (121.0, 117.2), turned to 90 degrees
- moved R11 3.25 mm to (122.5, 117.2), turned to -90 degrees
- moved F1 2.15 mm to (111.5, 108.5), turned to 90 degrees
- moved C13 1.85 mm to (124.0, 117.2), turned to -90 degrees
Connections:
- C11 pad 1: VCC -> +24V
- C12 pad 1: /sensors/PT- -> GND
- C12 pad 2: /sensors/PTout -> +5V
- D6 pad 1: /sensors/PT- -> VCC
- D6 pad 2: GND -> /ALS
- R11 pad 1: /sensors/PT- -> GND
- R11 pad 2: /sensors/PTout -> /ALS
- R13 pad 1: /MCU/PB1 -> /MCU/PB2
- R14 pad 1: /MCU/PB2 -> /MCU/PB1
Routing:
- net /sensors/PTout: track 8.81 -> 0.00 mm
- net VCC: track 68.8 -> 75.1 mm
- net /sensors/PT-: track 5.59 -> 0.00 mm
- net /Input/Vin: track 6.05 -> 11.1 mm
- net GND: track 0.00 -> 3.29 mm, vias 104 -> 91
- net /ALS: track 13.3 -> 16.2 mm
- net +24V: track 4.00 -> 6.34 mm
- net /MCU/PB2: track 14.8 -> 12.9 mm
- net /LED/LED+: track 7.26 -> 5.86 mm, vias 1 -> 5
- net /MCU/PB5: track 9.82 -> 9.66 mm, vias 0 -> 1
- net /LED/LED-: vias 0 -> 29
- added copper zone on F.Cu, net /LED/LED-

Commit message: working
Routing:
- net GND: vias 91 -> 148
Other:
- board text added: "I + C O R -"
- board text removed: "MI 3V CK MO RS V-"
