File: hardware/corridor_node/PWM2DC.kicad_sch (KiCad schematic)
At the start: 18 parts, among them U7 74LVC2G17, U8 LMV358

Commit message: nightLight pcb files version upgrade
Parts:
- renumbered C14 to C16, C14 to C17, C14 to C18, C14 to C19, C14 to C20, C14 to C21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
