File: hardware/corridor_node/corridor_node.kicad_sch (KiCad schematic)
At the start: 21 parts, among them J1 Screw_Terminal_01x06, J2 Screw_Terminal_01x04, U5 AP7384-50SA

Commit message: led balance and corridor ready
Parts:
- removed R3, R4: R, Resistor_SMD:R_0603_1608Metric_Pad0.98x0.95mm_HandSolder, symbol Device:R
- C1: value C_Polarized -> 470uF 50V; LCSC Part # (none) -> C88733
- C12, C13: value C -> 10u 50V; LCSC Part # (none) -> C440198
- C14: value C -> 22u 10V; LCSC Part # (none) -> C29277
- C6: value C -> 1n 1kV; LCSC Part # (none) -> C696365
- D1, D2: value D -> SM05; LCSC Part # (none) -> C460613
- D3: value D_Zener -> SMF36A; LCSC Part # (none) -> C374035
- F1: value Fuse -> 500mA; footprint Fuse:Fuse_0805_2012Metric_Pad1.15x1.40mm_HandSolder -> Fuse:Fuse_1206_3216Metric_Pad1.42x1.75mm_HandSolder; LCSC Part # (none) -> C206993
- FB1: value FerriteBead -> MMZ2012R102AT000; LCSC Part # (none) -> C76810
- J1: now left out of the parts list
- J2: LCSC Part # (none) -> C2757925; now left out of the parts list
- R6, R7: value R -> 100; LCSC Part # (none) -> C125923
- U5: LCSC Part # (none) -> C5370024
Other:
- added sheet PWM to DC (PWM2DC.kicad_sch)
